File: Flight Computer.kicad_sch (KiCad schematic)
At the start: 0 parts

Commit message: Schematics are love. Also I have no idea what I was doing last night so the power supply might be terrible, but I know I thought it was brilliant at the time
Parts:
- added U6: STM32L476VETx, Package_QFP:LQFP-100_14x14mm_P0.5mm, symbol MCU_ST_STM32L4:STM32L476VETx
Connections:
- new net: U6.10 (VSS), U6.27 (VSS), U6.49 (VSS), U6.74 (VSS), U6.99 (VSS)
Other:
- removed sheet Power Supply
- sheet Connectors ports: added External I2C SCL, External I2C SDA, External UART RX, External UART TX, Ignition Battery Voltage, NRST, Pyro Channel A, Pyro Channel B, Pyro Channel C, Pyro Channel D, Pyro Channel E, Pyro Channel F, SWCLK, SWDIO, SWO, USB D+, USB D-; removed none
- sheet Pyrotechnic Channels ports: added Pyro Channel A, Pyro Channel A Continuity Voltage, Pyro Channel A Trigger, Pyro Channel B, Pyro Channel B Continuity Voltage, Pyro Channel B Trigger, Pyro Channel C, Pyro Channel C Continuity Voltage, Pyro Channel C Trigger, Pyro Channel D, Pyro Channel D Continuity Voltage, Pyro Channel D Trigger, Pyro Channel E, Pyro Channel E Continuity Voltage, Pyro Channel E Trigger, Pyro Channel F, Pyro Channel F Continuity Voltage, Pyro Channel F Trigger; removed none
- sheet Sensors ports: added Altimeter Interrupt, Backup Battery, Chip Select Low G Accel, Chip Select Low G Gyro, GPS External Interrupt, GPS Reset, High G Interrupt 1, Low G Accel Interrupt 1, Low G Gyro Interrupt 3, Magnetometer Data Ready, Magnetometer Interrupt, SCL, SDA, SPI MISO, SPI MOSI, SPI SCK, UART RX, UART TX; removed none

Commit message: Began configuring STM32F476
Connections:
- net NRST: now reaches U6.14 (NRST)
- net Pyro A Continuity Voltage: now reaches U6.23 (PA0)
- net Pyro B Continuity Voltage: now reaches U6.24 (PA1)
- net Pyro C Continuity Voltage: now reaches U6.25 (PA2)
- net Pyro D Continuity Voltage: now reaches U6.26 (PA3)
- net Pyro E Continuity Voltage: now reaches U6.29 (PA4)
- net Pyro F Continuity Voltage: now reaches U6.30 (PA5)
- net Ignition Battery Voltage: now reaches U6.33 (PC4)
Other:
- sheet Connectors renamed Connectors and Power Supply
- moved on the sheet: U6

Commit message: --
Connections:
- net +3.3V: now reaches U6.100 (VDD)
- net +3.3V: now also U6.11 (VDD), U6.28 (VDD), U6.50 (VDD), U6.75 (VDD)
Changed lines of the file:
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@@
     (rev "1")
   )
+  (junction (at 92.71 31.75) (diameter 0) (color 0 0 0 0)
+  )
+  (junction (at 97.79 31.75) (diameter 0) (color 0 0 0 0)
+  )
+  (junction (at 90.17 31.75) (diameter 0) (color 0 0 0 0)
+  )
+  (junction (at 95.25 31.75) (diameter 0) (color 0 0 0 0)
+  )
   (wire (pts (xy 261.62 130.81) (xy 281.94 130.81))
     (stroke (width 0) (type default))
@@
     (stroke (width 0) (type default))
   )
+  (wire (pts (xy 100.33 34.29) (xy 100.33 31.75))
+    (stroke (width 0) (type default))
+  )
+  (wire (pts (xy 92.71 31.75) (xy 95.25 31.75))
+    (stroke (width 0) (type default))
+  )
   (wire (pts (xy 196.85 133.35) (xy 167.64 133.35))
     (stroke (width 0) (type default))
@@
     (stroke (width 0) (type default))
   )
+  (wire (pts (xy 90.17 25.4) (xy 90.17 31.75))
+    (stroke (width 0) (type default))
+  )
   (wire (pts (xy 196.85 125.73) (xy 167.64 125.73))
     (stroke (width 0) (type default))
@@
     (stroke (width 0) (type default))
   )
+  (wire (pts (xy 102.87 34.29) (xy 102.87 31.75))
+    (stroke (width 0) (type default))
+  )
+  (wire (pts (xy 92.71 31.75) (xy 90.17 31.75))
+    (stroke (width 0) (type default))
+  )
+  (wire (pts (xy 100.33 31.75) (xy 97.79 31.75))
+    (stroke (width 0) (type default))
+  )
+  (wire (pts (xy 95.25 34.29) (xy 95.25 31.75))
+    (stroke (width 0) (type default))
+  )
+  (wire (pts (xy 95.25 31.75) (xy 97.79 31.75))
+    (stroke (width 0) (type default))
+  )
+  (wire (pts (xy 54.61 72.39) (xy 72.39 72.39))
+    (stroke (width 0) (type default))
+  )
   (wire (pts (xy 196.85 80.01) (xy 176.53 80.01))
     (stroke (width 0) (type default))
@@
     (stroke (width 0) (type default))
   )
+  (wire (pts (xy 97.79 34.29) (xy 97.79 31.75))
+    (stroke (width 0) (type default))
+  )
   (wire (pts (xy 261.62 120.65) (xy 281.94 120.65))
     (stroke (width 0) (type default))
   )
+  (wire (pts (xy 92.71 34.29) (xy 92.71 31.75))
+    (stroke (width 0) (type default))
+  )
   (wire (pts (xy 59.69 41.91) (xy 72.39 41.91))
     (stroke (width 0) (type default))
   )
+  (wire (pts (xy 90.17 34.29) (xy 90.17 31.75))
+    (stroke (width 0) (type default))
+  )
   (wire (pts (xy 118.11 46.99) (xy 149.86 46.99))
     (stroke (width 0) (type default))
@@
     (effects (font (size 1.27 1.27)) (justify left bottom))
   )
+  (symbol (lib_id "power:+3.3V") (at 90.17 25.4 0) (unit 1)
+    (in_bom yes) (on_board yes) (dnp no) (fields_autoplaced)
+    (property "Reference" "#PWR024" (at 90.17 29.21 0)
+      (effects (font (size 1.27 1.27)) hide)
+    )
+    (property "Value" "+3.3V" (at 90.17 21.59 0)
+      (effects (font (size 1.27 1.27)))
+    )
+    (property "Footprint" "" (at 90.17 25.4 0)
+      (effects (font (size 1.27 1.27)) hide)
+    )
+    (property "Datasheet" "" (at 90.17 25.4 0)
+      (effects (font (size 1.27 1.27)) hide)
+    )
+    (pin "1")
+    (instances
+      (project "Flight Computer"
+        (path "/0c1188a1-706b-46cd-a73a-5b3f8187d77a"
+          (reference "#PWR024") (unit 1)
+        )
+      )
+    )
+  )
   (symbol (lib_id "MCU_ST_STM32L4:STM32L476VETx") (at 95.25 105.41 0) (unit 1)
