File: Flight Computer.kicad_sch (KiCad schematic)
At the start: 26 parts, among them Q1 MMBT2222A, U6 STM32L476VETx, Y1 16MHz

Commit message: 173 Errors. I'm going to take a break
Parts:
- added R32, R33: 2.7k, symbol Device:R
Connections:
- net +3.3V: now also R32.1, R33.1
- net I2C2 SCL: now also R26.2
- net I2C2 SDA: now also R27.2
- net I2C3 SCL: now also R32.2; no longer R26.2
- net I2C3 SDA: now also R33.2; no longer R27.2
- net Pyro Channel A: no longer U6.37 (PB2)
- net Pyro Channel A Trigger: now also U6.37 (PB2)
- net Pyro Channel B: no longer U6.40 (PE9)
- net Pyro Channel B Trigger: now also U6.40 (PE9)
- net Pyro Channel C: no longer U6.39 (PE8)
- net Pyro Channel C Trigger: now also U6.39 (PE8)
- net Pyro Channel D: no longer U6.38 (PE7)
- net Pyro Channel D Trigger: now also U6.38 (PE7)
- net Pyro Channel E: no longer U6.44 (PE13)
- net Pyro Channel E Trigger: now also U6.44 (PE13)
- net Pyro Channel F: no longer U6.43 (PE12)
- net Pyro Channel F Trigger: now also U6.43 (PE12)
Other:
- sheet Sensors ports: added Chip Select Flash Memory, Flash CLK, Flash SPI IO0, Flash SPI IO1, Flash SPI IO2, Flash SPI IO3, SCL1, SCL3, SD CLK, SD CMD, SD DAT0, SD DAT1, SD DAT2, SD DAT3, SDA1, SDA3; removed SCL, SDA
- note added: "Cload = 2 * (Cl + Cstray)"
- note added: "Pull-up resistors for I2C busses. Internal busses have 2.7k, external has 5.1k in case we need to interface with something with integrated pull-ups."
- moved on the sheet: D1, R26, R27, R28, R29, R3

Commit message: Fixed all correct errors
Parts:
- renumbered R1 to R34
Changed lines of the file:
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@@
   (junction (at 96.52 33.02) (diameter 0) (color 0 0 0 0)
+  )
+  (junction (at 111.76 27.94) (diameter 0) (color 0 0 0 0)
   )
   (no_connect (at 81.28 106.68))
@@
   (symbol (lib_id "Device:R") (at 64.77 48.26 90) (unit 1)
     (in_bom yes) (on_board yes) (dnp no) (fields_autoplaced)
-    (property "Reference" "R1" (at 64.77 43.18 90)
+    (property "Reference" "R34" (at 64.77 43.18 90)
       (effects (font (size 1.27 1.27)))
     )
@@
       (project "Flight Computer"
         (path "/0c1188a1-706b-46cd-a73a-5b3f8187d77a"
-          (reference "R1") (unit 1)
+          (reference "R34") (unit 1)
         )
       )
@@
         )
       )
+    )
+  )
+  (symbol (lib_id "power:PWR_FLAG") (at 111.76 27.94 0) (unit 1)
+    (in_bom yes) (on_board yes) (dnp no) (fields_autoplaced)
+    (property "Reference" "#FLG02" (at 111.76 26.035 0)
+      (effects (font (size 1.27 1.27)) hide)
+    )
+    (property "Value" "PWR_FLAG" (at 111.76 24.13 0)
+      (effects (font (size 1.27 1.27)))
+    )
+    (property "Footprint" "" (at 111.76 27.94 0)
+      (effects (font (size 1.27 1.27)) hide)
+    )
+    (property "Datasheet" "~" (at 111.76 27.94 0)
+      (effects (font (size 1.27 1.27)) hide)
+    )
+    (pin "1")
+    (instances
+      (project "Flight Computer"
+        (path "/0c1188a1-706b-46cd-a73a-5b3f8187d77a"
+          (reference "#FLG02") (unit 1)
+        )
+      )

Commit message: Chose footprints for most components
Parts:
- BZ1: footprint (none) -> Buzzer_Beeper:Buzzer_TDK_PS1240P02BT_D12.2mm_H6.5mm
- C10, C11, C12, C13, C14, C15, C26, C27: footprint (none) -> Capacitor_SMD:C_0402_1005Metric
- C16: footprint (none) -> Capacitor_SMD:C_0603_1608Metric
- C24, C25: footprint (none) -> Capacitor_SMD:C_0805_2012Metric
- D1: footprint (none) -> LED_SMD:LED_0805_2012Metric
- R2, R3, R30, R31: footprint (none) -> Resistor_SMD:R_0603_1608Metric
- R26, R27, R28, R29, R32, R33, R34: footprint (none) -> Resistor_SMD:R_0402_1005Metric
Connections:
- net SD Card Detect: now reaches U6.81 (PD0)
- no-connect marks 27 -> 26
Other:
- sheet Sensors ports: added SD Card Detect; removed none
Changed lines of the file:
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@@
   (no_connect (at 127 124.46))
   (no_connect (at 81.28 83.82))
-  (no_connect (at 81.28 111.76))
   (wire (pts (xy 52.07 68.58) (xy 81.28 68.58))
     (stroke (width 0) (type default))
@@
     (stroke (width 0) (type default))
   )
+  (wire (pts (xy 62.23 111.76) (xy 81.28 111.76))
+    (stroke (width 0) (type default))
+  )
   (wire (pts (xy 99.06 33.02) (xy 99.06 35.56))
     (stroke (width 0) (type default))
@@
   )
   (wire (pts (xy 76.2 27.94) (xy 86.36 27.94))
+    (stroke (width 0) (type default))
+  )
+  (wire (pts (xy 250.19 36.83) (xy 278.13 36.83))
     (stroke (width 0) (type default))
   )
@@
     (effects (font (size 1.27 1.27)) (justify left bottom))
   )
+  (label "SD Card Detect" (at 278.13 36.83 180) (fields_autoplaced)
+    (effects (font (size 1.27 1.27)) (justify right bottom))
+  )
   (label "SWDIO" (at 274.32 105.41 180) (fields_autoplaced)
     (effects (font (size 1.27 1.27)) (justify right bottom))
@@
     (effects (font (size 1.27 1.27)) (justify left bottom))
   )
-  (label "I2C3 SCL" (at 181.61 33.02 0) (fields_autoplaced)
+  (label "I2C3 SDA" (at 181.61 33.02 0) (fields_autoplaced)
     (effects (font (size 1.27 1.27)) (justify left bottom))
   )
@@
   )
   (label "I2C2 SCL" (at 189.23 106.68 0) (fields_autoplaced)
+    (effects (font (size 1.27 1.27)) (justify left bottom))
+  )
+  (label "SD Card Detect" (at 62.23 111.76 0) (fields_autoplaced)
     (effects (font (size 1.27 1.27)) (justify left bottom))
   )
@@
       (effects (font (size 1.27 1.27)) (justify left))
     )
-    (property "Footprint" "" (at 27.6352 35.56 0)
+    (property "Footprint" "Capacitor_SMD:C_0603_1608Metric" (at 27.6352 35.56 0)
       (effects (font (size 1.27 1.27)) hide)
     )
@@
       (effects (font (size 1.27 1.27)) (justify right))
     )
-    (property "Footprint" "" (at 69.85 156.21 0)
+    (property "Footprint" "LED_SMD:LED_0805_2012Metric" (at 69.85 156.21 0)
       (effects (font (size 1.27 1.27)) hide)
     )
@@
       (effects (font (size 1.27 1.27)) (justify left))
     )
-    (property "Footprint" "" (at 55.372 179.07 90)
+    (property "Footprint" "Resistor_SMD:R_0402_1005Metric" (at 55.372 179.07 90)
       (effects (font (size 1.27 1.27)) hide)
     )
@@
       (effects (font (size 1.27 1.27)))
     )
-    (property "Footprint" "" (at 64.77 50.038 90)
+    (property "Footprint" "Resistor_SMD:R_0402_1005Metric" (at 64.77 50.038 90)
       (effects (font (size 1.27 1.27)) hide)
     )
@@
       (effects (font (size 1.27 1.27)) (justify left))
     )
-    (property "Footprint" "" (at 36.5252 35.56 0)
+    (property "Footprint" "Capacitor_SMD:C_0402_1005Metric" (at 36.5252 35.56 0)
       (effects (font (size 1.27 1.27)) hide)
     )
@@
       (effects (font (size 1.27 1.27)) (justify left))
     )
-    (property "Footprint" "" (at 41.6052 87.63 0)
+    (property "Footprint" "Capacitor_SMD:C_0402_1005Metric" (at 41.6052 87.63 0)
       (effects (font (size 1.27 1.27)) hide)
     )
@@
       (effects (font (size 1.27 1.27)) (justify left))
     )
-    (property "Footprint" "" (at 151.13 177.8 0)
+    (property "Footprint" "Resistor_SMD:R_0603_1608Metric" (at 151.13 177.8 0)
       (effects (font (size 1.27 1.27)) hide)
     )
@@
       (effects (font (size 1.27 1.27)) (justify left))
     )
-    (property "Footprint" "" (at 56.8452 35.56 0)
+    (property "Footprint" "Capacitor_SMD:C_0402_1005Metric" (at 56.8452 35.56 0)
       (effects (font (size 1.27 1.27)) hide)
     )
@@
       (effects (font (size 1.27 1.27)) (justify left))
     )
-    (property "Footprint" "" (at 156.845 175.26 90)
+    (property "Footprint" "Buzzer_Beeper:Buzzer_TDK_PS1240P02BT_D12.2mm_H6.5mm" (at 156.845 175.26 90)
       (effects (font (size 1.27 1.27)) hide)
     )
@@
       (effects (font (size 1.27 1.27)) (justify left))
     )
-    (property "Footprint" "" (at 67.0052 35.56 0)
+    (property "Footprint" "Capacitor_SMD:C_0402_1005Metric" (at 67.0052 35.56 0)
       (effects (font (size 1.27 1.27)) hide)
     )
@@
       (effects (font (size 1.27 1.27)) (justify left))
     )
-    (property "Footprint" "" (at 87.3252 35.56 0)
+    (property "Footprint" "Capacitor_SMD:C_0402_1005Metric" (at 87.3252 35.56 0)
       (effects (font (size 1.27 1.27)) hide)
     )
@@
       (effects (font (size 1.27 1.27)) (justify left))
     )
-    (property "Footprint" "" (at 139.3952 35.56 0)
+    (property "Footprint" "Capacitor_SMD:C_0805_2012Metric" (at 139.3952 35.56 0)
       (effects (font (size 1.27 1.27)) hide)
     )
@@
       (effects (font (size 1.27 1.27)) (justify left))
     )
-    (property "Footprint" "" (at 130.5052 35.56 0)
+    (property "Footprint" "Capacitor_SMD:C_0805_2012Metric" (at 130.5052 35.56 0)
       (effects (font (size 1.27 1.27)) hide)
     )
@@
       (effects (font (size 1.27 1.27)) (justify left))
     )
-    (property "Footprint" "" (at 40.132 179.07 90)
+    (property "Footprint" "Resistor_SMD:R_0402_1005Metric" (at 40.132 179.07 90)
       (effects (font (size 1.27 1.27)) hide)
     )
@@
       (effects (font (size 1.27 1.27)) (justify left))
     )
-    (property "Footprint" "" (at 20.0152 87.63 0)
+    (property "Footprint" "Capacitor_SMD:C_0402_1005Metric" (at 20.0152 87.63 0)
       (effects (font (size 1.27 1.27)) hide)
     )
@@
       (effects (font (size 1.27 1.27)) (justify left))
     )
-    (property "Footprint" "" (at 17.272 179.07 90)
+    (property "Footprint" "Resistor_SMD:R_0402_1005Metric" (at 17.272 179.07 90)
       (effects (font (size 1.27 1.27)) hide)
     )
@@
       (effects (font (size 1.27 1.27)) (justify left))
     )
-    (property "Footprint" "" (at 46.6852 35.56 0)
+    (property "Footprint" "Capacitor_SMD:C_0402_1005Metric" (at 46.6852 35.56 0)
       (effects (font (size 1.27 1.27)) hide)
     )
@@
       (effects (font (size 1.27 1.27)) (justify left))
     )
-    (property "Footprint" "" (at 47.752 179.07 90)
+    (property "Footprint" "Resistor_SMD:R_0402_1005Metric" (at 47.752 179.07 90)
       (effects (font (size 1.27 1.27)) hide)
     )
@@
       (effects (font (size 1.27 1.27)))
     )
-    (property "Footprint" "" (at 140.97 188.468 90)
+    (property "Footprint" "Resistor_SMD:R_0603_1608Metric" (at 140.97 188.468 90)
       (effects (font (size 1.27 1.27)) hide)
     )
@@
       (effects (font (size 1.27 1.27)) (justify left))
     )
-    (property "Footprint" "" (at 24.892 179.07 90)
+    (property "Footprint" "Resistor_SMD:R_0402_1005Metric" (at 24.892 179.07 90)
       (effects (font (size 1.27 1.27)) hide)
     )
@@
       (effects (font (size 1.27 1.27)) (justify left))
     )
-    (property "Footprint" "" (at 38.862 68.58 90)
+    (property "Footprint" "Resistor_SMD:R_0603_1608Metric" (at 38.862 68.58 90)
       (effects (font (size 1.27 1.27)) hide)
     )
@@
       (effects (font (size 1.27 1.27)) (justify left))
     )
-    (property "Footprint" "" (at 77.1652 35.56 0)
+    (property "Footprint" "Capacitor_SMD:C_0402_1005Metric" (at 77.1652 35.56 0)
       (effects (font (size 1.27 1.27)) hide)
     )
@@
       (effects (font (size 1.27 1.27)) (justify left))
     )
-    (property "Footprint" "" (at 32.512 179.07 90)
+    (property "Footprint" "Resistor_SMD:R_0402_1005Metric" (at 32.512 179.07 90)
       (effects (font (size 1.27 1.27)) hide)
     )
@@
       (effects (font (size 1.27 1.27)) (justify left))
     )
-    (property "Footprint" "" (at 68.072 165.1 90)
+    (property "Footprint" "Resistor_SMD:R_0603_1608Metric" (at 68.072 165.1 90)
       (effects (font (size 1.27 1.27)) hide)
     )
@@
       (effects (font (size 1.27 1.27)) (justify left))
     )
-    (instances
+    (pin "SD Card Detect" input (at 250.19 36.83 0)
+      (effects (font (size 1.27 1.27)) (justify right))
+    )
+    (instances

Commit message: Added custom footprints and started layout
Parts:
- removed L1: 68n, symbol Device:L
- added FB2: GZ2012D601TF, Inductor_SMD:L_0805_2012Metric, symbol Device:FerriteBead
- C24: value 10u -> 100n
- C25: value 10u -> 1u
- R26, R27: value 5.1k -> 4.7k
- R28, R29, R32, R33: value 2.7k -> 4.7k
- Y1: footprint (none) -> Crystal:Crystal_SMD_3225-4Pin_3.2x2.5mm
Connections:
- net +3.3V: now also FB2.2
- net VDDA: now also FB2.1
Other:
- note added: "Pull-up resistors for I2C busses, 4.7k"
- note removed: "Pull-up resistors for I2C busses. Internal busses have 2.7k, external has 5.1k in case we need to interface with something with integrated pull-ups."
Changed lines of the file:
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@@
     (stroke (width 0) (type default))
   )
-  (text "Pull-up resistors for I2C busses. Internal\nbusses have 2.7k, external has 5.1k in case\nwe need to interface with something with\nintegrated pull-ups."
-    (at 15.24 163.83 0)
+  (text "Pull-up resistors for I2C busses, 4.7k" (at 15.24 163.83 0)
     (effects (font (size 1.27 1.27)) (justify left bottom))
   )
@@
   (label "Pyro Channel D" (at 182.88 88.9 0) (fields_autoplaced)
     (effects (font (size 1.27 1.27)) (justify left bottom))
-  )
-  (symbol (lib_id "Device:L") (at 148.59 27.94 90) (unit 1)
-    (in_bom yes) (on_board yes) (dnp no)
-    (property "Reference" "L1" (at 148.59 25.4 90)
-      (effects (font (size 1.27 1.27)))
-    )
-    (property "Value" "68n" (at 148.59 29.21 90)
-      (effects (font (size 1.27 1.27)))
-    )
-    (property "Footprint" "" (at 148.59 27.94 0)
-      (effects (font (size 1.27 1.27)) hide)
-    )
-    (property "Datasheet" "~" (at 148.59 27.94 0)
-      (effects (font (size 1.27 1.27)) hide)
-    )
-    (pin "1")
-    (pin "2")
-    (instances
-      (project "Flight Computer"
-        (path "/0c1188a1-706b-46cd-a73a-5b3f8187d77a"
-          (reference "L1") (unit 1)
-        )
-      )
-    )
   )
   (symbol (lib_id "power:GND") (at 153.67 194.31 0) (unit 1)
@@
       (effects (font (size 1.27 1.27)) (justify left))
     )
-    (property "Value" "2.7k" (at 58.42 180.34 0)
+    (property "Value" "4.7k" (at 58.42 180.34 0)
       (effects (font (size 1.27 1.27)) (justify left))
     )
@@
       (effects (font (size 1.27 1.27)))
     )
-    (property "Footprint" "" (at 30.48 74.93 0)
+    (property "Footprint" "Crystal:Crystal_SMD_3225-4Pin_3.2x2.5mm" (at 30.48 74.93 0)
       (effects (font (size 1.27 1.27)) hide)
     )
@@
       (effects (font (size 1.27 1.27)) (justify left))
     )
-    (property "Value" "10u" (at 140.97 33.02 0)
+    (property "Value" "1u" (at 140.97 33.02 0)
       (effects (font (size 1.27 1.27)) (justify left))
     )
@@
       (effects (font (size 1.27 1.27)) (justify left))
     )
-    (property "Value" "10u" (at 132.08 33.02 0)
+    (property "Value" "100n" (at 132.08 33.02 0)
       (effects (font (size 1.27 1.27)) (justify left))
     )
@@
       (effects (font (size 1.27 1.27)) (justify left))
     )
-    (property "Value" "5.1k" (at 43.18 180.34 0)
+    (property "Value" "4.7k" (at 43.18 180.34 0)
       (effects (font (size 1.27 1.27)) (justify left))
     )
@@
     )
   )
+  (symbol (lib_id "Device:FerriteBead") (at 148.59 27.94 90) (unit 1)
+    (in_bom yes) (on_board yes) (dnp no) (fields_autoplaced)
+    (property "Reference" "FB2" (at 148.5392 21.59 90)
+      (effects (font (size 1.27 1.27)))
+    )
+    (property "Value" "GZ2012D601TF" (at 148.5392 24.13 90)
+      (effects (font (size 1.27 1.27)))
+    )
+    (property "Footprint" "Inductor_SMD:L_0805_2012Metric" (at 148.59 29.718 90)
+      (effects (font (size 1.27 1.27)) hide)
+    )
+    (property "Datasheet" "~" (at 148.59 27.94 0)
+      (effects (font (size 1.27 1.27)) hide)
+    )
+    (pin "1")
+    (pin "2")
+    (instances
+      (project "Flight Computer"
+        (path "/0c1188a1-706b-46cd-a73a-5b3f8187d77a/afc466af-6d84-4e19-b5b5-aea43618ea20"
+          (reference "FB2") (unit 1)
+        )
+        (path "/0c1188a1-706b-46cd-a73a-5b3f8187d77a"
+          (reference "FB1") (unit 1)
+        )
+      )
+    )
+  )
   (symbol (lib_id "power:+3.3V") (at 34.29 171.45 0) (unit 1)
     (in_bom yes) (on_board yes) (dnp no) (fields_autoplaced)
@@
       (effects (font (size 1.27 1.27)) (justify left))
     )
-    (property "Value" "2.7k" (at 20.32 180.34 0)
+    (property "Value" "4.7k" (at 20.32 180.34 0)
       (effects (font (size 1.27 1.27)) (justify left))
     )
@@
       (effects (font (size 1.27 1.27)) (justify left))
     )
-    (property "Value" "2.7k" (at 50.8 180.34 0)
+    (property "Value" "4.7k" (at 50.8 180.34 0)
       (effects (font (size 1.27 1.27)) (justify left))
     )
@@
       (effects (font (size 1.27 1.27)) (justify left))
     )
-    (property "Value" "2.7k" (at 27.94 180.34 0)
+    (property "Value" "4.7k" (at 27.94 180.34 0)
       (effects (font (size 1.27 1.27)) (justify left))
     )
@@
       (effects (font (size 1.27 1.27)) (justify left))
     )
-    (property "Value" "5.1k" (at 35.56 180.34 0)
-      (effects (font (size 1.27 1.27)) (justify left))
-    )
+    (property "Value" "4.7k" (at 35.56 180.34 0)
+      (effects (font (size 1.27 1.27)) (justify left))
+    )

Commit message: Started footprint
Parts:
- C24: footprint Capacitor_SMD:C_0805_2012Metric -> Capacitor_SMD:C_0402_1005Metric
- C25: footprint Capacitor_SMD:C_0805_2012Metric -> Capacitor_SMD:C_0603_1608Metric
Changed lines of the file:
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@@
       (effects (font (size 1.27 1.27)) (justify left))
     )
-    (property "Footprint" "Capacitor_SMD:C_0805_2012Metric" (at 139.3952 35.56 0)
+    (property "Footprint" "Capacitor_SMD:C_0603_1608Metric" (at 139.3952 35.56 0)
       (effects (font (size 1.27 1.27)) hide)
     )
@@
       (effects (font (size 1.27 1.27)) (justify left))
     )
-    (property "Footprint" "Capacitor_SMD:C_0805_2012Metric" (at 130.5052 35.56 0)
+    (property "Footprint" "Capacitor_SMD:C_0402_1005Metric" (at 130.5052 35.56 0)
       (effects (font (size 1.27 1.27)) hide)
     )

Commit message: Made more progress on layout
Connections:
- net USB 5V in: now reaches U6.68 (PA9)
- no-connect marks 26 -> 25
Other:
- sheet Connectors and Power Supply ports: added USB 5V in; removed none
Changed lines of the file:
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@@
   (no_connect (at 127 162.56))
   (no_connect (at 81.28 81.28))
-  (no_connect (at 127 66.04))
   (no_connect (at 255.27 110.49))
   (no_connect (at 81.28 78.74))
@@
     (stroke (width 0) (type default))
   )
+  (wire (pts (xy 127 66.04) (xy 147.32 66.04))
+    (stroke (width 0) (type default))
+  )
   (wire (pts (xy 127 55.88) (xy 158.75 55.88))
     (stroke (width 0) (type default))
@@
     (stroke (width 0) (type default))
   )
+  (wire (pts (xy 255.27 86.36) (xy 269.24 86.36))
+    (stroke (width 0) (type default))
+  )
   (wire (pts (xy 170.18 151.13) (xy 196.85 151.13))
     (stroke (width 0) (type default))
@@
     (effects (font (size 1.27 1.27)) (justify left bottom))
   )
+  (label "USB 5V in" (at 147.32 66.04 180) (fields_autoplaced)
+    (effects (font (size 1.27 1.27)) (justify right bottom))
+  )
   (label "Chip Select Low G Accel" (at 276.86 19.05 180) (fields_autoplaced)
     (effects (font (size 1.27 1.27)) (justify right bottom))
@@
   (label "Pyro Channel D" (at 182.88 88.9 0) (fields_autoplaced)
     (effects (font (size 1.27 1.27)) (justify left bottom))
+  )
+  (label "USB 5V in" (at 269.24 86.36 180) (fields_autoplaced)
+    (effects (font (size 1.27 1.27)) (justify right bottom))
   )
   (symbol (lib_id "power:GND") (at 153.67 194.31 0) (unit 1)
@@
       (effects (font (size 1.27 1.27)) (justify right))
     )
+    (pin "USB 5V in" input (at 255.27 86.36 0)
+      (effects (font (size 1.27 1.27)) (justify right))
+    )

Commit message: I sure hope I come up with a better layout than this for the pyro channels
Connections:
- net Pyro Channel B Trigger: now also U6.38 (PE7); no longer U6.40 (PE9)
- net Pyro Channel D Trigger: now also U6.40 (PE9); no longer U6.38 (PE7)
- no-connect marks 25 -> 24
Other:
- sheet Connectors and Power Supply ports: added none; removed Backup Battery, SWO
- sheet Sensors ports: added none; removed Backup Battery
Changed lines of the file:
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@@
   (no_connect (at 127 162.56))
   (no_connect (at 81.28 81.28))
-  (no_connect (at 255.27 110.49))
   (no_connect (at 81.28 78.74))
   (no_connect (at 127 144.78))
@@
     (stroke (width 0) (type default))
   )
-  (wire (pts (xy 171.45 54.61) (xy 194.31 54.61))
-    (stroke (width 0) (type default))
-  )
   (wire (pts (xy 127 91.44) (xy 153.67 91.44))
     (stroke (width 0) (type default))
@@
     (stroke (width 0) (type default))
   )
-  (wire (pts (xy 255.27 115.57) (xy 276.86 115.57))
-    (stroke (width 0) (type default))
-  )
   (wire (pts (xy 250.19 64.77) (xy 270.51 64.77))
     (stroke (width 0) (type default))
@@
     (effects (font (size 1.27 1.27)) (justify left bottom))
   )
-  (label "Pyro Channel D Trigger" (at 55.88 86.36 0) (fields_autoplaced)
+  (label "Pyro Channel B Trigger" (at 55.88 86.36 0) (fields_autoplaced)
     (effects (font (size 1.27 1.27)) (justify left bottom))
   )
@@
     (effects (font (size 1.27 1.27)) (justify left bottom))
   )
-  (label "Backup Battery" (at 171.45 54.61 0) (fields_autoplaced)
-    (effects (font (size 1.27 1.27)) (justify left bottom))
-  )
   (label "QSPI Chip Select" (at 270.51 67.31 180) (fields_autoplaced)
     (effects (font (size 1.27 1.27)) (justify right bottom))
@@
     (effects (font (size 1.27 1.27)) (justify right bottom))
   )
-  (label "Backup Battery" (at 276.86 115.57 180) (fields_autoplaced)
-    (effects (font (size 1.27 1.27)) (justify right bottom))
-  )
   (label "SDMMC Data 3" (at 278.13 46.99 180) (fields_autoplaced)
     (effects (font (size 1.27 1.27)) (justify right bottom))
@@
     (effects (font (size 1.27 1.27)) (justify left bottom))
   )
-  (label "Pyro Channel B Trigger" (at 55.88 91.44 0) (fields_autoplaced)
+  (label "Pyro Channel D Trigger" (at 55.88 91.44 0) (fields_autoplaced)
     (effects (font (size 1.27 1.27)) (justify left bottom))
   )
@@
       (effects (font (size 1.27 1.27)) (justify left))
     )
-    (pin "Backup Battery" input (at 194.31 54.61 180)
-      (effects (font (size 1.27 1.27)) (justify left))
-    )
     (pin "UART RX" input (at 194.31 52.07 180)
       (effects (font (size 1.27 1.27)) (justify left))
@@
       (effects (font (size 1.27 1.27)) (justify right))
     )
-    (pin "SWO" input (at 255.27 110.49 0)
-      (effects (font (size 1.27 1.27)) (justify right))
-    )
-    (pin "Backup Battery" input (at 255.27 115.57 0)
-      (effects (font (size 1.27 1.27)) (justify right))
-    )
