File: Flight Computer.kicad_sch (KiCad schematic)
At the start: 28 parts, among them Q1 MMBT2222A, U6 STM32L476VETx, Y1 16MHz

Commit message: How many sheets do you want? Yes
Parts:
- removed BZ1: Buzzer, Buzzer_Beeper:Buzzer_TDK_PS1240P02BT_D12.2mm_H6.5mm, symbol Device:Buzzer
- removed C10, C11, C12, C13, C14, C15, C24: 100n, Capacitor_SMD:C_0402_1005Metric, symbol Device:C
- removed C16: 4u7, Capacitor_SMD:C_0603_1608Metric, symbol Device:C
- removed C25: 1u, Capacitor_SMD:C_0603_1608Metric, symbol Device:C
- removed C26, C27: 12p, Capacitor_SMD:C_0402_1005Metric, symbol Device:C
- removed D1: Blue, LED_SMD:LED_0805_2012Metric, symbol Device:LED
- removed FB2: GZ2012D601TF, Inductor_SMD:L_0805_2012Metric, symbol Device:FerriteBead
- removed Q1: MMBT2222A, Package_TO_SOT_SMD:SOT-23, symbol Transistor_BJT:MMBT3904
- removed R2: 47, Resistor_SMD:R_0603_1608Metric, symbol Device:R
- removed R28, R29, R32, R33: 4.7k, Resistor_SMD:R_0402_1005Metric, symbol Device:R
- removed R3: 1.5k, Resistor_SMD:R_0603_1608Metric, symbol Device:R
- removed R30: 1k, Resistor_SMD:R_0603_1608Metric, symbol Device:R
- removed R31: 1k, Resistor_SMD:R_0603_1608Metric, symbol Device:R_Small
- removed R34: 10k, Resistor_SMD:R_0402_1005Metric, symbol Device:R
- removed U6: STM32L476VETx, Package_QFP:LQFP-100_14x14mm_P0.5mm, symbol MCU_ST_STM32L4:STM32L476VETx
- removed Y1: 16MHz, Crystal:Crystal_SMD_3225-4Pin_3.2x2.5mm, symbol Device:Crystal_GND24
Connections:
- no-connect marks 24 -> 0
Other:
- added sheet Microcontroller (microcontroller.kicad_sch)
- sheet Connectors and Power Supply ports: added Main battery connector, Main battery in; removed Ignition Battery Voltage, Pyro Channel A, Pyro Channel B, Pyro Channel C, Pyro Channel D, Pyro Channel E, Pyro Channel F
- sheet Pyrotechnic Channels ports: added Ignition Battery Voltage, Main battery connector, Main battery in; removed Pyro Channel A, Pyro Channel B, Pyro Channel C, Pyro Channel D, Pyro Channel E, Pyro Channel F
- sheet Sensors ports: added Chip Select Altimeter, Chip Select High G Accel, High G Interrupt, Low G Accel Interrupt, Low G Gyro Interrupt; removed High G Interrupt 1, Low G Accel Interrupt 1, Low G Gyro Interrupt 3, Magnetometer Data Ready, Magnetometer Interrupt, SCL1, SCL3, SDA1, SDA3
- note added: "Pull-up resistors for external I2C buss, 4.7k"
- note removed: "Cload = 2 * (Cl + Cstray)"
- note removed: "Pull-up resistors for I2C busses, 4.7k"
- moved on the sheet: R26, R27

Commit message: Finished updating the schematics
Parts:
- removed R26, R27: 4.7k, Resistor_SMD:R_0402_1005Metric, symbol Device:R
Other:
- sheet Microcontroller ports: added Altimeter Interrupt, Chip Select Altimeter, Chip Select High G Accel, Chip Select Low G Accel, Chip Select Low G Gyro, GPS External Interrupt, GPS Reset, High G Interrupt, I2C2 SCL, I2C2 SDA, Ignition Battery Voltage, Low G Accel Interrupt, Low G Gyro Interrupt, NRST, Pyro A Continuity Voltage, Pyro B Continuity Voltage, Pyro C Continuity Voltage, Pyro Channel A Trigger, Pyro Channel B Trigger, Pyro Channel C Trigger, Pyro Channel D Trigger, Pyro Channel E Trigger, Pyro Channel F Trigger, Pyro D Continuity Voltage, Pyro E Continuity Voltage, Pyro F Continuity Voltage, QSPI Chip Select, QSPI Clock, QSPI IO0, QSPI IO1, QSPI IO2, QSPI IO3, SD Card Detect, SDMMC Command, SDMMC Data 0, SDMMC Data 1, SDMMC Data 2, SDMMC Data 3, SDMMC Data Clock, SPI1 MISO, SPI1 MOSI, SPI1 SCK, SWCLK, SWDIO, UART2 RX, UART2 TX, UART3 RX, UART3 TX, USB 5V in, USB D+, USB D-; removed none
- note removed: "Pull-up resistors for external I2C buss, 4.7k"

Commit message: Started doing layout for v1.1
Changed lines of the file:
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@@
       (effects (font (size 1.27 1.27)) (justify left top))
     )
-    (pin "Pyro Channel A Continuity Voltage" input (at 198.12 123.19 180)
-      (effects (font (size 1.27 1.27)) (justify left))
-    )
     (pin "Pyro Channel A Trigger" input (at 198.12 143.51 180)
-      (effects (font (size 1.27 1.27)) (justify left))
-    )
-    (pin "Pyro Channel E Continuity Voltage" input (at 198.12 133.35 180)
       (effects (font (size 1.27 1.27)) (justify left))
     )
@@
       (effects (font (size 1.27 1.27)) (justify left))
     )
-    (pin "Pyro Channel B Continuity Voltage" input (at 198.12 125.73 180)
-      (effects (font (size 1.27 1.27)) (justify left))
-    )
-    (pin "Pyro Channel C Continuity Voltage" input (at 198.12 128.27 180)
-      (effects (font (size 1.27 1.27)) (justify left))
-    )
-    (pin "Pyro Channel D Continuity Voltage" input (at 198.12 130.81 180)
-      (effects (font (size 1.27 1.27)) (justify left))
-    )
-    (pin "Pyro Channel F Continuity Voltage" input (at 198.12 135.89 180)
-      (effects (font (size 1.27 1.27)) (justify left))
-    )
     (pin "Pyro Channel F Trigger" input (at 198.12 156.21 180)
       (effects (font (size 1.27 1.27)) (justify left))
@@
       (effects (font (size 1.27 1.27)) (justify right))
     )
+    (pin "Pyro Channel D Continuity Voltage" output (at 198.12 130.81 180)
+      (effects (font (size 1.27 1.27)) (justify left))
+    )
+    (pin "Pyro Channel F Continuity Voltage" output (at 198.12 135.89 180)
+      (effects (font (size 1.27 1.27)) (justify left))
+    )
+    (pin "Pyro Channel C Continuity Voltage" output (at 198.12 128.27 180)
+      (effects (font (size 1.27 1.27)) (justify left))
+    )
+    (pin "Pyro Channel B Continuity Voltage" output (at 198.12 125.73 180)
+      (effects (font (size 1.27 1.27)) (justify left))
+    )
+    (pin "Pyro Channel E Continuity Voltage" output (at 198.12 133.35 180)
+      (effects (font (size 1.27 1.27)) (justify left))
+    )
+    (pin "Pyro Channel A Continuity Voltage" output (at 198.12 123.19 180)
+      (effects (font (size 1.27 1.27)) (justify left))
+    )
     (instances

Commit message: How many test points do you want? Yes.
Parts:
- added TP1: 5V, TestPoint:TestPoint_Pad_D1.5mm, symbol Connector:TestPoint
- added TP1: QSPI Clock, TestPoint:TestPoint_Pad_D1.5mm, symbol Connector:TestPoint
- added TP1: SDMMC Clock, TestPoint:TestPoint_Pad_D1.5mm, symbol Connector:TestPoint
- added TP1: Gnd, TestPoint:TestPoint_Pad_D1.5mm, symbol Connector:TestPoint
- added TP1: SDMMC Command, TestPoint:TestPoint_Pad_D1.5mm, symbol Connector:TestPoint
- added TP10: UART2 TX, TestPoint:TestPoint_Pad_D1.5mm, symbol Connector:TestPoint
- added TP11: UART2 RX, TestPoint:TestPoint_Pad_D1.5mm, symbol Connector:TestPoint
- added TP2: 3.3V, TestPoint:TestPoint_Pad_D1.5mm, symbol Connector:TestPoint
- added TP3: SPI1 MISO, TestPoint:TestPoint_Pad_D1.5mm, symbol Connector:TestPoint
- added TP4: SPI1 MOSI, TestPoint:TestPoint_Pad_D1.5mm, symbol Connector:TestPoint
- added TP5: SPI1 SCK, TestPoint:TestPoint_Pad_D1.5mm, symbol Connector:TestPoint
- added TP6: CS Altimeter, TestPoint:TestPoint_Pad_D1.5mm, symbol Connector:TestPoint
- added TP7: CS High G, TestPoint:TestPoint_Pad_D1.5mm, symbol Connector:TestPoint
- added TP8: CS Low G Gyro, TestPoint:TestPoint_Pad_D1.5mm, symbol Connector:TestPoint
- added TP9: CS Low G Accel, TestPoint:TestPoint_Pad_D1.5mm, symbol Connector:TestPoint
Connections:
- net Chip Select Altimeter: now also TP6.1
- net Chip Select High G Accel: now also TP7.1
- net Chip Select Low G Accel: now also TP8.1
- net Chip Select Low G Gyro: now also TP9.1
- net QSPI Clock: now also TP1.1
- net SDMMC Clock: now also TP1.1
- net SDMMC Command: now also TP1.1
- net SPI1 MISO: now also TP3.1
- net SPI1 MOSI: now also TP4.1
- net SPI1 SCK: now also TP5.1
- net UART2 RX: now also TP11.1
- net UART2 TX: now also TP10.1
- new net +3.3V: TP2.1
- new net +5V: TP1.1
- new net GND: TP1.1

Commit message: Updating with notes from Adam
Other:
- sheet Connectors and Power Supply ports: added External SPI MISO, External SPI MOSI, External SPI SCK; removed none
- sheet Microcontroller ports: added SPI2 MISO, SPI2 MOSI, SPI2 SCK; removed none
Changed lines of the file:
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@@
+    (stroke (width 0) (type default))
+  )
+  (wire (pts (xy 233.68 115.57) (xy 254 115.57))
     (stroke (width 0) (type default))
   )
@@
     (stroke (width 0) (type default))
   )
+  (wire (pts (xy 45.72 148.59) (xy 29.21 148.59))
+    (stroke (width 0) (type default))
+  )
   (wire (pts (xy 35.56 92.71) (xy 45.72 92.71))
     (stroke (width 0) (type default))
@@
     (stroke (width 0) (type default))
   )
+  (wire (pts (xy 233.68 110.49) (xy 254 110.49))
+    (stroke (width 0) (type default))
+  )
   (wire (pts (xy 21.59 129.54) (xy 45.72 129.54))
     (stroke (width 0) (type default))
@@
     (stroke (width 0) (type default))
   )
+  (wire (pts (xy 233.68 113.03) (xy 254 113.03))
+    (stroke (width 0) (type default))
+  )
   (wire (pts (xy 233.68 58.42) (xy 255.27 58.42))
     (stroke (width 0) (type default))
@@
     (stroke (width 0) (type default))
   )
+  (wire (pts (xy 29.21 146.05) (xy 45.72 146.05))
+    (stroke (width 0) (type default))
+  )
   (wire (pts (xy 97.79 160.02) (xy 139.7 160.02))
     (stroke (width 0) (type default))
@@
     (stroke (width 0) (type default))
   )
+  (wire (pts (xy 29.21 151.13) (xy 45.72 151.13))
+    (stroke (width 0) (type default))
+  )
   (wire (pts (xy 45.72 179.07) (xy 29.21 179.07))
     (stroke (width 0) (type default))
@@
     (effects (font (size 1.27 1.27)) (justify right bottom))
   )
+  (label "SPI2 SCK" (at 29.21 151.13 0) (fields_autoplaced)
+    (effects (font (size 1.27 1.27)) (justify left bottom))
+  )
   (label "SDMMC Command" (at 127 173.99 180) (fields_autoplaced)
     (effects (font (size 1.27 1.27)) (justify right bottom))
@@
     (effects (font (size 1.27 1.27)) (justify left bottom))
   )
+  (label "SPI2 MOSI" (at 254 110.49 180) (fields_autoplaced)
+    (effects (font (size 1.27 1.27)) (justify right bottom))
+  )
   (label "Chip Select Altimeter" (at 139.7 148.59 180) (fields_autoplaced)
     (effects (font (size 1.27 1.27)) (justify right bottom))
@@
     (effects (font (size 1.27 1.27)) (justify right bottom))
   )
+  (label "SPI2 SCK" (at 254 115.57 180) (fields_autoplaced)
+    (effects (font (size 1.27 1.27)) (justify right bottom))
+  )
   (label "GPS Reset" (at 157.48 59.69 0) (fields_autoplaced)
     (effects (font (size 1.27 1.27)) (justify left bottom))
@@
     (effects (font (size 1.27 1.27)) (justify right bottom))
   )
+  (label "SPI2 MISO" (at 254 113.03 180) (fields_autoplaced)
+    (effects (font (size 1.27 1.27)) (justify right bottom))
+  )
   (label "QSPI IO0" (at 254 45.72 180) (fields_autoplaced)
     (effects (font (size 1.27 1.27)) (justify right bottom))
@@
     (effects (font (size 1.27 1.27)) (justify left bottom))
   )
+  (label "SPI2 MOSI" (at 29.21 146.05 0) (fields_autoplaced)
+    (effects (font (size 1.27 1.27)) (justify left bottom))
+  )
   (label "Pyro Channel A Trigger" (at 21.59 124.46 0) (fields_autoplaced)
     (effects (font (size 1.27 1.27)) (justify left bottom))
@@
   )
   (label "I2C2 SCL" (at 165.1 88.9 0) (fields_autoplaced)
+    (effects (font (size 1.27 1.27)) (justify left bottom))
+  )
+  (label "SPI2 MISO" (at 29.21 148.59 0) (fields_autoplaced)
     (effects (font (size 1.27 1.27)) (justify left bottom))
   )
@@
       (effects (font (size 1.27 1.27)) (justify right))
     )
+    (pin "SPI2 SCK" output (at 45.72 151.13 180)
+      (effects (font (size 1.27 1.27)) (justify left))
+    )
+    (pin "SPI2 MISO" input (at 45.72 148.59 180)
+      (effects (font (size 1.27 1.27)) (justify left))
+    )
+    (pin "SPI2 MOSI" output (at 45.72 146.05 180)
+      (effects (font (size 1.27 1.27)) (justify left))
+    )
     (instances
       (project "Flight Computer"
@@
     )
   )
-  (sheet (at 181.61 80.01) (size 52.07 30.48)
+  (sheet (at 181.61 80.01) (size 52.07 36.83)
     (stroke (width 0.1524) (type solid))
     (fill (color 0 0 0 0.0000))
@@
       (effects (font (size 1.27 1.27)) (justify left bottom))
     )
-    (property "Sheetfile" "connectors.kicad_sch" (at 181.61 111.76 0)
+    (property "Sheetfile" "connectors.kicad_sch" (at 181.61 114.3 0)
       (effects (font (size 1.27 1.27)) (justify left top))
     )
@@
       (effects (font (size 1.27 1.27)) (justify right))
     )
+    (pin "External SPI MOSI" input (at 233.68 110.49 0)
+      (effects (font (size 1.27 1.27)) (justify right))
+    )
+    (pin "External SPI MISO" input (at 233.68 113.03 0)
+      (effects (font (size 1.27 1.27)) (justify right))
+    )
+    (pin "External SPI SCK" input (at 233.68 115.57 0)
+      (effects (font (size 1.27 1.27)) (justify right))
+    )

Commit message: Finished final(tm) updates for v1.1
Other:
- sheet Microcontroller ports: added Channel A Continuity LED, Channel B Continuity LED, Channel C Continuity LED, Channel D Continuity LED, Channel E Continuity LED, Channel F Continuity LED; removed none
- sheet Pyrotechnic Channels ports: added Channel A Continuity LED, Channel B Continuity LED, Channel C Continuity LED, Channel D Continuity LED, Channel E Continuity LED, Channel F Continuity LED; removed none
- moved on the sheet: TP1

Commit message: Added new buck converter
Parts:
- removed TP1: 5V, TestPoint:TestPoint_Pad_D1.5mm, symbol Connector:TestPoint
Changed lines of the file:
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@@
-    (stroke (width 0) (type default))
-  )
-  (wire (pts (xy 78.74 29.21) (xy 78.74 30.48))
     (stroke (width 0) (type default))
   )
@@
         (path "/0c1188a1-706b-46cd-a73a-5b3f8187d77a"
           (reference "TP8") (unit 1)
-        )
-      )
-    )
-  )
-  (symbol (lib_id "Connector:TestPoint") (at 78.74 30.48 180) (unit 1)
-    (in_bom yes) (on_board yes) (dnp no)
-    (property "Reference" "TP1" (at 77.47 39.37 0)
-      (effects (font (size 1.27 1.27)) (justify right))
-    )
-    (property "Value" "5V" (at 77.47 36.83 0)
-      (effects (font (size 1.27 1.27)) (justify right))
-    )
-    (property "Footprint" "TestPoint:TestPoint_Pad_D1.5mm" (at 73.66 30.48 0)
-      (effects (font (size 1.27 1.27)) hide)
-    )
-    (property "Datasheet" "~" (at 73.66 30.48 0)
-      (effects (font (size 1.27 1.27)) hide)
-    )
-    (pin "1")
-    (instances
-      (project "Flight Computer"
-        (path "/0c1188a1-706b-46cd-a73a-5b3f8187d77a/afc466af-6d84-4e19-b5b5-aea43618ea20/d3a2bed6-f277-4c18-9b19-db934fe0c906"
-          (reference "TP1") (unit 1)
-        )
-        (path "/0c1188a1-706b-46cd-a73a-5b3f8187d77a"
-          (reference "TP1") (unit 1)
         )
       )
@@
         )
       )
-    )
-  )
-  (symbol (lib_id "power:+5V") (at 78.74 29.21 0) (unit 1)
-    (in_bom yes) (on_board yes) (dnp no) (fields_autoplaced)
-    (property "Reference" "#PWR0109" (at 78.74 33.02 0)
-      (effects (font (size 1.27 1.27)) hide)
-    )
-    (property "Value" "+5V" (at 78.74 25.4 0)
-      (effects (font (size 1.27 1.27)))
-    )
-    (property "Footprint" "" (at 78.74 29.21 0)
-      (effects (font (size 1.27 1.27)) hide)
-    )
-    (property "Datasheet" "" (at 78.74 29.21 0)
-      (effects (font (size 1.27 1.27)) hide)
-    )
-    (pin "1")
-    (instances
-      (project "Flight Computer"
-        (path "/0c1188a1-706b-46cd-a73a-5b3f8187d77a"
-          (reference "#PWR0109") (unit 1)
-        )
-      )

Commit message: Swapped out sensors in schematic for v3
Parts:
- removed TP1: SDMMC Clock, TestPoint:TestPoint_Pad_D1.5mm, symbol Connector:TestPoint
- removed TP1: SDMMC Command, TestPoint:TestPoint_Pad_D1.5mm, symbol Connector:TestPoint
- added TP13: SPI2 MOSI, TestPoint:TestPoint_Pad_D1.5mm, symbol Connector:TestPoint
- added TP14: SPI2 SCK, TestPoint:TestPoint_Pad_D1.5mm, symbol Connector:TestPoint
- added TP16: CS High G Accel, TestPoint:TestPoint_Pad_D1.5mm, symbol Connector:TestPoint
- added TP17: CS Magnetometer, TestPoint:TestPoint_Pad_D1.5mm, symbol Connector:TestPoint
- TP7: value CS High G -> SPI2 MISO
Connections:
- net Chip Select High G Accel is gone; now on net SPI2 SCK: TP7.1
- net SPI2 MISO: now also TP14.1
- net SPI2 MOSI: now also TP13.1
- new net High G Accel Chip Select: TP16.1
- new net Magnetometer Chip Select: TP17.1
Other:
- sheet Microcontroller ports: added High G Accel Chip Select, High G Accel Interrupt, Magnetometer Chip Select, Magnetometer Interrupt; removed Chip Select High G Accel, High G Interrupt, SD Card Detect, SDMMC Command, SDMMC Data 0, SDMMC Data 1, SDMMC Data 2, SDMMC Data 3, SDMMC Data Clock
- sheet Sensors ports: added High G Accelerometer Chip Select, High G Accelerometer Interrupt, Magnetometer Chip Select, Magnetometer Interrupt, SPI1 MISO, SPI1 MOSI, SPI1 SCK, SPI2 MISO, SPI2 MOSI, SPI2 SCK; removed Chip Select High G Accel, High G Interrupt, SD CLK, SD CMD, SD Card Detect, SD DAT0, SD DAT1, SD DAT2, SD DAT3, SPI MISO, SPI MOSI, SPI SCK
- moved on the sheet: TP1, TP10, TP11, TP2, TP3, TP4, TP5, TP6, TP8, TP9
