File: sensors.kicad_sch (KiCad schematic)
At the start: 5 parts, among them U1 LIS3MDL, U2 MAX-M10S

Commit message: Finished Updating Sensor Schematics
Parts:
- added C1, C7: 1u, symbol Device:C
- added C2, C3, C4, C5, C6, C8, C9: 100n, symbol Device:C
- added J1: GPS antenna, symbol Connector:Conn_Coaxial
Connections:
- net +3.3V: now reaches U3.1 (Vdd)
- net +3.3V: now also U1.10 (~{CS}), U1.5 (Vdd), U1.6 (Vdd_IO), U1.9 (SDO/SA1), U2.7 (VCC_IO), U2.8 (VCC), U3.12 (SDO/Addr_sel), U3.6 (Vs), U3.7 (Chip_Select), U4.11 (Vddio), U4.3 (Vdd), U5.1 (Vddio), U5.10 (Vdd), U5.6 (Chip_Select), C1.1, C2.1, C3.1, C4.1, C6.1, C7.1, C8.1, C9.1
- net SDA: now reaches U3.13 (SDA)
- net SDA: now also U1.11 (SDA/SDI/SDO), U5.4 (SDI)
- net SCL: now reaches U3.14 (SCL)
- net SCL: now also U1.1 (SCL/SPC), U5.2 (SCK)
- net GND: now reaches U3.2 (GND)
- net GND: now also U1.12 (GND), U1.2 (GND), U1.3 (GND), U2.1 (GND), U2.10 (GND), U2.12 (GND), U2.13 (LNA_EN), U3.4 (GND), U3.5 (GND), U4.2 (NC), U4.4 (GNDA), U4.6 (GNDIO), U4.7 (Protocol_Select), U5.3 (GND), U5.5 (SDO), U5.8 (GND), U5.9 (GND), C1.2, C2.2, C3.2, C4.2, C5.2, C6.2, C7.2, C8.2, C9.2, J1.2 (Ext)
- net High G Interrupt 1: now reaches U3.8 (Interrupt_1)
- net High G Interrupt 2: now reaches U3.9 (Interrupt_2)
- net at U1.4 (C1): now also C5.1
- net Magnetometer Interrupt: now reaches U1.7 (INT)
- net Magnetometer Data Ready: now reaches U1.8 (DRDY)
- net at U2.11 (RF_IN): now also J1.1 (In)
- net UART TX: now reaches U2.2 (TXD)
- net UART RX: now reaches U2.3 (RXD)
- net GPS External Interrupt: now reaches U2.5 (EXTINT)
- net Backup Battery: now reaches U2.6 (V_BCKP)
- net GPS Reset: now reaches U2.9 (~{RESET})
- net Low G Accel Interrupt 2: now reaches U4.1 (Interrupt_2)
- net SPI MISO: now reaches U4.10 (SDO2)
- net SPI MISO: now also U4.15 (SDO1)
- net Low G Gyro Interrupt 3: now reaches U4.12 (Interrupt_3)
- net Low G Gyro Interrupt 4: now reaches U4.13 (Interrupt_4)
- net Chip Select Low G Accel: now reaches U4.14 (Chip_Select_Accel)
- net Low G Accel Interrupt 1: now reaches U4.16 (Interrupt_1)
- net Chip Select Low G Gyro: now reaches U4.5 (Chip_Select_Gyro)
- net SPI SCK: now reaches U4.8 (SCL/SCK)
- net SPI MOSI: now reaches U4.9 (SDA/SDI)
- net Altimeter Interrupt: now reaches U5.7 (Interrupt)
- no-connect marks 0 -> 8
Other:
- moved on the sheet: U1, U2, U3, U4

Commit message: Schematics are love. Also I have no idea what I was doing last night so the power supply might be terrible, but I know I thought it was brilliant at the time
Connections:
- net High G Interrupt 2: no longer names the net of U3.9 (Interrupt_2)
- net Low G Accel Interrupt 2: no longer names the net of U4.1 (Interrupt_2)
- net Low G Gyro Interrupt 4: no longer names the net of U4.13 (Interrupt_4)
- no-connect marks 8 -> 11
Changed lines of the file:
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@@
   (junction (at 64.77 93.98) (diameter 0) (color 0 0 0 0)
   )
+  (no_connect (at 251.46 127))
   (no_connect (at 215.9 63.5))
   (no_connect (at 246.38 63.5))
   (no_connect (at 215.9 53.34))
+  (no_connect (at 72.39 57.15))
   (no_connect (at 72.39 45.72))
   (no_connect (at 215.9 68.58))
@@
   (no_connect (at 215.9 55.88))
   (no_connect (at 72.39 43.18))
+  (no_connect (at 251.46 132.08))
   (wire (pts (xy 247.65 129.54) (xy 251.46 129.54))
     (stroke (width 0) (type default))
@@
     (effects (font (size 1.27 1.27)) (justify right))
   )
-  (hierarchical_label "Low G Accel Interrupt 2" (shape bidirectional) (at 251.46 127 0) (fields_autoplaced)
-    (effects (font (size 1.27 1.27)) (justify left))
-  )
   (hierarchical_label "SPI MOSI" (shape input) (at 208.28 132.08 180) (fields_autoplaced)
     (effects (font (size 1.27 1.27)) (justify right))
   )
-  (hierarchical_label "Low G Gyro Interrupt 4" (shape output) (at 251.46 132.08 0) (fields_autoplaced)
-    (effects (font (size 1.27 1.27)) (justify left))
-  )
   (hierarchical_label "GPS Reset" (shape input) (at 209.55 66.04 180) (fields_autoplaced)
     (effects (font (size 1.27 1.27)) (justify right))
@@
     (effects (font (size 1.27 1.27)) (justify right))
   )
-  (hierarchical_label "High G Interrupt 2" (shape output) (at 72.39 57.15 180) (fields_autoplaced)
-    (effects (font (size 1.27 1.27)) (justify right))
-  )

Commit message: --
Other:
- note added: "There are two different acceleromters, this one is lower G, which is more accurate for most scenarios"
Changed lines of the file:
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@@
     (fill (type none))
+  )
+  (text "There are two different acceleromters, this one is\nlower G, which is more accurate for most scenarios"
+    (at 182.88 110.49 0)
+    (effects (font (size 1.27 1.27)) (justify left bottom))
   )
   (text "SPI\n" (at 185.42 96.52 0)
