File: sensors.kicad_sch (KiCad schematic)
At the start: 20 parts, among them J1 GPS antenna, J10 Micro_SD_Card, U1 LIS3MDL, U2 MAX-M10S, U7 W25Q128JVS

Commit message: 173 Errors. I'm going to take a break
Connections:
- net SCL renamed SCL1
- net SCL1: no longer U5.2 (SCK)
- net SDA renamed SDA1
- net SDA1: no longer U5.4 (SDI)
- new net SCL3: U5.2 (SCK)
- new net SDA3: U5.4 (SDI)
Other:
- note added: "Data Storage"
- note added: "Honestly don't know why I bother with a magnetometer, it's not like heading is relevant beyond what GPS coordinates give us"
- note added: "This is worse than the MS5611 we were planning on using, but it is easier to find at JLC"
- note added: "Thisis the high G accelerometer, (±64 Gs), for events like chute deployment"
- moved on the sheet: C10, C11, J10, R1, U7

Commit message: Fixed all correct errors
Parts:
- C28: renamed from C11; value C -> 4u7
- renumbered C10 to C29
Changed lines of the file:
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@@
+    (stroke (width 0) (type default))
+  )
+  (wire (pts (xy 246.38 50.8) (xy 273.05 50.8))
     (stroke (width 0) (type default))
   )
@@
     (stroke (width 0) (type default))
   )
+  (wire (pts (xy 273.05 50.8) (xy 273.05 54.61))
+    (stroke (width 0) (type default))
+  )
   (wire (pts (xy 232.41 146.05) (xy 229.87 146.05))
     (stroke (width 0) (type default))
@@
   )
   (wire (pts (xy 247.65 124.46) (xy 251.46 124.46))
-    (stroke (width 0) (type default))
-  )
-  (wire (pts (xy 246.38 50.8) (xy 262.89 50.8))
     (stroke (width 0) (type default))
   )
@@
     (effects (font (size 3 3) (thickness 0.6) bold italic) (justify left bottom))
   )
-  (label "SDA" (at 29.21 99.06 0) (fields_autoplaced)
+  (label "SDA1" (at 29.21 99.06 0) (fields_autoplaced)
     (effects (font (size 1.27 1.27)) (justify left bottom))
   )
-  (label "SCL" (at 29.21 96.52 0) (fields_autoplaced)
+  (label "SCL1" (at 29.21 96.52 0) (fields_autoplaced)
     (effects (font (size 1.27 1.27)) (justify left bottom))
   )
-  (label "SCL" (at 86.36 52.07 180) (fields_autoplaced)
+  (label "SCL1" (at 86.36 52.07 180) (fields_autoplaced)
     (effects (font (size 1.27 1.27)) (justify right bottom))
   )
-  (label "SDA" (at 86.36 49.53 180) (fields_autoplaced)
+  (label "SDA1" (at 86.36 49.53 180) (fields_autoplaced)
     (effects (font (size 1.27 1.27)) (justify right bottom))
   )
@@
   (symbol (lib_id "Device:C") (at 157.48 152.4 0) (unit 1)
     (in_bom yes) (on_board yes) (dnp no)
-    (property "Reference" "C10" (at 160.02 151.13 0)
+    (property "Reference" "C29" (at 160.02 151.13 0)
       (effects (font (size 1.27 1.27)) (justify left))
     )
@@
       (project "Flight Computer"
         (path "/0c1188a1-706b-46cd-a73a-5b3f8187d77a/319f0b8f-53e5-472b-a337-7eaa627afef4"
-          (reference "C10") (unit 1)
+          (reference "C29") (unit 1)
         )
       )
@@
     )
   )
-  (symbol (lib_id "power:GND") (at 262.89 50.8 0) (unit 1)
-    (in_bom yes) (on_board yes) (dnp no) (fields_autoplaced)
-    (property "Reference" "#PWR017" (at 262.89 57.15 0)
-      (effects (font (size 1.27 1.27)) hide)
-    )
-    (property "Value" "GND" (at 262.89 55.88 0)
-      (effects (font (size 1.27 1.27)) hide)
-    )
-    (property "Footprint" "" (at 262.89 50.8 0)
-      (effects (font (size 1.27 1.27)) hide)
-    )
-    (property "Datasheet" "" (at 262.89 50.8 0)
+  (symbol (lib_id "power:GND") (at 273.05 54.61 0) (unit 1)
+    (in_bom yes) (on_board yes) (dnp no) (fields_autoplaced)
+    (property "Reference" "#PWR017" (at 273.05 60.96 0)
+      (effects (font (size 1.27 1.27)) hide)
+    )
+    (property "Value" "GND" (at 273.05 59.69 0)
+      (effects (font (size 1.27 1.27)) hide)
+    )
+    (property "Footprint" "" (at 273.05 54.61 0)
+      (effects (font (size 1.27 1.27)) hide)
+    )
+    (property "Datasheet" "" (at 273.05 54.61 0)
       (effects (font (size 1.27 1.27)) hide)
     )
@@
   (symbol (lib_id "Device:C") (at 29.21 166.37 0) (unit 1)
     (in_bom yes) (on_board yes) (dnp no)
-    (property "Reference" "C11" (at 31.75 165.1 0)
-      (effects (font (size 1.27 1.27)) (justify left))
-    )
-    (property "Value" "C" (at 31.75 167.64 0)
+    (property "Reference" "C28" (at 31.75 165.1 0)
+      (effects (font (size 1.27 1.27)) (justify left))
+    )
+    (property "Value" "4u7" (at 31.75 167.64 0)
       (effects (font (size 1.27 1.27)) (justify left))
     )
@@
       (project "Flight Computer"
         (path "/0c1188a1-706b-46cd-a73a-5b3f8187d77a/319f0b8f-53e5-472b-a337-7eaa627afef4"
-          (reference "C11") (unit 1)
-        )
-      )
+          (reference "C28") (unit 1)
+        )
+      )

Commit message: Chose footprints for most components
Parts:
- removed R1: 1M, symbol Device:R
- C1, C28, C7: footprint (none) -> Capacitor_SMD:C_0603_1608Metric
- C2, C29, C3, C4, C5, C6, C8, C9: footprint (none) -> Capacitor_SMD:C_0402_1005Metric
- J10: footprint (none) -> Connector_Card:microSD_HC_Hirose_DM3D-SF; symbol Connector:Micro_SD_Card -> Connector:Micro_SD_Card_Det2
Connections:
- net +3.3V: no longer J10.6 (VSS)
- net GND: now also J10.11 (SHIELD), J10.6 (VSS)
- net SD Card Detect: now reaches J10.9 (DET_B)
- net SD Card Detect: now also J10.10 (DET_A)
- net Backup Battery: no longer names the net of U2.6 (V_BCKP)
- no-connect marks 11 -> 12

Commit message: Added custom footprints and started layout
Parts:
- removed J1: GPS antenna, symbol Connector:Conn_Coaxial
- removed U2: MAX-M10S, RF_GPS:ublox_MAX, symbol RF_GPS:MAX-M10S
- added U11: SAM-M8Q, RF_GPS:ublox_SAM-M8Q_HandSolder, symbol RF_GPS:SAM-M8Q
- U3: footprint (none) -> custom-footprints:ADXL375
- U4: footprint (none) -> custom-footprints:BMI088
- U5: footprint (none) -> custom-footprints:BMP388
- U7: value W25Q128JVS -> W25Q128JVEIQ; footprint Package_SO:SOIC-8_5.23x5.23mm_P1.27mm -> Package_SON:WSON-8-1EP_8x6mm_P1.27mm_EP3.4x4.3mm
Connections:
- net +3.3V: now also U11.17 (VCC), U11.2 (VCC_IO)
- net GND: now also U11.1 (GND), U11.10 (GND), U11.11 (GND), U11.15 (GND), U11.16 (GND), U11.20 (GND), U11.4 (GND), U11.5 (GND), U11.6 (GND)
- net GPS External Interrupt: now also U11.19 (EXTINT)
- net GPS Reset: now also U11.18 (~{RESET})
- net UART RX: now also U11.14 (RXD)
- net UART TX: now also U11.13 (TXD)
- no-connect marks 12 -> 10
Other:
- note added: "Fortune smiles upon those who spend more money for the drop-in solution"

Commit message: Finished first draft of layout
Parts:
- U7: value W25Q128JVEIQ -> W25Q128JVSIQ; footprint Package_SON:WSON-8-1EP_8x6mm_P1.27mm_EP3.4x4.3mm -> Package_SO:SOIC-8_5.23x5.23mm_P1.27mm
Changed lines of the file:
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@@
       (effects (font (size 1.27 1.27)) (justify left))
     )
-    (property "Value" "W25Q128JVEIQ" (at 151.13 165.1 0)
+    (property "Value" "W25Q128JVSIQ" (at 151.13 165.1 0)
       (effects (font (size 1.27 1.27)) (justify left))
     )
-    (property "Footprint" "Package_SON:WSON-8-1EP_8x6mm_P1.27mm_EP3.4x4.3mm" (at 142.24 163.83 0)
+    (property "Footprint" "Package_SO:SOIC-8_5.23x5.23mm_P1.27mm" (at 142.24 163.83 0)
       (effects (font (size 1.27 1.27)) hide)
     )

Commit message: How many sheets do you want? Yes
Parts:
- removed C6, C9: 100n, Capacitor_SMD:C_0402_1005Metric, symbol Device:C
- removed C7: 1u, Capacitor_SMD:C_0603_1608Metric, symbol Device:C
- removed U1: LIS3MDL, Package_LGA:LGA-12_2x2mm_P0.5mm, symbol Sensor_Magnetic:LIS3MDL
Connections:
- net SCL1 is gone; now on net SPI SCK: U3.14 (SCL/SCK)
- net SCL3 is gone; now on net SPI SCK: U5.2 (SCK)
- net SDA1 is gone; now on net SPI MOSI: U3.13 (SDA/SDI)
- net SDA3 is gone; now on net SPI MOSI: U5.4 (SDI)
- net +3.3V: now also C5.1; no longer U3.12 (SDO/Addr_sel), U3.7 (Chip_Select), U5.6 (Chip_Select)
- net GND: no longer U5.5 (SDO)
- net SPI MISO: now also U3.12 (SDO/Addr_sel), U5.5 (SDO)
- net High G Interrupt 1 renamed High G Interrupt
- net Low G Accel Interrupt 1 renamed Low G Accel Interrupt
- net Low G Gyro Interrupt 3 renamed Low G Gyro Interrupt
- new net Chip Select Altimeter: U5.6 (Chip_Select)
- new net Chip Select High G Accel: U3.7 (Chip_Select)
Other:
- note added: "Also fortune would smile upon U-blox for not making me use UART or I2C, but they don't seem to care about that. External GPS for stuff like Pixhawks always seem to use UART, so nothing will **ever** go wrong with this"
- note added: "NOR flash which is kinda sad, but it is a basic part at JLC (no $3 fee for this part woohoo)"
- note added: "This is the high G accelerometer, (±64 Gs), for events like chute deployment and really *chonky* motors"
- note added: "This is worse than the MS5611 we were planning on using, but it is easier to find at JLC (AKA JLC forgot to buy new MS5611s and ran out)"
- note added: "U-blox SAM-M10 (the latest and greatest GPS module that does everything for you A.K.A. I'm not an RF engineer"
- note removed: "Honestly don't know why I bother with a magnetometer, it's not like heading is relevant beyond what GPS coordinates give us"
- note removed: "I2C"
- note removed: "This is worse than the MS5611 we were planning on using, but it is easier to find at JLC"
- note removed: "Thisis the high G accelerometer, (±64 Gs), for events like chute deployment"
- moved on the sheet: C2, C28, C3, C8, J10, U11, U3, U4, U5
