File: sensors.kicad_sch (KiCad schematic)
At the start: 14 parts, among them J10 Micro_SD_Card, U11 SAM-M8Q, U7 W25Q128JVSIQ

Commit message: Started doing layout for v1.1
Other:
- note added: "U-blox SAM-M10 the latest and greatest GPS module that does everything for you A.K.A. I'm not an RF engineer"
- note removed: "U-blox SAM-M10 (the latest and greatest GPS module that does everything for you A.K.A. I'm not an RF engineer"
Changed lines of the file:
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@@
     (effects (font (size 3 3) (thickness 0.6) bold italic) (justify left bottom))
   )
-  (text "U-blox SAM-M10 (the latest and greatest GPS module that\ndoes everything for you A.K.A. I'm not an RF engineer"
+  (text "U-blox SAM-M10 the latest and greatest GPS module that\ndoes everything for you A.K.A. I'm not an RF engineer"
     (at 210.82 72.39 0)
     (effects (font (size 1.27 1.27)) (justify left bottom))

Commit message: Updated with notes from Erik Welsh
Parts:
- added R48, R49, R50, R51, R52, R53, R54, R55: 0, Resistor_SMD:R_0402_1005Metric, symbol Device:R
Connections:
- net +3.3V: now also R48.1, R50.1, R52.1, R54.1
- net Chip Select Altimeter: now also R54.2, R55.1
- net Chip Select High G Accel: now also R48.2, R49.1
- net Chip Select Low G Accel: now also R50.2, R51.1
- net Chip Select Low G Gyro: now also R52.2, R53.1
- net GND: now also R49.2, R51.2, R53.2, R55.2

Commit message: Finished final(tm) updates for v1.1
Other:
- note added: "NOR flash (I think, honestly unclear) basic part at JLC (no $3 fee for this part woohoo); current draw of 20mA is fine"
- note removed: "NOR flash which is kinda sad, but it is a basic part at JLC (no $3 fee for this part woohoo)"
Changed lines of the file:
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@@
     (effects (font (size 1.27 1.27)) (justify left bottom))
   )
-  (text "NOR flash which is kinda sad, but it is a basic\npart at JLC (no $3 fee for this part woohoo)"
-    (at 116.84 189.23 0)
+  (text "NOR flash (I think, honestly unclear)\nbasic part at JLC (no $3 fee for this\npart woohoo); current draw of 20mA is\nfine"
+    (at 119.38 193.04 0)
     (effects (font (size 1.27 1.27)) (justify left bottom))
   )

Commit message: Swapped out sensors in schematic for v3
Parts:
- removed C28: 4u7, Capacitor_SMD:C_0603_1608Metric, symbol Device:C
- removed J10: Micro_SD_Card, Connector_Card:microSD_HC_Hirose_DM3D-SF, symbol Connector:Micro_SD_Card_Det2
- removed R48, R49, R50, R51, R52, R53, R54, R55: 0, Resistor_SMD:R_0402_1005Metric, symbol Device:R
- removed U3: ~, custom-footprints:ADXL375, symbol custom-symbols:ADXL375
- added C17, C18, C19: 100n, Capacitor_SMD:C_0402_1005Metric, symbol Device:C
- added U10: ~, symbol custom-symbols:KX134-1211
- added U9: LIS3MDL, Package_LGA:LGA-12_2x2mm_P0.5mm, symbol Sensor_Magnetic:LIS3MDL
- C1: value 1u -> 100n; footprint Capacitor_SMD:C_0603_1608Metric -> Capacitor_SMD:C_0402_1005Metric
Connections:
- net +3.3V: now also C17.1, C18.1, U10.3 (IO_Vdd), U10.7 (Vdd), U9.5 (Vdd), U9.6 (Vdd_IO)
- net GND: now also C17.2, C18.2, C19.2, U10.4 (Trig), U10.8 (GND), U10.9 (GND), U9.12 (GND), U9.2 (GND), U9.3 (GND)
- net SPI MISO renamed SPI1 MISO
- net SPI MOSI renamed SPI1 MOSI
- net SPI SCK renamed SPI1 SCK
- new net: C19.1, U9.4 (C1)
- new net High G Accelerometer Chip Select: U10.10 (nCS)
- new net High G Accelerometer Interrupt: U10.5 (Int_1)
- new net Magnetometer Chip Select: U9.10 (~{CS})
- new net Magnetometer Interrupt: U9.7 (INT)
- new net SPI2 MISO: U10.1 (SDO/ADDR), U9.9 (SDO/SA1)
- new net SPI2 MOSI: U10.2 (SDI/SDA), U9.11 (SDA/SDI/SDO)
- new net SPI2 SCK: U10.12 (SCK), U9.1 (SCL/SPC)
- no-connect marks 10 -> 9
Other:
- note added: "SPI1"
- note added: "SPI2"
- note added: "This high-g accelerometer is new for version 3, because it has ~20x the precision and might not be designed by buffoons"
- note removed: "Also fortune would smile upon U-blox for not making me use UART or I2C, but they don't seem to care about that. External GPS for stuff like Pixhawks always seem to use UART, so nothing will **ever** go wrong with this"
- note removed: "Fortune smiles upon those who spend more money for the drop-in solution"
- note removed: "SPI"
- note removed: "This is the high G accelerometer, (±64 Gs), for events like chute deployment and really *chonky* motors"
- note removed: "This is worse than the MS5611 we were planning on using, but it is easier to find at JLC (AKA JLC forgot to buy new MS5611s and ran out)"
- note removed: "U-blox SAM-M10 the latest and greatest GPS module that does everything for you A.K.A. I'm not an RF engineer"
- moved on the sheet: C29, C3, C4, C5, C8, U11, U4, U5, U7

Commit message: STarted layout for v3
Parts:
- U10: footprint (none) -> custom-footprints:KX134-1211
Connections:
- net SPI2 MISO renamed SPI3 MISO
- net SPI2 MOSI renamed SPI3 MOSI
- net SPI2 SCK renamed SPI3 SCK
Other:
- note added: "KX134-1211"
Changed lines of the file:
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@@
+    (effects (font (size 1.27 1.27)) (justify left bottom))
+  )
+  (text "KX134-1211" (at 227.33 118.11 0)
     (effects (font (size 1.27 1.27)) (justify left bottom))
   )
@@
     (effects (font (size 3 3) (thickness 0.6) bold italic) (justify left bottom))
   )
-  (label "SPI2 SCK" (at 187.96 102.87 0) (fields_autoplaced)
+  (label "SPI3 SCK" (at 187.96 102.87 0) (fields_autoplaced)
     (effects (font (size 1.27 1.27)) (justify left bottom))
   )
@@
     (effects (font (size 1.27 1.27)) (justify left bottom))
   )
-  (label "SPI2 MISO" (at 186.69 54.61 0) (fields_autoplaced)
+  (label "SPI3 MISO" (at 186.69 54.61 0) (fields_autoplaced)
     (effects (font (size 1.27 1.27)) (justify left bottom))
   )
-  (label "SPI2 MOSI" (at 186.69 52.07 0) (fields_autoplaced)
+  (label "SPI3 MOSI" (at 186.69 52.07 0) (fields_autoplaced)
     (effects (font (size 1.27 1.27)) (justify left bottom))
   )
-  (label "SPI2 MOSI" (at 187.96 107.95 0) (fields_autoplaced)
+  (label "SPI3 MOSI" (at 187.96 107.95 0) (fields_autoplaced)
     (effects (font (size 1.27 1.27)) (justify left bottom))
   )
@@
     (effects (font (size 1.27 1.27)) (justify left bottom))
   )
-  (label "SPI2 SCK" (at 186.69 49.53 0) (fields_autoplaced)
+  (label "SPI3 SCK" (at 186.69 49.53 0) (fields_autoplaced)
     (effects (font (size 1.27 1.27)) (justify left bottom))
   )
@@
     (effects (font (size 1.27 1.27)) (justify left bottom))
   )
-  (label "SPI2 MISO" (at 187.96 105.41 0) (fields_autoplaced)
+  (label "SPI3 MISO" (at 187.96 105.41 0) (fields_autoplaced)
     (effects (font (size 1.27 1.27)) (justify left bottom))
   )
@@
     (effects (font (size 1.27 1.27)) (justify right))
   )
-  (hierarchical_label "SPI2 SCK" (shape input) (at 185.42 49.53 180) (fields_autoplaced)
+  (hierarchical_label "SPI3 SCK" (shape input) (at 185.42 49.53 180) (fields_autoplaced)
     (effects (font (size 1.27 1.27)) (justify right))
   )
@@
     (effects (font (size 1.27 1.27)) (justify right))
   )
-  (hierarchical_label "SPI2 MISO" (shape output) (at 185.42 54.61 180) (fields_autoplaced)
+  (hierarchical_label "SPI3 MISO" (shape output) (at 185.42 54.61 180) (fields_autoplaced)
     (effects (font (size 1.27 1.27)) (justify right))
   )
-  (hierarchical_label "SPI2 MOSI" (shape input) (at 185.42 52.07 180) (fields_autoplaced)
+  (hierarchical_label "SPI3 MOSI" (shape input) (at 185.42 52.07 180) (fields_autoplaced)
     (effects (font (size 1.27 1.27)) (justify right))
   )
@@
       (effects (font (size 1.27 1.27)))
     )
-    (property "Footprint" "" (at 214.63 110.49 0)
+    (property "Footprint" "custom-footprints:KX134-1211" (at 214.63 110.49 0)
       (effects (font (size 1.27 1.27)) hide)
     )
