File: connectors.kicad_sch (KiCad schematic)
At the start: 11 parts, among them J4 JST-PH, J5 External SPI, J6 Serial Wire Debug, J7 USB_C_Receptacle_USB2.0, J8 External UART, J9 External I2C, U2 USBLC6-2SC6

Commit message: Added new buck converter
Parts:
- removed J6: Serial Wire Debug, Connector_Molex:Molex_PicoBlade_53048-0410_1x04_P1.25mm_Horizontal, symbol Connector_Generic:Conn_01x04
- added J3: External SPI, Connector_Molex:Molex_PicoBlade_53048-0510_1x05_P1.25mm_Horizontal, symbol Connector_Generic:Conn_01x05
Connections:
- net +5V is gone; now on net Main battery in: J8.1 (Pin_1)
- net +3.3V: now also J3.1 (Pin_1)
- net GND: now also J3.5 (Pin_5)
- net NRST: now also J3.2 (Pin_2)
- net SWCLK: now also J3.3 (Pin_3)
- net SWDIO: now also J3.4 (Pin_4)
Changed lines of the file:
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@@
     (stroke (width 0) (type default))
   )
-  (wire (pts (xy 116.84 138.43) (xy 116.84 135.89))
-    (stroke (width 0) (type default))
-  )
-  (wire (pts (xy 116.84 130.81) (xy 124.46 130.81))
+  (wire (pts (xy 114.3 143.51) (xy 114.3 140.97))
+    (stroke (width 0) (type default))
+  )
+  (wire (pts (xy 114.3 135.89) (xy 121.92 135.89))
     (stroke (width 0) (type default))
   )
@@
     (stroke (width 0) (type default))
   )
-  (wire (pts (xy 231.14 63.5) (xy 231.14 66.04))
-    (stroke (width 0) (type default))
-  )
   (wire (pts (xy 59.69 102.87) (xy 67.31 102.87))
     (stroke (width 0) (type default))
@@
     (stroke (width 0) (type default))
   )
-  (wire (pts (xy 116.84 133.35) (xy 124.46 133.35))
+  (wire (pts (xy 114.3 138.43) (xy 121.92 138.43))
     (stroke (width 0) (type default))
   )
@@
     (stroke (width 0) (type default))
   )
-  (wire (pts (xy 116.84 128.27) (xy 124.46 128.27))
+  (wire (pts (xy 114.3 133.35) (xy 121.92 133.35))
     (stroke (width 0) (type default))
   )
@@
     (stroke (width 0) (type default))
   )
+  (wire (pts (xy 114.3 128.27) (xy 114.3 130.81))
+    (stroke (width 0) (type default))
+  )
   (wire (pts (xy 234.95 121.92) (xy 231.14 121.92))
     (stroke (width 0) (type default))
@@
     (stroke (width 0) (type default))
   )
+  (wire (pts (xy 121.92 130.81) (xy 114.3 130.81))
+    (stroke (width 0) (type default))
+  )
   (wire (pts (xy 231.14 132.08) (xy 231.14 134.62))
     (stroke (width 0) (type default))
@@
     (stroke (width 0) (type default))
   )
-  (wire (pts (xy 116.84 135.89) (xy 124.46 135.89))
+  (wire (pts (xy 114.3 140.97) (xy 121.92 140.97))
     (stroke (width 0) (type default))
   )
@@
     (effects (font (size 1.27 1.27)) (justify right))
   )
+  (hierarchical_label "Main battery in" (shape input) (at 231.14 66.04 180) (fields_autoplaced)
+    (effects (font (size 1.27 1.27)) (justify right))
+  )
   (hierarchical_label "USB 5V in" (shape input) (at 105.41 54.61 0) (fields_autoplaced)
     (effects (font (size 1.27 1.27)) (justify left))
@@
     (effects (font (size 1.27 1.27)) (justify right))
   )
-  (hierarchical_label "SWCLK" (shape input) (at 116.84 130.81 180) (fields_autoplaced)
+  (hierarchical_label "SWCLK" (shape input) (at 114.3 135.89 180) (fields_autoplaced)
     (effects (font (size 1.27 1.27)) (justify right))
   )
@@
     (effects (font (size 1.27 1.27)) (justify right))
   )
-  (hierarchical_label "SWDIO" (shape input) (at 116.84 133.35 180) (fields_autoplaced)
+  (hierarchical_label "SWDIO" (shape input) (at 114.3 138.43 180) (fields_autoplaced)
     (effects (font (size 1.27 1.27)) (justify right))
   )
@@
     (effects (font (size 1.27 1.27)) (justify left))
   )
-  (hierarchical_label "NRST" (shape input) (at 116.84 128.27 180) (fields_autoplaced)
+  (hierarchical_label "NRST" (shape input) (at 114.3 133.35 180) (fields_autoplaced)
     (effects (font (size 1.27 1.27)) (justify right))
   )
@@
     )
   )
+  (symbol (lib_id "power:+3.3V") (at 114.3 128.27 0) (unit 1)
+    (in_bom yes) (on_board yes) (dnp no) (fields_autoplaced)
+    (property "Reference" "#PWR064" (at 114.3 132.08 0)
+      (effects (font (size 1.27 1.27)) hide)
+    )
+    (property "Value" "+3.3V" (at 114.3 124.46 0)
+      (effects (font (size 1.27 1.27)))
+    )
+    (property "Footprint" "" (at 114.3 128.27 0)
+      (effects (font (size 1.27 1.27)) hide)
+    )
+    (property "Datasheet" "" (at 114.3 128.27 0)
+      (effects (font (size 1.27 1.27)) hide)
+    )
+    (pin "1")
+    (instances
+      (project "Flight Computer"
+        (path "/0c1188a1-706b-46cd-a73a-5b3f8187d77a/afc466af-6d84-4e19-b5b5-aea43618ea20"
+          (reference "#PWR064") (unit 1)
+        )
+      )
+    )
+  )
   (symbol (lib_id "Device:C") (at 50.8 97.79 0) (unit 1)
     (in_bom yes) (on_board yes) (dnp no)
@@
     )
   )
-  (symbol (lib_id "power:GND") (at 116.84 138.43 0) (unit 1)
-    (in_bom yes) (on_board yes) (dnp no)
-    (property "Reference" "#PWR051" (at 116.84 144.78 0)
-      (effects (font (size 1.27 1.27)) hide)
-    )
-    (property "Value" "GND" (at 116.84 143.51 0)
-      (effects (font (size 1.27 1.27)) hide)
-    )
-    (property "Footprint" "" (at 116.84 138.43 0)
-      (effects (font (size 1.27 1.27)) hide)
-    )
-    (property "Datasheet" "" (at 116.84 138.43 0)
+  (symbol (lib_id "power:GND") (at 114.3 143.51 0) (unit 1)
+    (in_bom yes) (on_board yes) (dnp no)
+    (property "Reference" "#PWR051" (at 114.3 149.86 0)
+      (effects (font (size 1.27 1.27)) hide)
+    )
+    (property "Value" "GND" (at 114.3 148.59 0)
+      (effects (font (size 1.27 1.27)) hide)
+    )
+    (property "Footprint" "" (at 114.3 143.51 0)
+      (effects (font (size 1.27 1.27)) hide)
+    )
+    (property "Datasheet" "" (at 114.3 143.51 0)
       (effects (font (size 1.27 1.27)) hide)
     )
@@
         (path "/0c1188a1-706b-46cd-a73a-5b3f8187d77a/afc466af-6d84-4e19-b5b5-aea43618ea20"
           (reference "#PWR048") (unit 1)
-        )
-      )
-    )
-  )
-  (symbol (lib_id "power:+5V") (at 231.14 63.5 0) (unit 1)
-    (in_bom yes) (on_board yes) (dnp no) (fields_autoplaced)
-    (property "Reference" "#PWR059" (at 231.14 67.31 0)
-      (effects (font (size 1.27 1.27)) hide)
-    )
-    (property "Value" "+5V" (at 231.14 59.69 0)
-      (effects (font (size 1.27 1.27)))
-    )
-    (property "Footprint" "" (at 231.14 63.5 0)
-      (effects (font (size 1.27 1.27)) hide)
-    )
-    (property "Datasheet" "" (at 231.14 63.5 0)
-      (effects (font (size 1.27 1.27)) hide)
-    )
-    (pin "1")
-    (instances
-      (project "Flight Computer"
-        (path "/0c1188a1-706b-46cd-a73a-5b3f8187d77a/afc466af-6d84-4e19-b5b5-aea43618ea20"
-          (reference "#PWR059") (unit 1)
         )
       )
@@
         (path "/0c1188a1-706b-46cd-a73a-5b3f8187d77a/afc466af-6d84-4e19-b5b5-aea43618ea20"
           (reference "#PWR0118") (unit 1)
+        )
+      )
+    )
+  )
+  (symbol (lib_id "Connector_Generic:Conn_01x05") (at 127 135.89 0) (unit 1)
+    (in_bom yes) (on_board yes) (dnp no)
+    (property "Reference" "J3" (at 129.54 135.255 0)
+      (effects (font (size 1.27 1.27)) (justify left))
+    )
+    (property "Value" "External SPI" (at 120.65 143.51 0)
+      (effects (font (size 1.27 1.27)) (justify left))
+    )
+    (property "Footprint" "Connector_Molex:Molex_PicoBlade_53048-0510_1x05_P1.25mm_Horizontal" (at 127 135.89 0)
+      (effects (font (size 1.27 1.27)) hide)
+    )
+    (property "Datasheet" "~" (at 127 135.89 0)
+      (effects (font (size 1.27 1.27)) hide)
+    )
+    (pin "1")
+    (pin "2")
+    (pin "3")
+    (pin "4")
+    (pin "5")
+    (instances
+      (project "Flight Computer"
+        (path "/0c1188a1-706b-46cd-a73a-5b3f8187d77a/afc466af-6d84-4e19-b5b5-aea43618ea20"
+          (reference "J3") (unit 1)
         )
       )
@@
         )
       )
-    )
-  )
-  (symbol (lib_id "Connector_Generic:Conn_01x04") (at 129.54 130.81 0) (unit 1)
-    (in_bom yes) (on_board yes) (dnp no)
-    (property "Reference" "J6" (at 132.08 131.445 0)
-      (effects (font (size 1.27 1.27)) (justify left))
-    )
-    (property "Value" "Serial Wire Debug" (at 121.92 138.43 0)
-      (effects (font (size 1.27 1.27)) (justify left))
-    )
-    (property "Footprint" "Connector_Molex:Molex_PicoBlade_53048-0410_1x04_P1.25mm_Horizontal" (at 129.54 130.81 0)
-      (effects (font (size 1.27 1.27)) hide)
-    )
-    (property "Datasheet" "~" (at 129.54 130.81 0)
-      (effects (font (size 1.27 1.27)) hide)
-    )
-    (pin "1")
-    (pin "2")
-    (pin "3")
-    (pin "4")
-    (instances
-      (project "Flight Computer"
-        (path "/0c1188a1-706b-46cd-a73a-5b3f8187d77a/afc466af-6d84-4e19-b5b5-aea43618ea20"
-          (reference "J6") (unit 1)
-        )
-      )

Commit message: finished preliminary v2 modifications
Connections:
- net Main battery in: no longer J8.1 (Pin_1)
- net USB 5V in: now also J8.1 (Pin_1)
Changed lines of the file:
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@@
     (stroke (width 0) (type default))
   )
-  (wire (pts (xy 234.95 66.04) (xy 231.14 66.04))
+  (wire (pts (xy 234.95 66.04) (xy 220.98 66.04))
     (stroke (width 0) (type default))
   )
@@
     (effects (font (size 1.27 1.27)) (justify right bottom))
   )
+  (label "USB 5V in" (at 220.98 66.04 0) (fields_autoplaced)
+    (effects (font (size 1.27 1.27)) (justify left bottom))
+  )
   (label "USB CONN D-" (at 99.06 67.31 180) (fields_autoplaced)
     (effects (font (size 1.27 1.27)) (justify right bottom))
@@
     (effects (font (size 1.27 1.27)) (justify right))
   )
-  (hierarchical_label "Main battery in" (shape input) (at 231.14 66.04 180) (fields_autoplaced)
-    (effects (font (size 1.27 1.27)) (justify right))
-  )
