File: connectors.kicad_sch (KiCad schematic)
At the start: 11 parts, among them J3 External SPI, J4 JST-PH, J5 External SPI, J7 USB_C_Receptacle_USB2.0, J8 External UART, J9 External I2C, U2 USBLC6-2SC6

Commit message: added switch to USB power and to bypass screw switch for main battery
Parts:
- added SW1: Screw Switch Bypass, Button_Switch_SMD:SW_SPDT_PCM12, symbol Switch:SW_SPDT
Connections:
- net Main battery connector: now also SW1.2 (B)
- net Main battery in: now also SW1.1 (A)
- net USB 5V in: no longer J8.1 (Pin_1)
- new net Vin_combined: J8.1 (Pin_1)
- no-connect marks 2 -> 3
Other:
- sheet Power Supply ports: added Vin_combined; removed none
- moved on the sheet: J3, J4

Commit message: Fixed BOM
Parts:
- C25: value 0.01u -> 100n
Changed lines of the file:
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@@
       (effects (font (size 1.27 1.27)) (justify left))
     )
-    (property "Value" "0.01u" (at 53.34 99.06 0)
+    (property "Value" "100n" (at 53.34 99.06 0)
       (effects (font (size 1.27 1.27)) (justify left))
     )

Commit message: Minor changes to fit jlc capabilities
Parts:
- J7: footprint Connector_USB:USB_C_Receptacle_G-Switch_GT-USB-7010ASV -> Connector_USB:USB_C_Receptacle_HRO_TYPE-C-31-M-12
Changed lines of the file:
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@@
       (effects (font (size 1.27 1.27)))
     )
-    (property "Footprint" "Connector_USB:USB_C_Receptacle_G-Switch_GT-USB-7010ASV" (at 71.12 69.85 0)
+    (property "Footprint" "Connector_USB:USB_C_Receptacle_HRO_TYPE-C-31-M-12" (at 71.12 69.85 0)
       (effects (font (size 1.27 1.27)) hide)
     )

Commit message: Swapped out sensors in schematic for v3
Changed lines of the file:
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@@
   (junction (at 100.33 54.61) (diameter 0) (color 0 0 0 0)
+  )
+  (junction (at 80.01 137.16) (diameter 0) (color 0 0 0 0)
   )
   (no_connect (at 96.52 134.62))
@@
     (stroke (width 0) (type default))
   )
+  (wire (pts (xy 80.01 137.16) (xy 86.36 137.16))
+    (stroke (width 0) (type default))
+  )
   (wire (pts (xy 85.09 74.93) (xy 85.09 72.39))
     (stroke (width 0) (type default))
@@
     (stroke (width 0) (type default))
   )
-  (wire (pts (xy 57.15 137.16) (xy 86.36 137.16))
+  (wire (pts (xy 57.15 137.16) (xy 80.01 137.16))
     (stroke (width 0) (type default))
   )
@@
         )
       )
+    )
+  )
+  (symbol (lib_id "power:PWR_FLAG") (at 80.01 137.16 180) (unit 1)
+    (in_bom yes) (on_board yes) (dnp no)
+    (property "Reference" "#FLG02" (at 80.01 139.065 0)
+      (effects (font (size 1.27 1.27)) hide)
+    )
+    (property "Value" "PWR_FLAG" (at 83.82 140.97 0)
+      (effects (font (size 1.27 1.27)) (justify left))
+    )
+    (property "Footprint" "" (at 80.01 137.16 0)
+      (effects (font (size 1.27 1.27)) hide)
+    )
+    (property "Datasheet" "~" (at 80.01 137.16 0)
+      (effects (font (size 1.27 1.27)) hide)
+    )
+    (pin "1")
+    (instances
+      (project "Flight Computer"
+        (path "/0c1188a1-706b-46cd-a73a-5b3f8187d77a"
+          (reference "#FLG02") (unit 1)
+        )
+        (path "/0c1188a1-706b-46cd-a73a-5b3f8187d77a/afc466af-6d84-4e19-b5b5-aea43618ea20"
+          (reference "#FLG01") (unit 1)
+        )
+      )

Commit message: STarted layout for v3
Parts:
- removed J5: External SPI, Connector_Molex:Molex_PicoBlade_53048-0510_1x05_P1.25mm_Horizontal, symbol Connector_Generic:Conn_01x05
Other:
- moved on the sheet: J8, J9

Commit message: Finished preliminary layout of v3
Parts:
- removed J7: USB_C_Receptacle_USB2.0, Connector_USB:USB_C_Receptacle_HRO_TYPE-C-31-M-12, symbol Connector:USB_C_Receptacle_USB2.0
- removed R20, R21: 5.1k, Resistor_SMD:R_0603_1608Metric, symbol Device:R
- added J5: USB_B_Micro, Connector_USB:USB_Micro-B_Amphenol_10118194_Horizontal, symbol Connector:USB_B_Micro
Connections:
- net GND: now also J5.5 (GND)
- net USB 5V in: now also J5.1 (VBUS)
- net USB CONN D+: now also J5.3 (D+)
- net USB CONN D-: now also J5.2 (D-)
- net at C25.1, R19.1: now also J5.6 (Shield)
- no-connect marks 3 -> 2
Other:
- note added: "Using micro-usb because USB wasn't enumerating with USBC, so this might fix the problem"
- moved on the sheet: C25, R19
