File: pyro-channels.kicad_sch (KiCad schematic)
At the start: 0 parts

Commit message: Added power supply circuitry, as well as example pyrotechnic channel MOSFET
Parts:
- added Q2: AO3400A, Package_TO_SOT_SMD:SOT-23, symbol Transistor_FET:AO3400A
- added R4: 220k, symbol Device:R
- added R6: 22k, symbol Device:R
Connections:
- new net GND: Q2.2 (S), R6.2
- new net Pyro Channel A: Q2.3 (D), R4.1
- new net Pyro Channel A Continuity Voltage: R4.2, R6.1
- new net Pyro Channel A Trigger: Q2.1 (G)
Other:
- note added: "This is the actual Pyro Channel. One of the charge's leads connects to this, the other to the positive ignition battery voltage. To trigger, this input is shorted to ground."
- note added: "We want to be able to measure voltage on Pyro Channel, since this is how we can detect continuity. To avoid damaging the MCU's ADC, we use a voltage divider, so the voltage read is 1/11 of the ignition battery voltage"
- note added: "When the pyro channel is triggered, MCU applies voltage to this pin"
Changed lines of the file:
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@@
   (title_block
     (title "Pyrotechnic Channels")
-    (date "2023-09-19")
-    (rev "0")
+    (date "2023-09-23")
+    (rev "0.5")
+  )
+  (junction (at 71.12 34.29) (diameter 0) (color 0 0 0 0)
+  )
+  (junction (at 71.12 45.72) (diameter 0) (color 0 0 0 0)
+  )
+  (wire (pts (xy 71.12 34.29) (xy 80.01 34.29))
+    (stroke (width 0) (type default))
+  )
+  (wire (pts (xy 71.12 54.61) (xy 71.12 57.15))
+    (stroke (width 0) (type default))
+  )
+  (wire (pts (xy 71.12 34.29) (xy 71.12 36.83))
+    (stroke (width 0) (type default))
+  )
+  (wire (pts (xy 71.12 45.72) (xy 71.12 46.99))
+    (stroke (width 0) (type default))
+  )
+  (wire (pts (xy 66.04 45.72) (xy 71.12 45.72))
+    (stroke (width 0) (type default))
+  )
+  (wire (pts (xy 90.17 34.29) (xy 99.06 34.29))
+    (stroke (width 0) (type default))
+  )
+  (wire (pts (xy 85.09 45.72) (xy 88.9 45.72))
+    (stroke (width 0) (type default))
+  )
+  (wire (pts (xy 85.09 45.72) (xy 85.09 41.91))
+    (stroke (width 0) (type default))
+  )
+  (wire (pts (xy 71.12 44.45) (xy 71.12 45.72))
+    (stroke (width 0) (type default))
+  )
+  (wire (pts (xy 67.31 34.29) (xy 71.12 34.29))
+    (stroke (width 0) (type default))
+  )
+  (wire (pts (xy 99.06 34.29) (xy 99.06 36.83))
+    (stroke (width 0) (type default))
+  )
+  (text "When the pyro channel is triggered, \nMCU applies voltage to this pin"
+    (at 90.17 54.61 0)
+    (effects (font (size 1.27 1.27)) (justify left bottom))
+  )
+  (text "This is the actual Pyro Channel. One of the\ncharge's leads connects to this, the other to the\npositive ignition battery voltage. To trigger,\nthis input is shorted to ground."
+    (at 33.02 26.67 0)
+    (effects (font (size 1.27 1.27)) (justify left bottom))
+  )
+  (text "We want to be able to measure voltage on\nPyro Channel, since this is how we can\ndetect continuity. To avoid damaging the\nMCU's ADC, we use a voltage divider, so\nthe voltage read is 1/11 of the ignition\nbattery voltage"
+    (at 21.59 69.85 0)
+    (effects (font (size 1.27 1.27)) (justify left bottom))
+  )
+  (hierarchical_label "Pyro Channel A Trigger" (shape input) (at 88.9 45.72 0) (fields_autoplaced)
+    (effects (font (size 1.27 1.27)) (justify left))
+  )
+  (hierarchical_label "Pyro Channel A Continuity Voltage" (shape input) (at 66.04 45.72 180) (fields_autoplaced)
+    (effects (font (size 1.27 1.27)) (justify right))
+  )
+  (hierarchical_label "Pyro Channel A" (shape input) (at 67.31 34.29 180) (fields_autoplaced)
+    (effects (font (size 1.27 1.27)) (justify right))
+  )
+  (symbol (lib_id "power:GND") (at 99.06 36.83 0) (unit 1)
+    (in_bom yes) (on_board yes) (dnp no) (fields_autoplaced)
+    (property "Reference" "#PWR032" (at 99.06 43.18 0)
+      (effects (font (size 1.27 1.27)) hide)
+    )
+    (property "Value" "GND" (at 99.06 41.91 0)
+      (effects (font (size 1.27 1.27)) hide)
+    )
+    (property "Footprint" "" (at 99.06 36.83 0)
+      (effects (font (size 1.27 1.27)) hide)
+    )
+    (property "Datasheet" "" (at 99.06 36.83 0)
+      (effects (font (size 1.27 1.27)) hide)
+    )
+    (pin "1")
+    (instances
+      (project "Flight Computer"
+        (path "/0c1188a1-706b-46cd-a73a-5b3f8187d77a/8b5c3409-c69f-490d-a71d-45a34969a1f1"
+          (reference "#PWR032") (unit 1)
+        )
+      )
+    )
+  )
+  (symbol (lib_id "Device:R") (at 71.12 50.8 0) (unit 1)
+    (in_bom yes) (on_board yes) (dnp no)
+    (property "Reference" "R6" (at 72.39 49.53 0)
+      (effects (font (size 1.27 1.27)) (justify left))
+    )
+    (property "Value" "22k" (at 72.39 52.07 0)
+      (effects (font (size 1.27 1.27)) (justify left))
+    )
+    (property "Footprint" "" (at 69.342 50.8 90)
+      (effects (font (size 1.27 1.27)) hide)
+    )
+    (property "Datasheet" "~" (at 71.12 50.8 0)
+      (effects (font (size 1.27 1.27)) hide)
+    )
+    (pin "1")
+    (pin "2")
+    (instances
+      (project "Flight Computer"
+        (path "/0c1188a1-706b-46cd-a73a-5b3f8187d77a/8b5c3409-c69f-490d-a71d-45a34969a1f1"
+          (reference "R6") (unit 1)
+        )
+      )
+    )
+  )
+  (symbol (lib_id "power:GND") (at 71.12 57.15 0) (unit 1)
+    (in_bom yes) (on_board yes) (dnp no) (fields_autoplaced)
+    (property "Reference" "#PWR033" (at 71.12 63.5 0)
+      (effects (font (size 1.27 1.27)) hide)
+    )
+    (property "Value" "GND" (at 71.12 62.23 0)
+      (effects (font (size 1.27 1.27)) hide)
+    )
+    (property "Footprint" "" (at 71.12 57.15 0)
+      (effects (font (size 1.27 1.27)) hide)
+    )
+    (property "Datasheet" "" (at 71.12 57.15 0)
+      (effects (font (size 1.27 1.27)) hide)
+    )
+    (pin "1")
+    (instances
+      (project "Flight Computer"
+        (path "/0c1188a1-706b-46cd-a73a-5b3f8187d77a/8b5c3409-c69f-490d-a71d-45a34969a1f1"
+          (reference "#PWR033") (unit 1)
+        )
+      )
+    )
+  )
+  (symbol (lib_id "Transistor_FET:AO3400A") (at 85.09 36.83 90) (unit 1)
+    (in_bom yes) (on_board yes) (dnp no) (fields_autoplaced)
+    (property "Reference" "Q2" (at 85.09 27.94 90)
+      (effects (font (size 1.27 1.27)))
+    )
+    (property "Value" "AO3400A" (at 85.09 30.48 90)
+      (effects (font (size 1.27 1.27)))
+    )
+    (property "Footprint" "Package_TO_SOT_SMD:SOT-23" (at 86.995 31.75 0)
+      (effects (font (size 1.27 1.27) italic) (justify left) hide)
+    )
+    (property "Datasheet" "http://www.aosmd.com/pdfs/datasheet/AO3400A.pdf" (at 85.09 36.83 0)
+      (effects (font (size 1.27 1.27)) (justify left) hide)
+    )
+    (pin "1")
+    (pin "2")
+    (pin "3")
+    (instances
+      (project "Flight Computer"
+        (path "/0c1188a1-706b-46cd-a73a-5b3f8187d77a/8b5c3409-c69f-490d-a71d-45a34969a1f1"
+          (reference "Q2") (unit 1)
+        )
+      )
+    )
+  )
+  (symbol (lib_id "Device:R") (at 71.12 40.64 0) (unit 1)
+    (in_bom yes) (on_board yes) (dnp no)
+    (property "Reference" "R4" (at 72.39 39.37 0)
+      (effects (font (size 1.27 1.27)) (justify left))
+    )
+    (property "Value" "220k" (at 72.39 41.91 0)
+      (effects (font (size 1.27 1.27)) (justify left))
+    )
+    (property "Footprint" "" (at 69.342 40.64 90)
+      (effects (font (size 1.27 1.27)) hide)
+    )
+    (property "Datasheet" "~" (at 71.12 40.64 0)
+      (effects (font (size 1.27 1.27)) hide)
+    )
+    (pin "1")
+    (pin "2")
+    (instances
+      (project "Flight Computer"
+        (path "/0c1188a1-706b-46cd-a73a-5b3f8187d77a/8b5c3409-c69f-490d-a71d-45a34969a1f1"
+          (reference "R4") (unit 1)
+        )
+      )
+    )
   )
 )

Commit message: Schematics are love. Also I have no idea what I was doing last night so the power supply might be terrible, but I know I thought it was brilliant at the time
Parts:
- added Q3, Q5, Q6, Q7, Q8: AO3400A, Package_TO_SOT_SMD:SOT-23, symbol Transistor_FET:AO3400A
- added R10, R12, R14, R16, R8: 22k, symbol Device:R
- added R11, R13, R15, R7, R9: 220k, symbol Device:R
Connections:
- net GND: now also Q3.2 (S), Q5.2 (S), Q6.2 (S), Q7.2 (S), Q8.2 (S), R10.2, R12.2, R14.2, R16.2, R8.2
- new net Pyro Channel B: Q3.3 (D), R7.1
- new net Pyro Channel B Continuity Voltage: R7.2, R8.1
- new net Pyro Channel B Trigger: Q3.1 (G)
- new net Pyro Channel C: Q5.3 (D), R9.1
- new net Pyro Channel C Continuity Voltage: R10.1, R9.2
- new net Pyro Channel C Trigger: Q5.1 (G)
- new net Pyro Channel D: Q8.3 (D), R15.1
- new net Pyro Channel D Continuity Voltage: R15.2, R16.1
- new net Pyro Channel D Trigger: Q8.1 (G)
- new net Pyro Channel E: Q6.3 (D), R11.1
- new net Pyro Channel E Continuity Voltage: R11.2, R12.1
- new net Pyro Channel E Trigger: Q6.1 (G)
- new net Pyro Channel F: Q7.3 (D), R13.1
- new net Pyro Channel F Continuity Voltage: R13.2, R14.1
- new net Pyro Channel F Trigger: Q7.1 (G)

Commit message: Chose footprints for most components
Parts:
- R10, R11, R12, R13, R14, R15, R16, R4, R6, R7, R8, R9: footprint (none) -> Resistor_SMD:R_0402_1005Metric
Changed lines of the file:
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@@
       (effects (font (size 1.27 1.27)) (justify left))
     )
-    (property "Footprint" "" (at 201.422 97.79 90)
+    (property "Footprint" "Resistor_SMD:R_0402_1005Metric" (at 201.422 97.79 90)
       (effects (font (size 1.27 1.27)) hide)
     )
@@
       (effects (font (size 1.27 1.27)) (justify left))
     )
-    (property "Footprint" "" (at 109.982 156.21 90)
+    (property "Footprint" "Resistor_SMD:R_0402_1005Metric" (at 109.982 156.21 90)
       (effects (font (size 1.27 1.27)) hide)
     )
@@
       (effects (font (size 1.27 1.27)) (justify left))
     )
-    (property "Footprint" "" (at 69.342 50.8 90)
+    (property "Footprint" "Resistor_SMD:R_0402_1005Metric" (at 69.342 50.8 90)
       (effects (font (size 1.27 1.27)) hide)
     )
@@
       (effects (font (size 1.27 1.27)) (justify left))
     )
-    (property "Footprint" "" (at 201.422 132.08 90)
+    (property "Footprint" "Resistor_SMD:R_0402_1005Metric" (at 201.422 132.08 90)
       (effects (font (size 1.27 1.27)) hide)
     )
@@
       (effects (font (size 1.27 1.27)) (justify left))
     )
-    (property "Footprint" "" (at 109.982 97.79 90)
+    (property "Footprint" "Resistor_SMD:R_0402_1005Metric" (at 109.982 97.79 90)
       (effects (font (size 1.27 1.27)) hide)
     )
@@
       (effects (font (size 1.27 1.27)) (justify left))
     )
-    (property "Footprint" "" (at 201.422 87.63 90)
+    (property "Footprint" "Resistor_SMD:R_0402_1005Metric" (at 201.422 87.63 90)
       (effects (font (size 1.27 1.27)) hide)
     )
@@
       (effects (font (size 1.27 1.27)) (justify left))
     )
-    (property "Footprint" "" (at 109.982 121.92 90)
+    (property "Footprint" "Resistor_SMD:R_0402_1005Metric" (at 109.982 121.92 90)
       (effects (font (size 1.27 1.27)) hide)
     )
@@
       (effects (font (size 1.27 1.27)) (justify left))
     )
-    (property "Footprint" "" (at 201.422 121.92 90)
+    (property "Footprint" "Resistor_SMD:R_0402_1005Metric" (at 201.422 121.92 90)
       (effects (font (size 1.27 1.27)) hide)
     )
@@
       (effects (font (size 1.27 1.27)) (justify left))
     )
-    (property "Footprint" "" (at 69.342 40.64 90)
+    (property "Footprint" "Resistor_SMD:R_0402_1005Metric" (at 69.342 40.64 90)
       (effects (font (size 1.27 1.27)) hide)
     )
@@
       (effects (font (size 1.27 1.27)) (justify left))
     )
-    (property "Footprint" "" (at 109.982 132.08 90)
+    (property "Footprint" "Resistor_SMD:R_0402_1005Metric" (at 109.982 132.08 90)
       (effects (font (size 1.27 1.27)) hide)
     )
@@
       (effects (font (size 1.27 1.27)) (justify left))
     )
-    (property "Footprint" "" (at 109.982 166.37 90)
+    (property "Footprint" "Resistor_SMD:R_0402_1005Metric" (at 109.982 166.37 90)
       (effects (font (size 1.27 1.27)) hide)
     )
@@
       (effects (font (size 1.27 1.27)) (justify left))
     )
-    (property "Footprint" "" (at 109.982 87.63 90)
-      (effects (font (size 1.27 1.27)) hide)
-    )
+    (property "Footprint" "Resistor_SMD:R_0402_1005Metric" (at 109.982 87.63 90)
+      (effects (font (size 1.27 1.27)) hide)
+    )

Commit message: Started footprint
Parts:
- R11, R13, R15, R4, R7, R9: value 220k -> 200k
Changed lines of the file:
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@@
       (effects (font (size 1.27 1.27)) (justify left))
     )
-    (property "Value" "220k" (at 113.03 157.48 0)
+    (property "Value" "200k" (at 113.03 157.48 0)
       (effects (font (size 1.27 1.27)) (justify left))
     )
@@
       (effects (font (size 1.27 1.27)) (justify left))
     )
-    (property "Value" "220k" (at 204.47 88.9 0)
+    (property "Value" "200k" (at 204.47 88.9 0)
       (effects (font (size 1.27 1.27)) (justify left))
     )
@@
       (effects (font (size 1.27 1.27)) (justify left))
     )
-    (property "Value" "220k" (at 113.03 123.19 0)
+    (property "Value" "200k" (at 113.03 123.19 0)
       (effects (font (size 1.27 1.27)) (justify left))
     )
@@
       (effects (font (size 1.27 1.27)) (justify left))
     )
-    (property "Value" "220k" (at 204.47 123.19 0)
+    (property "Value" "200k" (at 204.47 123.19 0)
       (effects (font (size 1.27 1.27)) (justify left))
     )
@@
       (effects (font (size 1.27 1.27)) (justify left))
     )
-    (property "Value" "220k" (at 72.39 41.91 0)
+    (property "Value" "200k" (at 72.39 41.91 0)
       (effects (font (size 1.27 1.27)) (justify left))
     )
@@
       (effects (font (size 1.27 1.27)) (justify left))
     )
-    (property "Value" "220k" (at 113.03 88.9 0)
-      (effects (font (size 1.27 1.27)) (justify left))
-    )
+    (property "Value" "200k" (at 113.03 88.9 0)
+      (effects (font (size 1.27 1.27)) (justify left))
+    )

Commit message: How many sheets do you want? Yes
Parts:
- added J2: Pyro Channels, custom-footprints:Wago_Custom_218-108, symbol Connector_Generic:Conn_02x08_Odd_Even
- added J3: Screw Switches, custom-footprints:Wago_Custom_218-108, symbol Connector_Generic:Conn_02x08_Odd_Even
- added R17: 200k, Resistor_SMD:R_0402_1005Metric, symbol Device:R
- added R18: 22k, Resistor_SMD:R_0402_1005Metric, symbol Device:R
Connections:
- net GND: now also J3.15 (Pin_15), J3.16 (Pin_16), R18.2
- net Pyro Channel A: now also J2.3 (Pin_3), J2.4 (Pin_4)
- net Pyro Channel B: now also J2.7 (Pin_7), J2.8 (Pin_8)
- net Pyro Channel C: now also J2.11 (Pin_11), J2.12 (Pin_12)
- net Pyro Channel D: now also J2.15 (Pin_15), J2.16 (Pin_16)
- net Pyro Channel E: now also J3.1 (Pin_1), J3.2 (Pin_2)
- net Pyro Channel F: now also J3.5 (Pin_5), J3.6 (Pin_6)
- new net +12V: J2.1 (Pin_1), J2.10 (Pin_10), J2.13 (Pin_13), J2.14 (Pin_14), J2.2 (Pin_2), J2.5 (Pin_5), J2.6 (Pin_6), J2.9 (Pin_9), J3.13 (Pin_13), J3.14 (Pin_14), J3.3 (Pin_3), J3.4 (Pin_4), J3.7 (Pin_7), J3.8 (Pin_8), R17.1
- new net Ignition Battery Voltage: R17.2, R18.1
- new net Main battery connector: J3.10 (Pin_10), J3.9 (Pin_9)
- new net Main battery in: J3.11 (Pin_11), J3.12 (Pin_12)
Other:
- note added: "Pyro Channels A-D"
- note added: "Pyro Channels E, F, and Screw Switches"
- note added: "This connects to an ADC on the MCU, allowing it to monitor the voltage of the ignition battery"
- moved on the sheet: Q3, Q5, Q6, Q7, Q8, R10, R11, R12, R13, R14, R15, R16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

Commit message: Finished updating the schematics
Other:
- moved on the sheet: Q3, Q5, Q6, Q7, Q8, R10, R11, R12, R13, R14, R15, R16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

Commit message: Started doing layout for v1.1
Parts:
- added D10, D11, D12, D13, D14, D9: B5819W SL, Diode_SMD:D_SOD-123, symbol Device:D_Schottky
- added D3, D4, D5, D6, D7, D8: LED, LED_SMD:LED_0603_1608Metric_Pad1.05x0.95mm_HandSolder, symbol Device:LED
- added R29, R30, R31, R32, R33, R34: 22k, Resistor_SMD:R_0402_1005Metric, symbol Device:R
- added R36, R37, R38, R39, R40, R41: 1.5k, Resistor_SMD:R_0402_1005Metric, symbol Device:R
Connections:
- net GND: now also D10.2 (A), D11.2 (A), D12.2 (A), D13.2 (A), D14.2 (A), D3.1 (K), D4.1 (K), D5.1 (K), D6.1 (K), D7.1 (K), D8.1 (K), D9.2 (A), R29.2, R30.2, R31.2, R32.2, R33.2, R34.2
- net Pyro Channel A: now also D9.1 (K)
- net Pyro Channel A Trigger: now also R34.1, R36.1
- net Pyro Channel B: now also D10.1 (K)
- net Pyro Channel B Trigger: now also R29.1, R40.1
- net Pyro Channel C: now also D14.1 (K)
- net Pyro Channel C Trigger: now also R33.1, R41.1
- net Pyro Channel D: now also D13.1 (K)
- net Pyro Channel D Trigger: now also R32.1, R39.1
- net Pyro Channel E: now also D11.1 (K)
- net Pyro Channel E Trigger: now also R30.1, R37.1
- net Pyro Channel F: now also D12.1 (K)
- net Pyro Channel F Trigger: now also R31.1, R38.1
- new net: D5.2 (A), R38.2
- new net: D7.2 (A), R40.2
- new net: D3.2 (A), R36.2
- new net: D8.2 (A), R41.2
- new net: D6.2 (A), R39.2
- new net: D4.2 (A), R37.2
Other:
- note added: "One of the charge's leads connects to this, the other to the positive ignition battery voltage. To trigger, this input is shorted to ground."
- note removed: "This is the actual Pyro Channel. One of the charge's leads connects to this, the other to the positive ignition battery voltage. To trigger, this input is shorted to ground."
- moved on the sheet: J2, J3, Q2, Q3, Q5, Q6, Q7, Q8, R10, R11, R12, R13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
