File: pyro-channels.kicad_sch (KiCad schematic)
At the start: 46 parts, among them J2 Pyro Channels, J3 Screw Switches, Q2 AO3400A, Q3 AO3400A, Q5 AO3400A, Q6 AO3400A, Q7 AO3400A, Q8 AO3400A

Commit message: How many test points do you want? Yes.
Other:
- moved on the sheet: D9
Changed lines of the file:
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@@
     (stroke (width 0) (type default))
   )
-  (wire (pts (xy 73.66 21.59) (xy 78.74 21.59))
+  (wire (pts (xy 73.66 20.32) (xy 78.74 20.32))
     (stroke (width 0) (type default))
   )
@@
     (stroke (width 0) (type default))
   )
-  (wire (pts (xy 60.96 21.59) (xy 60.96 31.75))
+  (wire (pts (xy 60.96 20.32) (xy 60.96 31.75))
     (stroke (width 0) (type default))
   )
@@
     (stroke (width 0) (type default))
   )
-  (wire (pts (xy 66.04 21.59) (xy 60.96 21.59))
+  (wire (pts (xy 66.04 20.32) (xy 60.96 20.32))
     (stroke (width 0) (type default))
   )
@@
     (stroke (width 0) (type default))
   )
-  (wire (pts (xy 78.74 21.59) (xy 78.74 31.75))
+  (wire (pts (xy 78.74 20.32) (xy 78.74 31.75))
     (stroke (width 0) (type default))
   )
@@
     )
   )
-  (symbol (lib_id "Device:D_Schottky") (at 69.85 21.59 0) (unit 1)
-    (in_bom yes) (on_board yes) (dnp no) (fields_autoplaced)
-    (property "Reference" "D9" (at 69.5325 16.51 0)
+  (symbol (lib_id "Device:D_Schottky") (at 69.85 20.32 0) (unit 1)
+    (in_bom yes) (on_board yes) (dnp no)
+    (property "Reference" "D9" (at 69.5325 15.24 0)
       (effects (font (size 1.27 1.27)))
     )
-    (property "Value" "B5819W SL" (at 69.5325 19.05 0)
+    (property "Value" "B5819W SL" (at 69.5325 17.78 0)
       (effects (font (size 1.27 1.27)))
     )
-    (property "Footprint" "Diode_SMD:D_SOD-123" (at 69.85 21.59 0)
-      (effects (font (size 1.27 1.27)) hide)
-    )
-    (property "Datasheet" "~" (at 69.85 21.59 0)
-      (effects (font (size 1.27 1.27)) hide)
-    )
+    (property "Footprint" "Diode_SMD:D_SOD-123" (at 69.85 20.32 0)
+      (effects (font (size 1.27 1.27)) hide)
+    )
+    (property "Datasheet" "~" (at 69.85 20.32 0)
+      (effects (font (size 1.27 1.27)) hide)
+    )

Commit message: Now with 100% fewer faulty flyback diodes
Parts:
- removed D10, D11, D12, D13, D14, D9: B5819W SL, Diode_SMD:D_SOD-123, symbol Device:D_Schottky
