File: pyro-channels.kicad_sch (KiCad schematic)
At the start: 40 parts, among them J2 Pyro Channels, J3 Screw Switches, Q2 AO3400A, Q3 AO3400A, Q5 AO3400A, Q6 AO3400A, Q7 AO3400A, Q8 AO3400A

Commit message: Updated with notes from Erik Welsh
Parts:
- R36, R37, R38, R39, R40, R41: value 1.5k -> 1k
Other:
- note added: "This is where the +12V ignition line is connected to the battery through a screw switch"
- note added: "This physically disconnects main battery from the board for screw-switching"
- moved on the sheet: J2, J3, R17, R18

Commit message: Finished final(tm) updates for v1.1
Parts:
- added D10, D11, D12, D13, D14, D9: White, LED_SMD:LED_0603_1608Metric, symbol Device:LED
- added R47, R56, R57, R58, R59, R60: 1k, Resistor_SMD:R_0402_1005Metric, symbol Device:R
- D3: value LED -> Red
- D4, D5, D6, D7, D8: value White -> Red
Connections:
- net GND: now also D10.1 (K), D11.1 (K), D12.1 (K), D13.1 (K), D14.1 (K), D9.1 (K)
- new net: D9.2 (A), R47.2
- new net: D12.2 (A), R58.2
- new net: D13.2 (A), R59.2
- new net: D14.2 (A), R60.2
- new net: D10.2 (A), R56.2
- new net: D11.2 (A), R57.2
- new net Channel A Continuity LED: R47.1
- new net Channel B Continuity LED: R56.1
- new net Channel C Continuity LED: R57.1
- new net Channel D Continuity LED: R58.1
- new net Channel E Continuity LED: R59.1
- new net Channel F Continuity LED: R60.1
Other:
- note added: "Continuity Indication LEDs"
- moved on the sheet: D5, D6, D7, D8, J3, Q3, Q5, Q7, Q8, R10, R13, R14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

Commit message: Finished layout with modified pyro terminal blocks
Parts:
- J2, J3: footprint custom-footprints:Wago_Custom_218-108 -> custom-footprints:Wago_Custom_2601-1108
Changed lines of the file:
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@@
       (effects (font (size 1.27 1.27)))
     )
-    (property "Footprint" "custom-footprints:Wago_Custom_218-108" (at 66.04 111.76 0)
+    (property "Footprint" "custom-footprints:Wago_Custom_2601-1108" (at 66.04 111.76 0)
       (effects (font (size 1.27 1.27)) hide)
     )
@@
       (effects (font (size 1.27 1.27)))
     )
-    (property "Footprint" "custom-footprints:Wago_Custom_218-108" (at 54.61 158.75 0)
+    (property "Footprint" "custom-footprints:Wago_Custom_2601-1108" (at 54.61 158.75 0)
       (effects (font (size 1.27 1.27)) hide)
     )

Commit message: Added different 3d models for terminal blocks
Parts:
- J2, J3: footprint custom-footprints:Wago_Custom_2601-1108 -> custom-footprints:Pheonix-Contact-1861991
Changed lines of the file:
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@@
       (effects (font (size 1.27 1.27)))
     )
-    (property "Footprint" "custom-footprints:Wago_Custom_2601-1108" (at 66.04 111.76 0)
+    (property "Footprint" "custom-footprints:Pheonix-Contact-1861991" (at 66.04 111.76 0)
       (effects (font (size 1.27 1.27)) hide)
     )
@@
       (effects (font (size 1.27 1.27)))
     )
-    (property "Footprint" "custom-footprints:Wago_Custom_2601-1108" (at 54.61 158.75 0)
+    (property "Footprint" "custom-footprints:Pheonix-Contact-1861991" (at 54.61 158.75 0)
       (effects (font (size 1.27 1.27)) hide)
     )
