File: microcontroller.kicad_sch (KiCad schematic)
At the start: 22 parts, among them Q1 MMBT2222A, U6 STM32L476VETx, Y1 16MHz

Commit message: Finished updating the schematics
Parts:
- added R26, R27: 4.7k, Resistor_SMD:R_0402_1005Metric, symbol Device:R
Connections:
- net +3.3V: now also R26.1, R27.1
- net Altimeter Interrupt: now also U6.2 (PE3); no longer U6.17 (PC2)
- net Chip Select Low G Accel: now also U6.96 (PB9); no longer U6.88 (PD7)
- net I2C2 SCL: now also R26.2
- net I2C2 SDA: now also R27.2
- net Low G Gyro Interrupt: now also U6.1 (PE2); no longer U6.93 (PB7)
- net Chip Select High G Accel: now reaches U6.95 (PB8)
- net SDMMC Clock renamed SDMMC Data Clock
- new net Chip Select Altimeter: U6.93 (PB7)
- no-connect marks 30 -> 28
Other:
- note added: "Pull-up resistors for external I2C buss, 4.7k"
- title: (none) -> STM32 Microcontroller and Supporting Circuitry
- moved on the sheet: BZ1, Q1, R30, R31

Commit message: Started doing layout for v1.1
Parts:
- D1: value Blue -> LED; footprint LED_SMD:LED_0805_2012Metric -> LED_SMD:LED_0603_1608Metric
Changed lines of the file:
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@@
       (effects (font (size 1.27 1.27)) (justify right))
     )
-    (property "Value" "Blue" (at 88.9 171.45 90)
+    (property "Value" "LED" (at 88.9 171.45 90)
       (effects (font (size 1.27 1.27)) (justify right))
     )
-    (property "Footprint" "LED_SMD:LED_0805_2012Metric" (at 85.09 168.91 0)
+    (property "Footprint" "LED_SMD:LED_0603_1608Metric" (at 85.09 168.91 0)
       (effects (font (size 1.27 1.27)) hide)
     )

Commit message: finished layout for v1.1
Parts:
- R3: footprint Resistor_SMD:R_0603_1608Metric -> Resistor_SMD:R_0402_1005Metric
Connections:
- net Altimeter Interrupt: now also U6.1 (PE2); no longer U6.2 (PE3)
- net Chip Select Altimeter: now also U6.2 (PE3); no longer U6.93 (PB7)
- net Chip Select High G Accel: now also U6.92 (PB6); no longer U6.95 (PB8)
- net Chip Select Low G Accel: now also U6.97 (PE0); no longer U6.96 (PB9)
- net Chip Select Low G Gyro: now also U6.95 (PB8); no longer U6.92 (PB6)
- net GPS External Interrupt: now also U6.84 (PD3); no longer U6.85 (PD4)
- net GPS Reset: now also U6.85 (PD4); no longer U6.84 (PD3)
- net High G Interrupt: now also U6.93 (PB7); no longer U6.98 (PE1)
- net Low G Accel Interrupt: now also U6.98 (PE1); no longer U6.97 (PE0)
- net Low G Gyro Interrupt: now also U6.96 (PB9); no longer U6.1 (PE2)
- net Pyro E Continuity Voltage: now also U6.30 (PA5); no longer U6.29 (PA4)
- net Pyro F Continuity Voltage: now also U6.29 (PA4); no longer U6.30 (PA5)
Changed lines of the file:
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@@
     (effects (font (size 1.27 1.27)) (justify right))
   )
-  (hierarchical_label "Altimeter Interrupt" (shape input) (at 90.17 91.44 180) (fields_autoplaced)
+  (hierarchical_label "Altimeter Interrupt" (shape input) (at 90.17 88.9 180) (fields_autoplaced)
     (effects (font (size 1.27 1.27)) (justify right))
   )
@@
     (effects (font (size 1.27 1.27)) (justify right))
   )
-  (hierarchical_label "GPS External Interrupt" (shape output) (at 78.74 137.16 180) (fields_autoplaced)
+  (hierarchical_label "GPS External Interrupt" (shape output) (at 78.74 134.62 180) (fields_autoplaced)
     (effects (font (size 1.27 1.27)) (justify right))
   )
@@
     (effects (font (size 1.27 1.27)) (justify right))
   )
-  (hierarchical_label "Chip Select Altimeter" (shape output) (at 158.75 119.38 0) (fields_autoplaced)
-    (effects (font (size 1.27 1.27)) (justify left))
+  (hierarchical_label "Chip Select Altimeter" (shape output) (at 90.17 91.44 180) (fields_autoplaced)
+    (effects (font (size 1.27 1.27)) (justify right))
   )
   (hierarchical_label "Pyro Channel A Trigger" (shape output) (at 165.1 106.68 0) (fields_autoplaced)
@@
     (effects (font (size 1.27 1.27)) (justify right))
   )
-  (hierarchical_label "GPS Reset" (shape output) (at 78.74 134.62 180) (fields_autoplaced)
+  (hierarchical_label "GPS Reset" (shape output) (at 78.74 137.16 180) (fields_autoplaced)
     (effects (font (size 1.27 1.27)) (justify right))
   )
@@
     (effects (font (size 1.27 1.27)) (justify left))
   )
-  (hierarchical_label "Pyro F Continuity Voltage" (shape input) (at 144.78 71.12 0) (fields_autoplaced)
+  (hierarchical_label "Pyro F Continuity Voltage" (shape input) (at 144.78 68.58 0) (fields_autoplaced)
     (effects (font (size 1.27 1.27)) (justify left))
   )
@@
     (effects (font (size 1.27 1.27)) (justify left))
   )
-  (hierarchical_label "Chip Select High G Accel" (shape output) (at 158.75 121.92 0) (fields_autoplaced)
+  (hierarchical_label "Chip Select High G Accel" (shape output) (at 158.75 116.84 0) (fields_autoplaced)
     (effects (font (size 1.27 1.27)) (justify left))
   )
@@
     (effects (font (size 1.27 1.27)) (justify left))
   )
-  (hierarchical_label "Low G Gyro Interrupt" (shape input) (at 90.17 88.9 180) (fields_autoplaced)
-    (effects (font (size 1.27 1.27)) (justify right))
+  (hierarchical_label "Low G Gyro Interrupt" (shape input) (at 158.75 124.46 0) (fields_autoplaced)
+    (effects (font (size 1.27 1.27)) (justify left))
   )
   (hierarchical_label "QSPI IO3" (shape bidirectional) (at 151.13 73.66 0) (fields_autoplaced)
@@
     (effects (font (size 1.27 1.27)) (justify left))
   )
-  (hierarchical_label "Chip Select Low G Accel" (shape output) (at 158.75 124.46 0) (fields_autoplaced)
-    (effects (font (size 1.27 1.27)) (justify left))
+  (hierarchical_label "Chip Select Low G Accel" (shape output) (at 90.17 83.82 180) (fields_autoplaced)
+    (effects (font (size 1.27 1.27)) (justify right))
   )
   (hierarchical_label "Pyro Channel F Trigger" (shape output) (at 87.63 114.3 180) (fields_autoplaced)
@@
     (effects (font (size 1.27 1.27)) (justify left))
   )
-  (hierarchical_label "Low G Accel Interrupt" (shape input) (at 90.17 83.82 180) (fields_autoplaced)
-    (effects (font (size 1.27 1.27)) (justify right))
-  )
-  (hierarchical_label "Chip Select Low G Gyro" (shape output) (at 158.75 116.84 0) (fields_autoplaced)
-    (effects (font (size 1.27 1.27)) (justify left))
-  )
-  (hierarchical_label "High G Interrupt" (shape input) (at 90.17 86.36 180) (fields_autoplaced)
-    (effects (font (size 1.27 1.27)) (justify right))
+  (hierarchical_label "Low G Accel Interrupt" (shape input) (at 90.17 86.36 180) (fields_autoplaced)
+    (effects (font (size 1.27 1.27)) (justify right))
+  )
+  (hierarchical_label "Chip Select Low G Gyro" (shape output) (at 158.75 121.92 0) (fields_autoplaced)
+    (effects (font (size 1.27 1.27)) (justify left))
+  )
+  (hierarchical_label "High G Interrupt" (shape input) (at 158.75 119.38 0) (fields_autoplaced)
+    (effects (font (size 1.27 1.27)) (justify left))
   )
   (hierarchical_label "Pyro A Continuity Voltage" (shape input) (at 144.78 58.42 0) (fields_autoplaced)
@@
     (effects (font (size 1.27 1.27)) (justify left))
   )
-  (hierarchical_label "Pyro E Continuity Voltage" (shape input) (at 144.78 68.58 0) (fields_autoplaced)
+  (hierarchical_label "Pyro E Continuity Voltage" (shape input) (at 144.78 71.12 0) (fields_autoplaced)
     (effects (font (size 1.27 1.27)) (justify left))
   )
@@
       (effects (font (size 1.27 1.27)) (justify left))
     )
-    (property "Footprint" "Resistor_SMD:R_0603_1608Metric" (at 83.312 177.8 90)
-      (effects (font (size 1.27 1.27)) hide)
-    )
+    (property "Footprint" "Resistor_SMD:R_0402_1005Metric" (at 83.312 177.8 90)
+      (effects (font (size 1.27 1.27)) hide)
+    )
