File: microcontroller.kicad_sch (KiCad schematic)
At the start: 24 parts, among them Q1 MMBT2222A, U6 STM32L476VETx, Y1 16MHz

Commit message: Updated with notes from Erik Welsh
Parts:
- added R45: 51k, Resistor_SMD:R_0402_1005Metric, symbol Device:R
- added R46: 200k, Resistor_SMD:R_0402_1005Metric, symbol Device:R
- R3: value 1.5k -> 1k
Connections:
- net GND: now also R46.2
- net USB 5V in: now also R45.1; no longer U6.68 (PA9)
- new net: R45.2, R46.1, U6.68 (PA9)
Other:
- note added: "PA9 is 5V tolerant, which means the voltage cannot exceed VDD + 4 Volts. Thus, during a transient power on state, we need to lower this voltage with a voltage divider to between 3 and 4 volts"
- note added: "PA9 must be > 0.7 * Vdd to be detected"
Changed lines of the file:
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@@
   (junction (at 71.12 33.02) (diameter 0) (color 0 0 0 0)
+  )
+  (junction (at 182.88 81.28) (diameter 0) (color 0 0 0 0)
   )
   (junction (at 41.91 158.75) (diameter 0) (color 0 0 0 0)
@@
   (no_connect (at 96.52 93.98))
   (no_connect (at 142.24 144.78))
+  (no_connect (at 142.24 83.82))
   (no_connect (at 142.24 180.34))
   (no_connect (at 142.24 162.56))
@@
   (no_connect (at 96.52 157.48))
   (no_connect (at 142.24 157.48))
-  (no_connect (at 142.24 83.82))
   (no_connect (at 96.52 96.52))
   (no_connect (at 96.52 144.78))
@@
     (stroke (width 0) (type default))
   )
+  (wire (pts (xy 182.88 91.44) (xy 182.88 92.71))
+    (stroke (width 0) (type default))
+  )
   (wire (pts (xy 142.24 111.76) (xy 146.05 111.76))
     (stroke (width 0) (type default))
@@
     (stroke (width 0) (type default))
   )
+  (wire (pts (xy 185.42 67.31) (xy 182.88 67.31))
+    (stroke (width 0) (type default))
+  )
   (wire (pts (xy 71.12 25.4) (xy 81.28 25.4))
     (stroke (width 0) (type default))
@@
     (stroke (width 0) (type default))
   )
+  (wire (pts (xy 142.24 81.28) (xy 182.88 81.28))
+    (stroke (width 0) (type default))
+  )
   (wire (pts (xy 44.45 87.63) (xy 44.45 85.09))
     (stroke (width 0) (type default))
@@
     (stroke (width 0) (type default))
   )
+  (wire (pts (xy 182.88 81.28) (xy 182.88 83.82))
+    (stroke (width 0) (type default))
+  )
   (wire (pts (xy 142.24 129.54) (xy 161.29 129.54))
     (stroke (width 0) (type default))
@@
     (stroke (width 0) (type default))
   )
+  (wire (pts (xy 182.88 67.31) (xy 182.88 71.12))
+    (stroke (width 0) (type default))
+  )
   (wire (pts (xy 82.55 63.5) (xy 80.01 63.5))
     (stroke (width 0) (type default))
@@
     (stroke (width 0) (type default))
   )
+  (wire (pts (xy 182.88 78.74) (xy 182.88 81.28))
+    (stroke (width 0) (type default))
+  )
   (wire (pts (xy 44.45 85.09) (xy 39.37 85.09))
     (stroke (width 0) (type default))
@@
     (stroke (width 0) (type default))
   )
-  (wire (pts (xy 142.24 81.28) (xy 146.05 81.28))
-    (stroke (width 0) (type default))
-  )
   (wire (pts (xy 142.24 116.84) (xy 158.75 116.84))
     (stroke (width 0) (type default))
@@
   (wire (pts (xy 58.42 165.1) (xy 82.55 165.1))
     (stroke (width 0) (type default))
+  )
+  (text "PA9 must be > 0.7 * Vdd to be detected" (at 205.74 85.09 0)
+    (effects (font (size 1.27 1.27)) (justify left bottom))
   )
   (text "Pull-up resistors for external I2C buss, 4.7k" (at 204.47 142.24 0)
@@
     (effects (font (size 2 2) (thickness 0.4) bold) (justify left bottom))
   )
+  (text "PA9 is 5V tolerant, which means the voltage cannot exceed VDD + 4 Volts.\nThus, during a transient power on state, we need to lower this voltage\nwith a voltage divider to between 3 and 4 volts"
+    (at 205.74 78.74 0)
+    (effects (font (size 1.27 1.27)) (justify left bottom))
+  )
   (text "High Speed External Oscillator\n(16MHz) for STM32" (at 20.32 72.39 0)
     (effects (font (size 2 2) (thickness 0.4) bold) (justify left bottom))
@@
     (effects (font (size 1.27 1.27)) (justify left))
   )
-  (hierarchical_label "USB 5V in" (shape input) (at 146.05 81.28 0) (fields_autoplaced)
+  (hierarchical_label "USB 5V in" (shape input) (at 185.42 67.31 0) (fields_autoplaced)
     (effects (font (size 1.27 1.27)) (justify left))
   )
@@
     )
   )
+  (symbol (lib_id "Device:R") (at 182.88 74.93 0) (unit 1)
+    (in_bom yes) (on_board yes) (dnp no)
+    (property "Reference" "R45" (at 184.15 73.66 0)
+      (effects (font (size 1.27 1.27)) (justify left))
+    )
+    (property "Value" "51k" (at 184.15 76.2 0)
+      (effects (font (size 1.27 1.27)) (justify left))
+    )
+    (property "Footprint" "Resistor_SMD:R_0402_1005Metric" (at 181.102 74.93 90)
+      (effects (font (size 1.27 1.27)) hide)
+    )
+    (property "Datasheet" "~" (at 182.88 74.93 0)
+      (effects (font (size 1.27 1.27)) hide)
+    )
+    (pin "1")
+    (pin "2")
+    (instances
+      (project "Flight Computer"
+        (path "/0c1188a1-706b-46cd-a73a-5b3f8187d77a/1c711583-e10e-42d1-9de8-3f5bf7fe676f"
+          (reference "R45") (unit 1)
+        )
+      )
+    )
+  )
   (symbol (lib_id "Device:C") (at 54.61 101.6 0) (unit 1)
     (in_bom yes) (on_board yes) (dnp no)
@@
     )
   )
+  (symbol (lib_id "Device:R") (at 182.88 87.63 0) (unit 1)
+    (in_bom yes) (on_board yes) (dnp no)
+    (property "Reference" "R46" (at 184.15 86.36 0)
+      (effects (font (size 1.27 1.27)) (justify left))
+    )
+    (property "Value" "200k" (at 184.15 88.9 0)
+      (effects (font (size 1.27 1.27)) (justify left))
+    )
+    (property "Footprint" "Resistor_SMD:R_0402_1005Metric" (at 181.102 87.63 90)
+      (effects (font (size 1.27 1.27)) hide)
+    )
+    (property "Datasheet" "~" (at 182.88 87.63 0)
+      (effects (font (size 1.27 1.27)) hide)
+    )
+    (pin "1")
+    (pin "2")
+    (instances
+      (project "Flight Computer"
+        (path "/0c1188a1-706b-46cd-a73a-5b3f8187d77a/1c711583-e10e-42d1-9de8-3f5bf7fe676f"
+          (reference "R46") (unit 1)
+        )
+      )
+    )
+  )
   (symbol (lib_id "power:GND") (at 106.68 50.8 0) (mirror y) (unit 1)
     (in_bom yes) (on_board yes) (dnp no) (fields_autoplaced)
@@
         (path "/0c1188a1-706b-46cd-a73a-5b3f8187d77a/1c711583-e10e-42d1-9de8-3f5bf7fe676f"
           (reference "#PWR080") (unit 1)
+        )
+      )
+    )
+  )
+  (symbol (lib_id "power:GND") (at 182.88 92.71 0) (unit 1)
+    (in_bom yes) (on_board yes) (dnp no) (fields_autoplaced)
+    (property "Reference" "#PWR0112" (at 182.88 99.06 0)
+      (effects (font (size 1.27 1.27)) hide)
+    )
+    (property "Value" "GND" (at 182.88 97.79 0)
+      (effects (font (size 1.27 1.27)))
+    )
+    (property "Footprint" "" (at 182.88 92.71 0)
+      (effects (font (size 1.27 1.27)) hide)
+    )
+    (property "Datasheet" "" (at 182.88 92.71 0)
+      (effects (font (size 1.27 1.27)) hide)
+    )
+    (pin "1")
+    (instances
+      (project "Flight Computer"
+        (path "/0c1188a1-706b-46cd-a73a-5b3f8187d77a/1c711583-e10e-42d1-9de8-3f5bf7fe676f"
+          (reference "#PWR0112") (unit 1)
         )
       )
@@
       (effects (font (size 1.27 1.27)) (justify left))
     )
-    (property "Value" "1.5k" (at 87.63 179.705 0)
-      (effects (font (size 1.27 1.27)) (justify left))
-    )
+    (property "Value" "1k" (at 87.63 179.705 0)
+      (effects (font (size 1.27 1.27)) (justify left))
+    )

Commit message: Fabrication outputs
Parts:
- R45: value 51k -> 47k
Changed lines of the file:
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@@
       (effects (font (size 1.27 1.27)) (justify left))
     )
-    (property "Value" "51k" (at 184.15 76.2 0)
+    (property "Value" "47k" (at 184.15 76.2 0)
       (effects (font (size 1.27 1.27)) (justify left))
     )

Commit message: Updating with notes from Adam
Connections:
- net SPI2 MISO: now reaches U6.17 (PC2)
- net SPI2 MOSI: now reaches U6.18 (PC3)
- net SPI2 SCK: now reaches U6.52 (PB13)
- no-connect marks 28 -> 25
Changed lines of the file:
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@@
   (no_connect (at 96.52 165.1))
   (no_connect (at 142.24 177.8))
-  (no_connect (at 142.24 149.86))
   (no_connect (at 96.52 121.92))
   (no_connect (at 96.52 119.38))
@@
   (no_connect (at 96.52 99.06))
   (no_connect (at 142.24 182.88))
-  (no_connect (at 142.24 134.62))
-  (no_connect (at 142.24 152.4))
   (no_connect (at 96.52 152.4))
   (no_connect (at 96.52 157.48))
@@
     (stroke (width 0) (type default))
   )
+  (wire (pts (xy 142.24 149.86) (xy 148.59 149.86))
+    (stroke (width 0) (type default))
+  )
   (wire (pts (xy 142.24 106.68) (xy 165.1 106.68))
     (stroke (width 0) (type default))
@@
     (stroke (width 0) (type default))
   )
+  (wire (pts (xy 142.24 134.62) (xy 148.59 134.62))
+    (stroke (width 0) (type default))
+  )
   (wire (pts (xy 212.09 48.26) (xy 220.98 48.26))
     (stroke (width 0) (type default))
@@
   )
   (wire (pts (xy 127 45.72) (xy 127 50.8))
+    (stroke (width 0) (type default))
+  )
+  (wire (pts (xy 142.24 152.4) (xy 148.59 152.4))
     (stroke (width 0) (type default))
   )
@@
     (effects (font (size 1.27 1.27)) (justify left))
   )
+  (hierarchical_label "SPI2 MISO" (shape input) (at 148.59 149.86 0) (fields_autoplaced)
+    (effects (font (size 1.27 1.27)) (justify left))
+  )
+  (hierarchical_label "SPI2 MOSI" (shape output) (at 148.59 152.4 0) (fields_autoplaced)
+    (effects (font (size 1.27 1.27)) (justify left))
+  )
   (hierarchical_label "UART3 RX" (shape input) (at 91.44 149.86 180) (fields_autoplaced)
     (effects (font (size 1.27 1.27)) (justify right))
@@
     (effects (font (size 1.27 1.27)) (justify right))
   )
+  (hierarchical_label "SPI2 SCK" (shape output) (at 148.59 134.62 0) (fields_autoplaced)
+    (effects (font (size 1.27 1.27)) (justify left))
+  )
   (hierarchical_label "SDMMC Data 3" (shape bidirectional) (at 147.32 172.72 0) (fields_autoplaced)

Commit message: Finished final(tm) updates for v1.1
Connections:
- net at U6.51 (PB12): now also R30.1
- net Channel D Continuity LED: now reaches U6.53 (PB14)
- net Channel C Continuity LED: now reaches U6.54 (PB15)
- net Channel B Continuity LED: now reaches U6.57 (PD10)
- net Channel A Continuity LED: now reaches U6.58 (PD11)
- net Channel E Continuity LED: now reaches U6.59 (PD12)
- net Channel F Continuity LED: now reaches U6.60 (PD13)
- net Channel F Continuity LED: no longer R30.1
- no-connect marks 25 -> 19
Other:
- note added: "Buzzer"
- note added: "Status LED"
- note removed: "Feedback Buzzer and Status LED"
- moved on the sheet: BZ1, Q1, R26, R27, R30, R31

Commit message: Added new buck converter
Parts:
- R46: value 200k -> 100k
Connections:
- net +5V is gone; now on net +3.3V: BZ1.1 (-), R31.1
- net at U6.46 (PE15): now also R30.1
- net at U6.51 (PB12): no longer R30.1
Other:
- moved on the sheet: BZ1, Q1, R30, R31

Commit message: Swapped out sensors in schematic for v3
Connections:
- net Magnetometer Chip Select: now reaches U6.15 (PC0)
- net Magnetometer Interrupt: now reaches U6.16 (PC1)
- net High G Accel Chip Select: now reaches U6.8 (PC14)
- net High G Accel Interrupt: now reaches U6.9 (PC15)
- net Chip Select High G Accel: no longer names the net of U6.92 (PB6)
- net High G Interrupt: no longer names the net of U6.93 (PB7)
- net SD Card Detect: no longer names the net of U6.81 (PD0)
- net SDMMC Command: no longer names the net of U6.83 (PD2)
- net SDMMC Data 0: no longer names the net of U6.65 (PC8)
- net SDMMC Data 1: no longer names the net of U6.66 (PC9)
- net SDMMC Data 2: no longer names the net of U6.78 (PC10)
- net SDMMC Data 3: no longer names the net of U6.79 (PC11)
- net SDMMC Data Clock: no longer names the net of U6.80 (PC12)
- no-connect marks 19 -> 24
Changed lines of the file:
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@@
   )
   (no_connect (at 96.52 93.98))
-  (no_connect (at 142.24 144.78))
+  (no_connect (at 142.24 172.72))
   (no_connect (at 142.24 83.82))
-  (no_connect (at 142.24 180.34))
+  (no_connect (at 142.24 119.38))
   (no_connect (at 142.24 132.08))
+  (no_connect (at 142.24 167.64))
   (no_connect (at 142.24 162.56))
   (no_connect (at 96.52 165.1))
@@
   (no_connect (at 142.24 78.74))
   (no_connect (at 142.24 96.52))
+  (no_connect (at 142.24 116.84))
   (no_connect (at 96.52 99.06))
-  (no_connect (at 142.24 182.88))
+  (no_connect (at 142.24 170.18))
   (no_connect (at 142.24 157.48))
   (no_connect (at 96.52 96.52))
   (no_connect (at 96.52 144.78))
   (no_connect (at 96.52 129.54))
+  (no_connect (at 96.52 132.08))
+  (no_connect (at 96.52 127))
+  (no_connect (at 142.24 165.1))
   (no_connect (at 142.24 160.02))
-  (no_connect (at 142.24 147.32))
+  (no_connect (at 142.24 175.26))
   (wire (pts (xy 111.76 41.91) (xy 106.68 41.91))
     (stroke (width 0) (type default))
@@
     (stroke (width 0) (type default))
   )
+  (wire (pts (xy 142.24 144.78) (xy 149.86 144.78))
+    (stroke (width 0) (type default))
+  )
   (wire (pts (xy 224.79 48.26) (xy 231.14 48.26))
     (stroke (width 0) (type default))
@@
     (stroke (width 0) (type default))
   )
-  (wire (pts (xy 142.24 119.38) (xy 158.75 119.38))
-    (stroke (width 0) (type default))
-  )
   (wire (pts (xy 92.71 41.91) (xy 92.71 43.18))
     (stroke (width 0) (type default))
@@
     (stroke (width 0) (type default))
   )
+  (wire (pts (xy 142.24 147.32) (xy 149.86 147.32))
+    (stroke (width 0) (type default))
+  )
   (wire (pts (xy 142.24 109.22) (xy 146.05 109.22))
     (stroke (width 0) (type default))
@@
     (stroke (width 0) (type default))
   )
+  (wire (pts (xy 142.24 180.34) (xy 149.86 180.34))
+    (stroke (width 0) (type default))
+  )
   (wire (pts (xy 231.14 48.26) (xy 236.22 48.26))
     (stroke (width 0) (type default))
@@
     (stroke (width 0) (type default))
   )
-  (wire (pts (xy 91.44 132.08) (xy 96.52 132.08))
-    (stroke (width 0) (type default))
-  )
   (wire (pts (xy 85.09 172.72) (xy 85.09 173.99))
     (stroke (width 0) (type default))
@@
     (stroke (width 0) (type default))
   )
-  (wire (pts (xy 142.24 167.64) (xy 147.32 167.64))
-    (stroke (width 0) (type default))
-  )
   (wire (pts (xy 90.17 88.9) (xy 96.52 88.9))
     (stroke (width 0) (type default))
@@
     (stroke (width 0) (type default))
   )
-  (wire (pts (xy 91.44 127) (xy 96.52 127))
-    (stroke (width 0) (type default))
-  )
   (wire (pts (xy 44.45 97.79) (xy 44.45 99.06))
     (stroke (width 0) (type default))
@@
     (stroke (width 0) (type default))
   )
-  (wire (pts (xy 142.24 170.18) (xy 147.32 170.18))
+  (wire (pts (xy 142.24 182.88) (xy 149.86 182.88))
     (stroke (width 0) (type default))
   )
@@
     (stroke (width 0) (type default))
   )
-  (wire (pts (xy 142.24 172.72) (xy 147.32 172.72))
-    (stroke (width 0) (type default))
-  )
   (wire (pts (xy 36.83 129.54) (xy 34.29 129.54))
     (stroke (width 0) (type default))
@@
     (stroke (width 0) (type default))
   )
-  (wire (pts (xy 142.24 116.84) (xy 158.75 116.84))
-    (stroke (width 0) (type default))
-  )
   (wire (pts (xy 142.24 88.9) (xy 157.48 88.9))
     (stroke (width 0) (type default))
@@
     (stroke (width 0) (type default))
   )
-  (wire (pts (xy 142.24 165.1) (xy 147.32 165.1))
-    (stroke (width 0) (type default))
-  )
   (wire (pts (xy 96.52 160.02) (xy 82.55 160.02))
     (stroke (width 0) (type default))
   )
   (wire (pts (xy 40.64 92.71) (xy 33.02 92.71))
-    (stroke (width 0) (type default))
-  )
-  (wire (pts (xy 142.24 175.26) (xy 147.32 175.26))
     (stroke (width 0) (type default))
   )
@@
     (effects (font (size 1.27 1.27)) (justify right))
   )
+  (hierarchical_label "Magnetometer Chip Select" (shape output) (at 149.86 144.78 0) (fields_autoplaced)
+    (effects (font (size 1.27 1.27)) (justify left))
+  )
   (hierarchical_label "UART2 TX" (shape output) (at 91.44 139.7 180) (fields_autoplaced)
     (effects (font (size 1.27 1.27)) (justify right))
@@
     (effects (font (size 1.27 1.27)) (justify right))
   )
-  (hierarchical_label "SDMMC Data Clock" (shape output) (at 147.32 175.26 0) (fields_autoplaced)
-    (effects (font (size 1.27 1.27)) (justify left))
-  )
   (hierarchical_label "Pyro Channel B Trigger" (shape output) (at 87.63 101.6 180) (fields_autoplaced)
     (effects (font (size 1.27 1.27)) (justify right))
@@
     (effects (font (size 1.27 1.27)) (justify left))
   )
-  (hierarchical_label "SDMMC Command" (shape output) (at 91.44 132.08 180) (fields_autoplaced)
-    (effects (font (size 1.27 1.27)) (justify right))
-  )
   (hierarchical_label "I2C2 SDA" (shape bidirectional) (at 161.29 129.54 0) (fields_autoplaced)
     (effects (font (size 1.27 1.27)) (justify left))
@@
     (effects (font (size 1.27 1.27)) (justify right))
   )
-  (hierarchical_label "SD Card Detect" (shape input) (at 91.44 127 180) (fields_autoplaced)
-    (effects (font (size 1.27 1.27)) (justify right))
-  )
   (hierarchical_label "Chip Select Altimeter" (shape output) (at 90.17 91.44 180) (fields_autoplaced)
     (effects (font (size 1.27 1.27)) (justify right))
@@
     (effects (font (size 1.27 1.27)) (justify left))
   )
-  (hierarchical_label "SDMMC Data 1" (shape bidirectional) (at 147.32 167.64 0) (fields_autoplaced)
-    (effects (font (size 1.27 1.27)) (justify left))
-  )
   (hierarchical_label "Channel D Continuity LED" (shape output) (at 156.21 137.16 0) (fields_autoplaced)
     (effects (font (size 1.27 1.27)) (justify left))
@@
     (effects (font (size 1.27 1.27)) (justify left))
   )
+  (hierarchical_label "High G Accel Interrupt" (shape input) (at 149.86 182.88 0) (fields_autoplaced)
+    (effects (font (size 1.27 1.27)) (justify left))
+  )
   (hierarchical_label "SPI2 MOSI" (shape output) (at 148.59 152.4 0) (fields_autoplaced)
     (effects (font (size 1.27 1.27)) (justify left))
@@
     (effects (font (size 1.27 1.27)) (justify left))
   )
-  (hierarchical_label "SDMMC Data 0" (shape bidirectional) (at 147.32 165.1 0) (fields_autoplaced)
-    (effects (font (size 1.27 1.27)) (justify left))
-  )
   (hierarchical_label "QSPI IO2" (shape bidirectional) (at 151.13 76.2 0) (fields_autoplaced)
     (effects (font (size 1.27 1.27)) (justify left))
@@
     (effects (font (size 1.27 1.27)) (justify left))
   )
-  (hierarchical_label "Chip Select High G Accel" (shape output) (at 158.75 116.84 0) (fields_autoplaced)
-    (effects (font (size 1.27 1.27)) (justify left))
-  )
   (hierarchical_label "SPI1 SCK" (shape output) (at 146.05 109.22 0) (fields_autoplaced)
     (effects (font (size 1.27 1.27)) (justify left))
@@
     (effects (font (size 1.27 1.27)) (justify left))
   )
-  (hierarchical_label "SDMMC Data 2" (shape bidirectional) (at 147.32 170.18 0) (fields_autoplaced)
-    (effects (font (size 1.27 1.27)) (justify left))
-  )
   (hierarchical_label "Channel E Continuity LED" (shape output) (at 82.55 157.48 180) (fields_autoplaced)
     (effects (font (size 1.27 1.27)) (justify right))
@@
     (effects (font (size 1.27 1.27)) (justify left))
   )
-  (hierarchical_label "SDMMC Data 3" (shape bidirectional) (at 147.32 172.72 0) (fields_autoplaced)
+  (hierarchical_label "Magnetometer Interrupt" (shape input) (at 149.86 147.32 0) (fields_autoplaced)
     (effects (font (size 1.27 1.27)) (justify left))
   )
@@
     (effects (font (size 1.27 1.27)) (justify left))
   )
-  (hierarchical_label "High G Interrupt" (shape input) (at 158.75 119.38 0) (fields_autoplaced)
-    (effects (font (size 1.27 1.27)) (justify left))
-  )
   (hierarchical_label "Pyro A Continuity Voltage" (shape input) (at 144.78 58.42 0) (fields_autoplaced)
     (effects (font (size 1.27 1.27)) (justify left))
@@
     (effects (font (size 1.27 1.27)) (justify right))
   )
+  (hierarchical_label "High G Accel Chip Select" (shape output) (at 149.86 180.34 0) (fields_autoplaced)
+    (effects (font (size 1.27 1.27)) (justify left))
+  )
   (hierarchical_label "QSPI IO0" (shape bidirectional) (at 151.13 104.14 0) (fields_autoplaced)

Commit message: STarted layout for v3
Parts:
- R45: value 47k -> 100k
Connections:
- net Altimeter Interrupt: now also U6.98 (PE1); no longer U6.1 (PE2)
- net Chip Select Altimeter: now also U6.97 (PE0); no longer U6.2 (PE3)
- net Chip Select Low G Accel: now also U6.93 (PB7); no longer U6.97 (PE0)
- net High G Accel Chip Select: now also U6.83 (PD2); no longer U6.8 (PC14)
- net High G Accel Interrupt: now also U6.82 (PD1); no longer U6.9 (PC15)
- net Low G Accel Interrupt: now also U6.96 (PB9); no longer U6.98 (PE1)
- net Low G Gyro Interrupt: now also U6.92 (PB6); no longer U6.96 (PB9)
- net Magnetometer Chip Select: now also U6.77 (PA15); no longer U6.15 (PC0)
- net Magnetometer Interrupt: now also U6.81 (PD0); no longer U6.16 (PC1)
- net SPI3 SCK: now reaches U6.78 (PC10)
- net SPI3 MISO: now reaches U6.79 (PC11)
- net SPI3 MOSI: now reaches U6.80 (PC12)
- net SPI2 MISO: no longer names the net of U6.17 (PC2)
- net SPI2 MOSI: no longer names the net of U6.18 (PC3)
- net SPI2 SCK: no longer names the net of U6.52 (PB13)
Other:
- note added: "Pull-up resistors for external I2C bus, 4.7k"
- note removed: "Pull-up resistors for external I2C buss, 4.7k"
