File: _autosave-microcontroller.kicad_sch (KiCad schematic)
At the start: 24 parts, among them Q1 MMBT2222A, U6 STM32L476VETx, Y1 16MHz

Commit message: Updated BOM
Parts:
- D1: value Green -> Blue
Changed lines of the file:
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@@
       (effects (font (size 1.27 1.27)) (justify right))
     )
-    (property "Value" "Green" (at 88.9 171.45 90)
+    (property "Value" "Blue" (at 88.9 171.45 90)
       (effects (font (size 1.27 1.27)) (justify right))
     )
