File: _autosave-power-supply.kicad_sch (KiCad schematic)
At the start: 25 parts, among them Q10 AO3401A, Q9 AO3401A, U8 TPS61230DRC, U9 LM3670MF

Commit message: Updated BOM
Parts:
- D2: value Red -> Green
Changed lines of the file:
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@@
       (effects (font (size 1.27 1.27)) (justify right))
     )
-    (property "Value" "Red" (at 231.14 134.62 90)
+    (property "Value" "Green" (at 231.14 134.62 90)
       (effects (font (size 1.27 1.27)) (justify right))
     )
