File: _autosave-pyro-channels.kicad_sch (KiCad schematic)
At the start: 40 parts, among them J2 Pyro Channels, J3 Screw Switches, Q2 AO3400A, Q3 AO3400A, Q5 AO3400A, Q6 AO3400A, Q7 AO3400A, Q8 AO3400A

Commit message: Updated BOM
Parts:
- D3, D4, D5, D6, D7, D8: footprint LED_SMD:LED_0603_1608Metric_Pad1.05x0.95mm_HandSolder -> LED_SMD:LED_0603_1608Metric
Changed lines of the file:
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@@
       (effects (font (size 1.27 1.27)) (justify right))
     )
-    (property "Footprint" "LED_SMD:LED_0603_1608Metric_Pad1.05x0.95mm_HandSolder" (at 173.99 69.85 0)
+    (property "Footprint" "LED_SMD:LED_0603_1608Metric" (at 173.99 69.85 0)
       (effects (font (size 1.27 1.27)) hide)
     )
@@
       (effects (font (size 1.27 1.27)) (justify right))
     )
-    (property "Footprint" "LED_SMD:LED_0603_1608Metric_Pad1.05x0.95mm_HandSolder" (at 82.55 58.42 0)
+    (property "Footprint" "LED_SMD:LED_0603_1608Metric" (at 82.55 58.42 0)
       (effects (font (size 1.27 1.27)) hide)
     )
@@
       (effects (font (size 1.27 1.27)) (justify right))
     )
-    (property "Footprint" "LED_SMD:LED_0603_1608Metric_Pad1.05x0.95mm_HandSolder" (at 175.26 125.73 0)
+    (property "Footprint" "LED_SMD:LED_0603_1608Metric" (at 175.26 125.73 0)
       (effects (font (size 1.27 1.27)) hide)
     )
@@
       (effects (font (size 1.27 1.27)) (justify right))
     )
-    (property "Footprint" "LED_SMD:LED_0603_1608Metric_Pad1.05x0.95mm_HandSolder" (at 251.46 102.87 0)
+    (property "Footprint" "LED_SMD:LED_0603_1608Metric" (at 251.46 102.87 0)
       (effects (font (size 1.27 1.27)) hide)
     )
@@
       (effects (font (size 1.27 1.27)) (justify right))
     )
-    (property "Footprint" "LED_SMD:LED_0603_1608Metric_Pad1.05x0.95mm_HandSolder" (at 251.46 153.67 0)
+    (property "Footprint" "LED_SMD:LED_0603_1608Metric" (at 251.46 153.67 0)
       (effects (font (size 1.27 1.27)) hide)
     )
@@
       (effects (font (size 1.27 1.27)) (justify right))
     )
-    (property "Footprint" "LED_SMD:LED_0603_1608Metric_Pad1.05x0.95mm_HandSolder" (at 250.19 55.88 0)
-      (effects (font (size 1.27 1.27)) hide)
-    )
+    (property "Footprint" "LED_SMD:LED_0603_1608Metric" (at 250.19 55.88 0)
+      (effects (font (size 1.27 1.27)) hide)
+    )
