File: Flight Computer.kicad_pcb (KiCad board)
At the start: 4 copper layers, 39 x 80 mm, 135 parts, among them J1 Screw Switches, J10 Micro_SD_Card, J2 Pyro Channels, J3 Serial Wire Debug, J4 JST-PH, J7 USB_C_Receptacle_USB2.0, J8 External UART, J9 External I2C, Q1 MMBT2222A, Q2 AO3400A, Q3 AO3400A, Q4 AO3401A, Q5 AO3400A, Q6 AO3400A, Q7 AO3400A, Q8 AO3400A, Q9 AO3401A, U1 STM32L476VETx, U11 SAM-M8Q, U2 USBLC6-2SC6, U7 W25Q128JVSIQ, U8 TPS61230DRC, U9 LM3670MF, Y1 16MHz

Commit message: Now with 100% fewer faulty flyback diodes
Parts:
- removed D10, D11, D12, D13, D14, D9: B5819W SL, Diode_SMD:D_SOD-123
- moved R36 0.53 mm to (136.3, 136.1)
- moved R41 0.48 mm to (136.2, 126.1)
- moved R40 0.37 mm to (136.1, 131.1)
- moved R39 0.30 mm to (136.1, 121.2)
Routing:
- net GND: track 94.7 -> 87.6 mm, vias 88 -> 78
- net /Pyrotechnic Channels/Pyro Channel F: track 13.9 -> 11.1 mm
- net /Pyrotechnic Channels/Pyro Channel E: track 13.9 -> 11.2 mm
- net /Pyrotechnic Channels/Pyro Channel D: track 13.6 -> 11.3 mm
- net /Pyrotechnic Channels/Pyro Channel C: track 13.6 -> 11.2 mm
- net /Pyrotechnic Channels/Pyro Channel B: track 13.1 -> 10.7 mm
- net /Pyrotechnic Channels/Pyro Channel A: track 13.1 -> 10.7 mm
- net /Pyro Channel A Trigger: track 63.9 -> 62.8 mm
- net /Pyro Channel B Trigger: track 58.2 -> 57.3 mm
- net /Pyro Channel C Trigger: track 52.8 -> 52.0 mm
- net /Pyro Channel D Trigger: track 50.0 -> 49.3 mm

Commit message: Updated BOM
Parts:
- added R42: 510k, Resistor_SMD:R_0603_1608Metric, F.Cu at (137.3, 108.0)
- added R43: 100k, Resistor_SMD:R_0402_1005Metric, F.Cu at (141.8, 108.0)
- added R44: 47k, Resistor_SMD:R_0402_1005Metric, F.Cu at (139.8, 108.0)
- D1: value LED -> Green
- D2: value LED -> Red
- D3: moved to F.Cu
- D4, D5, D6, D7, D8: value LED -> White; moved to F.Cu
- moved R39 1.23 mm to (135.8, 120.0)
- moved R36 1.16 mm to (135.8, 135.0)
- moved R41 1.15 mm to (135.8, 125.0)
- moved R40 1.14 mm to (135.8, 130.0)
- moved D4 1.02 mm to (169.6, 118.7), turned to 180 degrees
- moved D5 1.02 mm to (169.6, 123.7), turned to 180 degrees
- moved D8 1.02 mm to (135.1, 123.7), turned to 0 degrees
- moved D3 0.99 mm to (135.1, 133.7), turned to 0 degrees
- moved D7 0.99 mm to (135.1, 128.7), turned to 0 degrees
- moved D6 0.99 mm to (135.1, 118.7), turned to 0 degrees
- moved C29 0.81 mm to (134.8, 96.8)
- moved U7 0.71 mm to (137.3, 102.0)
- moved R38 0.27 mm to (168.8, 122.4)
- moved R37 0.26 mm to (168.8, 117.4)
Connections:
- U9 pad 4: +3.3V -> Net-(U9-FB)
Routing:
- net +3.3V: track 55.4 -> 52.9 mm, vias 29 -> 28
- net Net-(U9-FB): track 0.00 -> 2.29 mm
- net /QSPI Clock: track 21.2 -> 19.8 mm
- net Net-(R42-Pad2): track 0.00 -> 1.26 mm
- net /QSPI IO1: track 17.8 -> 17.0 mm
- net /QSPI IO3: track 12.5 -> 13.3 mm
- net Net-(D6-A): track 2.23 -> 1.58 mm, vias 1 -> 0
- net Net-(D7-A): track 2.22 -> 1.58 mm, vias 1 -> 0
- net Net-(D8-A): track 2.22 -> 1.58 mm, vias 1 -> 0
- net Net-(D3-A): track 2.05 -> 1.58 mm, vias 1 -> 0
- net Net-(D5-A): track 2.05 -> 1.58 mm, vias 1 -> 0
- net Net-(D4-A): track 2.00 -> 1.58 mm, vias 1 -> 0
- net GND: track 87.6 -> 87.3 mm, vias 78 -> 83

Commit message: Updated to match JLC manufacturing capabilities
Routing:
- net /QSPI Clock: track 19.8 -> 21.9 mm
- net +3.3V: track 52.9 -> 54.5 mm, vias 28 -> 29
- net GND: vias 83 -> 84
Changed lines of the file:
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@@
     (fp_line (start 4.47 3.675) (end 4.47 -3.675)
       (stroke (width 0.1) (type solid)) (layer "F.Fab"))
-    (pad "" np_thru_hole circle (at -2.89 -2.605 90) (size 0.65 0.65) (drill 0.65) (layers "*.Cu" "*.Mask"))
-    (pad "" np_thru_hole circle (at 2.89 -2.605 90) (size 0.65 0.65) (drill 0.65) (layers "*.Cu" "*.Mask"))
     (pad "A1" smd rect (at -3.2 -3.725 90) (size 0.6 1.24) (layers "F.Cu" "F.Paste" "F.Mask")
       (net 4 "GND") (pinfunction "GND") (pintype "passive"))
@@
   (segment (start 155.35 99.9625) (end 155.45 99.8625) (width 0.3) (layer "F.Cu") (net 3))
   (segment (start 157.85 83.4625) (end 158.05 83.2625) (width 0.3) (layer "F.Cu") (net 3))
+  (segment (start 135.395 99.645) (end 135.4 99.65) (width 0.286004) (layer "F.Cu") (net 3))
   (segment (start 156.175 84.5625) (end 156.73 84.0075) (width 0.3) (layer "F.Cu") (net 3))
   (segment (start 143.755 99.8875) (end 143.755 100.555) (width 0.25) (layer "F.Cu") (net 3))
@@
   (segment (start 155.025 84.811459) (end 155.273959 84.5625) (width 0.3) (layer "F.Cu") (net 3))
   (segment (start 137.68 78.9375) (end 137.68 79.630497) (width 0.5) (layer "F.Cu") (net 3))
+  (segment (start 135.395 98.4) (end 135.395 99.645) (width 0.286004) (layer "F.Cu") (net 3))
   (segment (start 138.5045 89.4175) (end 139.15 89.4175) (width 0.5) (layer "F.Cu") (net 3))
   (segment (start 140.825 89.5625) (end 139.295 89.5625) (width 0.3) (layer "F.Cu") (net 3))
@@
   (via (at 136.4 109.7625) (size 0.7) (drill 0.3) (layers "F.Cu" "B.Cu") (free) (net 3))
   (via (at 135.97 96.8) (size 0.7) (drill 0.3) (layers "F.Cu" "B.Cu") (net 3))
+  (via (at 135.4 99.65) (size 0.8) (drill 0.4) (layers "F.Cu" "B.Cu") (net 3))
   (via (at 149.23 67.0425) (size 0.8) (drill 0.4) (layers "F.Cu" "B.Cu") (net 3))
-  (via (at 167.55 107) (size 0.8) (drill 0.4) (layers "F.Cu" "B.Cu") (net 3))
+  (via (at 167.55 106.65) (size 0.8) (drill 0.4) (layers "F.Cu" "B.Cu") (net 3))
   (via (at 136.1 113.6125) (size 0.7) (drill 0.3) (layers "F.Cu" "B.Cu") (free) (net 3))
   (via (at 137.737003 79.6875) (size 0.8) (drill 0.4) (layers "F.Cu" "B.Cu") (net 3))
@@
   (via (at 149.99 75.182003) (size 0.8) (drill 0.4) (layers "F.Cu" "B.Cu") (net 3))
   (segment (start 150.7 81.312) (end 150.3005 80.9125) (width 0.3) (layer "B.Cu") (net 3))
-  (segment (start 167.55 107) (end 167.55 108.15) (width 0.25) (layer "B.Cu") (net 3))
   (segment (start 159.8 88.3125) (end 158.65 88.3125) (width 0.3) (layer "B.Cu") (net 3))
   (segment (start 150.7 83.0125) (end 150.7 81.312) (width 0.3) (layer "B.Cu") (net 3))
+  (segment (start 167.55 106.65) (end 167.55 108.15) (width 0.25) (layer "B.Cu") (net 3))
   (segment (start 158.65 88.3125) (end 157.65 89.3125) (width 0.3) (layer "B.Cu") (net 3))
   (segment (start 139.797965 89.0625) (end 139.192965 88.4575) (width 0.3) (layer "F.Cu") (net 4))
@@
   (via (at 138.4 86.0625) (size 0.8) (drill 0.4) (layers "F.Cu" "B.Cu") (net 4))
   (via (at 150.3 105.0125) (size 0.7) (drill 0.3) (layers "F.Cu" "B.Cu") (free) (net 4))
+  (via (at 139.45 104.35) (size 0.8) (drill 0.4) (layers "F.Cu" "B.Cu") (free) (net 4))
   (via (at 149.6 131.3625) (size 0.7) (drill 0.3) (layers "F.Cu" "B.Cu") (free) (net 4))
   (via (at 141.467869 105.017869) (size 0.8) (drill 0.4) (layers "F.Cu" "B.Cu") (free) (net 4))
@@
   (segment (start 141.323959 98.0125) (end 139.5925 98.0125) (width 0.3) (layer "F.Cu") (net 96))
   (segment (start 142.80012 97.0875) (end 142.248959 97.0875) (width 0.3) (layer "F.Cu") (net 96))
+  (segment (start 137.935 98.4) (end 137.935 99.835) (width 0.286004) (layer "F.Cu") (net 97))
   (segment (start 145.8 106.4) (end 150 102.2) (width 0.3) (layer "F.Cu") (net 97))
   (segment (start 144.5 106.4) (end 145.8 106.4) (width 0.3) (layer "F.Cu") (net 97))
+  (segment (start 137.935 99.835) (end 138.4 100.3) (width 0.286004) (layer "F.Cu") (net 97))
   (segment (start 141.9 103.8) (end 144.5 106.4) (width 0.3) (layer "F.Cu") (net 97))
   (segment (start 150 102.2) (end 150 98.2375) (width 0.3) (layer "F.Cu") (net 97))
@@
   (segment (start 163.77 93.5325) (end 165.3 95.0625) (width 0.5) (layer "F.Cu") (net 127))
   (segment (start 170.5 103.1125) (end 170.5 109.398972) (width 0.5) (layer "F.Cu") (net 127))
+  (segment (start 164.075718 84.9025) (end 164.84 84.9025) (width 0.5) (layer "F.Cu") (net 127))
   (segment (start 166.6505 88.8625) (end 166.785 88.997) (width 0.5) (layer "F.Cu") (net 127))
   (segment (start 169.901472 109.9975) (end 168.6625 109.9975) (width 0.5) (layer "F.Cu") (net 127))
@@
   (segment (start 163.82 89.7025) (end 163.77 89.7525) (width 0.5) (layer "F.Cu") (net 127))
   (segment (start 160.35 88.344607) (end 160.35 87.430393) (width 0.3) (layer "F.Cu") (net 127))
+  (segment (start 163.680601 85.297617) (end 164.075718 84.9025) (width 0.5) (layer "F.Cu") (net 127))
   (segment (start 163.19 89.7025) (end 164.84 89.7025) (width 0.3) (layer "F.Cu") (net 127))
   (segment (start 168.6625 108.7575) (end 168.5025 108.5975) (width 0.3) (layer "F.Cu") (net 127))
-  (segment (start 164.84 84.9025) (end 163.94 84.9025) (width 0.5) (layer "F.Cu") (net 127))
   (segment (start 160.282107 88.4125) (end 161.9 88.4125) (width 0.3) (layer "F.Cu") (net 127))
   (segment (start 164.84 89.7025) (end 163.82 89.7025) (width 0.5) (layer "F.Cu") (net 127))
-  (segment (start 163.94 84.9025) (end 163.8 84.7625) (width 0.5) (layer "F.Cu") (net 127))
   (segment (start 162.7 104.5125) (end 169.1 104.5125) (width 0.5) (layer "F.Cu") (net 127))
   (via (at 166.6505 88.8625) (size 0.7) (drill 0.3) (layers "F.Cu" "B.Cu") (net 127))
-  (via (at 163.8 84.7625) (size 0.7) (drill 0.3) (layers "F.Cu" "B.Cu") (net 127))
+  (via (at 163.680601 85.297617) (size 0.7) (drill 0.3) (layers "F.Cu" "B.Cu") (net 127))
+  (segment (start 164.335117 85.297617) (end 166.6505 87.613) (width 0.5) (layer "B.Cu") (net 127))
   (segment (start 166.6505 87.613) (end 166.6505 88.8625) (width 0.5) (layer "B.Cu") (net 127))
-  (segment (start 163.8 84.7625) (end 166.6505 87.613) (width 0.5) (layer "B.Cu") (net 127))
+  (segment (start 163.680601 85.297617) (end 164.335117 85.297617) (width 0.5) (layer "B.Cu") (net 127))
   (segment (start 139.678249 85.0625) (end 136.582875 81.967125) (width 0.25) (layer "F.Cu") (net 132))
   (segment (start 137.760356 75.2875) (end 138.2575 75.784644) (width 0.25) (layer "F.Cu") (net 132))
@@
   )
   (zone (net 4) (net_name "GND") (layer "F.Cu") (hatch edge 0.5)
-    (connect_pads (clearance 0.3))
+    (connect_pads thru_hole_only (clearance 0.3))
     (min_thickness 0.25) (filled_areas_thickness no)
     (fill yes (thermal_gap 0.3) (thermal_bridge_width 0.3))

Commit message: More JLC stuff
Parts:
- moved C7 2.59 mm to (140.0, 81.7), turned to 90 degrees
- moved R3 1.61 mm to (137.9, 81.6)
- moved C11 1.12 mm to (141.3, 81.8), turned to 90 degrees
- moved R20 0.48 mm to (169.9, 80.5)
- moved R21 0.46 mm to (166.7, 80.5)
- moved R11 0.40 mm to (154.3, 117.4)
- moved R13 0.40 mm to (154.2, 122.5)
- moved C28 0.38 mm to (149.8, 67.8)
- moved C4 0.38 mm to (135.8, 77.1)
- moved R12 0.35 mm to (154.3, 119.5)
- moved C8 0.33 mm to (141.3, 70.8)
- moved C5 0.33 mm to (141.9, 76.0), turned to 180 degrees
- moved C3 0.31 mm to (137.2, 79.2)
- moved R22 0.30 mm to (160.5, 114.6)
- moved R5 0.30 mm to (158.5, 114.6)
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Routing:
- net GND: track 87.3 -> 91.9 mm, vias 84 -> 86
- net +3.3V: track 54.5 -> 57.3 mm
- net Net-(U1-BOOT0): track 9.00 -> 10.9 mm
- net /Altimeter Interrupt: track 15.5 -> 16.3 mm
- net /SWCLK: track 45.3 -> 46.2 mm
- net /SWDIO: track 48.2 -> 48.9 mm
- net Net-(J7-CC1): track 9.80 -> 10.3 mm
Other:
- board text added: "JLCJLCJLCJLC"

Commit message: Updated with notes from Erik Welsh
Parts:
- added C25: 0.01u, Capacitor_SMD:C_0402_1005Metric, F.Cu at (162.6, 83.1)
- added G***: LOGO, LOGO, F.Cu at (141.5, 139.3)
- added G***: LOGO, LOGO, B.Cu at (140.0, 109.0)
- added R45: 51k, Resistor_SMD:R_0402_1005Metric, F.Cu at (160.7, 89.2)
- added R46: 200k, Resistor_SMD:R_0402_1005Metric, F.Cu at (158.5, 89.2)
- added R48: 0, Resistor_SMD:R_0402_1005Metric, F.Cu at (135.2, 70.0)
- added R49: 0, Resistor_SMD:R_0402_1005Metric, F.Cu at (137.4, 70.0)
- added R50: 0, Resistor_SMD:R_0402_1005Metric, F.Cu at (135.2, 72.5)
- added R51: 0, Resistor_SMD:R_0402_1005Metric, F.Cu at (137.4, 72.5)
- added R52: 0, Resistor_SMD:R_0402_1005Metric, F.Cu at (135.2, 71.2)
- added R53: 0, Resistor_SMD:R_0402_1005Metric, F.Cu at (137.4, 71.2)
- added R54: 0, Resistor_SMD:R_0402_1005Metric, F.Cu at (135.2, 73.7)
- added R55: 0, Resistor_SMD:R_0402_1005Metric, F.Cu at (137.4, 73.7)
- D1: value Green -> Blue
- D2: value Red -> Green
- D3, D4, D5, D6, D7, D8: footprint LED_SMD:LED_0603_1608Metric_Pad1.05x0.95mm_HandSolder -> LED_SMD:LED_0603_1608Metric
- H1, H2, H3, H4: footprint MountingHole:MountingHole_2mm -> MountingHole:MountingHole_2.2mm_M2
- R17, R24, R36, R37, R38, R39, R40, R41: value 1.5k -> 1k
- moved D1 0.79 mm to (161.0, 92.2)
- moved R17 0.77 mm to (161.0, 90.8)
Connections:
- U1 pad 68: /USB 5V in -> Net-(U1-PA9)
Routing:
- net Net-(J7-SHIELD): track 1.77 -> 21.8 mm
- net /Chip Select High G Accel: track 19.1 -> 30.0 mm
- net /Chip Select Low G Accel: track 17.9 -> 23.9 mm
- net +3.3V: track 57.3 -> 62.4 mm, vias 29 -> 30
- net Net-(U1-PA9): track 0.00 -> 4.76 mm
- net /Chip Select Low G Gyro: track 17.6 -> 22.4 mm, vias 2 -> 3
- net /USB 5V in: track 64.6 -> 61.2 mm
- net /SD Card Detect: track 17.9 -> 14.6 mm
- net GND: track 91.9 -> 94.9 mm, vias 86 -> 91
- net /Chip Select Altimeter: track 20.8 -> 23.5 mm
- net /Pyro B Continuity Voltage: track 41.2 -> 39.6 mm
- net /Pyro D Continuity Voltage: track 27.1 -> 25.9 mm
- net /Pyro C Continuity Voltage: track 35.2 -> 34.0 mm
- net /NRST: track 36.7 -> 35.7 mm
- net /Pyro Channel A Trigger: track 63.0 -> 62.0 mm
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Other:
- board text added: "2023/10/13"
- board text added: "STRIX v1.1"
- board text removed: "2023/10/4"
- board text removed: "Flight Computer V1.1"

Commit message: KiCAD is broken
Parts:
- removed the G*** at (141.5, 139.3)
- removed the G*** at (140.0, 109.0)
- added G***: LOGO, LOGO, F.Cu at (141.8, 139.6)
- added G***: LOGO, LOGO, B.Cu at (141.1, 109.8)
- moved J3 0.97 mm to (144.1, 65.7)
- moved R39 0.70 mm to (136.5, 120.2)
- moved R36 0.65 mm to (136.4, 135.2)
- moved R40 0.65 mm to (136.4, 130.2)
- moved R41 0.65 mm to (136.4, 125.2)
- moved R8 0.33 mm to (150.8, 126.7)
- moved R6 0.30 mm to (150.7, 131.7)
- moved R7 0.20 mm to (150.8, 128.0)
- moved R15 0.16 mm to (150.3, 117.3)
- moved R4 0.15 mm to (150.7, 132.9)
- moved R11 0.14 mm to (154.3, 117.2)
- moved D4 0.11 mm to (169.5, 118.8)
- moved R13 0.10 mm to (154.2, 122.3)
- moved R16 0.07 mm to (150.3, 119.4)
- moved R22 0.07 mm to (160.5, 114.6)
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Routing:
- net GND: track 94.9 -> 92.2 mm, vias 91 -> 98
- net +3.3V: track 62.4 -> 60.1 mm
- net /Pyro A Continuity Voltage: track 46.6 -> 44.7 mm
- net /Pyro B Continuity Voltage: track 39.6 -> 38.4 mm
- net /High G Interrupt: track 18.7 -> 17.6 mm
- net /SWDIO: track 48.5 -> 47.5 mm
- net /SWCLK: track 45.9 -> 45.0 mm
- net /NRST: track 35.7 -> 34.7 mm
Other:
- board text added: "GND"
- board text added: "GND SCL SDA +3.3"
- board text added: "GND TX RX +5"
- board text added: "gnd"
- board text added: "nrst"
- board text added: "swclk"
- board text added: "swdio"
- board text removed: "13"
- board text removed: "14"
- board text removed: "6"
- board text removed: "7"
- board text removed: "8"
- board text removed: "9"
- board text removed: "Gnd SCL SDA +3.3"
- board text removed: "Gnd TX RX +5"
- board text removed: "MISO"
- board text removed: "MOSI"
- board text removed: "NRST"
- board text removed: "QSPI Clk"
- board text removed: "SCK"
- board text removed: "SWCLK"
- board text removed: "SWDIO"

Commit message: Fabrication outputs
Parts:
- removed H1, H2, H3, H4: MountingHole, MountingHole:MountingHole_2.2mm_M2
- R45: value 51k -> 47k
- moved R26 0.75 mm to (165.8, 69.0), turned to -90 degrees
- moved C17 0.49 mm to (163.7, 114.3)
- moved FB2 0.30 mm to (148.8, 110.8)
- moved Q9 0.30 mm to (169.3, 110.9)
- moved C23 0.24 mm to (152.5, 111.0)
- moved C21 0.20 mm to (156.9, 110.6)
- moved C22 0.20 mm to (154.7, 110.6)
- moved L1 0.20 mm to (164.9, 110.4)
- moved F1 0.16 mm to (146.7, 112.0)
- moved U8 0.10 mm to (160.3, 110.5)
Routing:
- net +5V: track 20.2 -> 26.3 mm
- net /SD Card Detect: track 14.6 -> 17.7 mm
- net GND: track 92.2 -> 94.8 mm, vias 98 -> 100
- net +3.3V: track 60.1 -> 61.6 mm, vias 30 -> 31
- net /Chip Select High G Accel: track 29.6 -> 30.9 mm
- net /USB 5V in: track 61.0 -> 62.0 mm
- net /I2C2 SCL: track 45.8 -> 45.1 mm
Other:
- outline, holes or cut-outs redrawn
- board text added: "+"
