File: Flight Computer.kicad_pcb (KiCad board)
At the start: 4 copper layers, 39 x 80 mm, 141 parts, among them J1 Screw Switches, J10 Micro_SD_Card, J2 Pyro Channels, J3 Serial Wire Debug, J4 JST-PH, J7 USB_C_Receptacle_USB2.0, J8 External UART, J9 External I2C, Q1 MMBT2222A, Q2 AO3400A, Q3 AO3400A, Q4 AO3401A, Q5 AO3400A, Q6 AO3400A, Q7 AO3400A, Q8 AO3400A, Q9 AO3401A, U1 STM32L476VETx, U11 SAM-M8Q, U2 USBLC6-2SC6, U7 W25Q128JVSIQ, U8 TPS61230DRC, U9 LM3670MF, Y1 16MHz

Commit message: Minore changes and updates
Parts:
- moved C12 66.6 mm to (109.2, 39.0)
- moved BZ1 66.4 mm to (103.5, 63.2)
- moved C10 66.4 mm to (86.0, 47.8)
- moved C19 66.4 mm to (95.8, 65.6)
- moved C25 66.4 mm to (113.8, 38.1)
- moved C5 66.4 mm to (93.1, 31.0)
- moved C9 66.4 mm to (90.1, 41.5)
- moved D15 66.4 mm to (94.0, 68.5)
- moved D5 66.4 mm to (120.8, 78.7)
- moved J2 66.4 mm to (90.5, 90.5)
- moved Q9 66.4 mm to (120.5, 66.0)
- moved R10 66.4 mm to (101.5, 76.5)
- moved R2 66.4 mm to (89.3, 46.1)
- moved R30 66.4 mm to (107.0, 70.6)
- moved R33 66.4 mm to (99.8, 80.3)
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Routing:
- net /Connectors and Power Supply/USB CONN D-: track 5.45 -> 6.08 mm
- net GND: track 94.8 -> 94.9 mm, vias 100 -> 101
Other:
- outline, holes or cut-outs redrawn
- board text added: "System for Total Real-time In-flight eXecution"

Commit message: Fixed battery polarity
Parts:
- removed the G*** at (93.0, 94.6)
- removed the G*** at (92.3, 64.8)
Connections:
- J4 pad 1: /Main battery connector -> GND
- J4 pad 2: GND -> /Main battery connector
Routing:
- net /Main battery connector: track 20.4 -> 21.2 mm

Commit message: Updating with notes from Adam
Parts:
- removed J3: Serial Wire Debug, Connector_PinHeader_2.54mm:PinHeader_2x02_P2.54mm_Vertical
- added J5: External SPI, Connector_Molex:Molex_PicoBlade_53048-0510_1x05_P1.25mm_Horizontal, F.Cu at (88.8, 32.8)
- added J6: Serial Wire Debug, Connector_Molex:Molex_PicoBlade_53048-0410_1x04_P1.25mm_Horizontal, F.Cu at (99.9, 23.2)
- moved C28 16.1 mm to (117.1, 22.3)
- moved TP6 13.9 mm to (87.6, 25.4)
- moved C3 9.99 mm to (89.2, 24.3), turned to -90 degrees
- moved R48 7.91 mm to (90.8, 18.4)
- moved R49 7.91 mm to (93.0, 18.4)
- moved R50 7.91 mm to (90.8, 20.9)
- moved R51 7.91 mm to (93.0, 20.9)
- moved R52 7.91 mm to (90.8, 19.6)
- moved R53 7.91 mm to (93.0, 19.6)
- moved R54 7.91 mm to (90.8, 22.1)
- moved R55 7.91 mm to (93.0, 22.1)
- moved U5 7.38 mm to (86.8, 26.0), turned to 90 degrees
- moved C4 7.03 mm to (85.2, 25.3)
- moved R3 4.31 mm to (87.3, 40.5), turned to 0 degrees
- moved R26 0.95 mm to (117.8, 24.5), turned to 180 degrees
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Connections:
- U1 pad 17: unconnected-(U1-PC2-Pad17) -> /SPI2 MISO
- U1 pad 18: unconnected-(U1-PC3-Pad18) -> /SPI2 MOSI
- U1 pad 52: unconnected-(U1-PB13-Pad52) -> /SPI2 SCK
Routing:
- net /SPI2 SCK: track 0.00 -> 26.8 mm, vias 0 -> 1
- net /SPI2 MISO: track 0.00 -> 18.3 mm, vias 0 -> 1
- net /SPI2 MOSI: track 0.00 -> 18.1 mm, vias 0 -> 2
- net /Chip Select High G Accel: track 30.9 -> 19.2 mm
- net /NRST: track 34.7 -> 43.9 mm
- net /SPI1 SCK: track 26.6 -> 34.0 mm
- net /SWCLK: track 45.0 -> 52.2 mm
- net /SPI1 MOSI: track 20.2 -> 26.7 mm
- net /Chip Select Low G Accel: track 23.7 -> 17.2 mm
- net /SPI1 MISO: track 23.9 -> 29.5 mm
- net /Chip Select Low G Gyro: track 22.0 -> 17.2 mm, vias 3 -> 2
- net /SWDIO: track 47.5 -> 52.1 mm, vias 1 -> 2
- net /Altimeter Interrupt: track 16.3 -> 19.9 mm, vias 0 -> 2
- net +3.3V: track 61.9 -> 58.6 mm, vias 31 -> 30
- net /Chip Select Altimeter: track 23.7 -> 21.0 mm, vias 1 -> 2
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Other:
- board text removed: "gnd"
- board text removed: "nrst"
- board text removed: "swclk"
- board text removed: "swdio"

Commit message: Finished final(tm) updates for v1.1
Parts:
- added D10: White, LED_SMD:LED_0603_1608Metric, F.Cu at (86.3, 82.7)
- added D11: White, LED_SMD:LED_0603_1608Metric, F.Cu at (86.3, 77.7)
- added D12: White, LED_SMD:LED_0603_1608Metric, F.Cu at (86.3, 72.7)
- added D13: White, LED_SMD:LED_0603_1608Metric, F.Cu at (120.8, 72.7)
- added D14: White, LED_SMD:LED_0603_1608Metric, F.Cu at (120.8, 77.7)
- added D9: White, LED_SMD:LED_0603_1608Metric, F.Cu at (86.3, 87.7)
- added R47: 1k, Resistor_SMD:R_0402_1005Metric, F.Cu at (88.4, 87.5)
- added R56: 1k, Resistor_SMD:R_0402_1005Metric, F.Cu at (88.4, 82.5)
- added R57: 1k, Resistor_SMD:R_0402_1005Metric, F.Cu at (88.4, 77.5)
- added R58: 1k, Resistor_SMD:R_0402_1005Metric, F.Cu at (88.5, 72.5)
- added R59: 1k, Resistor_SMD:R_0402_1005Metric, F.Cu at (118.7, 72.5)
- added R60: 1k, Resistor_SMD:R_0402_1005Metric, F.Cu at (118.7, 77.5)
- D3: value LED -> Red
- D4, D5, D6, D7, D8: value White -> Red
- J4: footprint Connector_JST:JST_PH_B2B-PH-K_1x02_P2.00mm_Vertical -> Connector_JST:JST_PH_S2B-PH-K_1x02_P2.00mm_Horizontal
- moved D2 16.3 mm to (111.6, 37.1)
- moved R24 13.6 mm to (111.8, 38.5)
- moved R48 4.45 mm to (93.2, 22.1), turned to 90 degrees
- moved R51 3.59 mm to (89.5, 19.9), turned to 90 degrees
- moved R55 3.13 mm to (90.8, 19.9), turned to 90 degrees
- moved R52 2.77 mm to (92.0, 22.1), turned to 90 degrees
- moved R38 2.60 mm to (118.7, 79.5), turned to -90 degrees
- moved J4 2.60 mm to (104.5, 90.4)
- moved R37 2.59 mm to (118.7, 74.5), turned to -90 degrees
- moved Q1 2.44 mm to (107.6, 58.2)
- moved R18 1.74 mm to (110.6, 56.9)
- moved R50 1.71 mm to (89.5, 22.1), turned to 90 degrees
- moved R49 1.52 mm to (93.2, 19.9), turned to 90 degrees
- moved D7 1.06 mm to (86.3, 84.7)
- moved R36 1.04 mm to (88.4, 89.5), turned to -90 degrees
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Connections:
- R18 pad 1: Net-(U1-PD13) -> Net-(U1-PB12)
- U1 pad 51: unconnected-(U1-PB12-Pad51) -> Net-(U1-PB12)
- U1 pad 53: unconnected-(U1-PB14-Pad53) -> /Pyro D Continuity LED
- U1 pad 54: unconnected-(U1-PB15-Pad54) -> /Pyro C Continuity LED
- U1 pad 57: unconnected-(U1-PD10-Pad57) -> /Pyro B Continuity LED
- U1 pad 58: unconnected-(U1-PD11-Pad58) -> /Pyro A Continuity LED
- U1 pad 59: unconnected-(U1-PD12-Pad59) -> /Pyro E Continuity LED
- U1 pad 60: Net-(U1-PD13) -> /Pyro F Continuity LED
Routing:
- net /Pyro A Continuity LED: track 0.00 -> 63.6 mm, vias 0 -> 4
- net /Pyro B Continuity LED: track 0.00 -> 57.9 mm, vias 0 -> 4
- net /Pyro C Continuity LED: track 0.00 -> 52.9 mm, vias 0 -> 4
- net /Pyro D Continuity LED: track 0.00 -> 46.2 mm, vias 0 -> 4
- net /Pyro F Continuity LED: track 0.00 -> 36.9 mm, vias 0 -> 2
- net /Pyro E Continuity LED: track 0.00 -> 30.8 mm, vias 0 -> 2
- net Net-(U1-PD13): track 18.4 -> 0.00 mm, vias 2 -> 0
- net /Chip Select Low G Accel: track 17.2 -> 26.8 mm
- net /Chip Select Altimeter: track 21.0 -> 29.2 mm, vias 2 -> 3
- net /Chip Select High G Accel: track 19.2 -> 27.1 mm
- net /Chip Select Low G Gyro: track 17.2 -> 24.1 mm
- net Net-(U1-PB12): track 0.00 -> 5.88 mm
- net /Main battery connector: track 21.2 -> 18.7 mm
- net Net-(BZ1-+): track 8.34 -> 5.82 mm
- net /Pyro C Continuity Voltage: track 34.1 -> 31.9 mm
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Other:
- board text added: "+3.3 MISO MOSI SCK GND"
- board text added: "ADXL 375"
- board text added: "BMI 088"
- board text added: "BMP 388"
- board text added: "Boost"
- board text added: "Buck"
- board text added: "GND DIO CLK RST"
- board text added: "Pyros E,F"
- board text added: "Pyrotechnic Channels A-D"
- board text added: "QSPI Flash"
- board text added: "STM32 L476"
- board text added: "Screw Switches"

Commit message: Added logo and 3D model for 5-pin picoblade
Parts:
- added G***: LOGO, LOGO, B.Cu at (93.2, 64.8)
Other:
- board text added: "2023/10/20"
- board text added: "MISO"
- board text added: "MOSI"
- board text added: "SCK"
- board text removed: "2023/10/13"

Commit message: Finished layout with modified pyro terminal blocks
Parts:
- J1, J2: footprint custom-footprints:Wago_Custom_218-108 -> custom-footprints:Wago_Custom_2601-1108
- moved J4 33.0 mm to (116.2, 59.5), turned to -90 degrees
- moved TP2 31.0 mm to (88.6, 55.6)
- moved R31 12.9 mm to (118.5, 81.9)
- moved R30 12.4 mm to (118.2, 75.8)
- moved R33 11.4 mm to (88.4, 81.9)
- moved R32 11.3 mm to (88.4, 76.2)
- moved R29 9.87 mm to (90.2, 83.1)
- moved Q2 9.48 mm to (90.0, 91.5), turned to 0 degrees
- moved Q3 9.15 mm to (90.0, 85.5), turned to 0 degrees
- moved Q5 8.93 mm to (90.0, 79.5), turned to 0 degrees
- moved Q7 8.88 mm to (117.0, 79.5), turned to 180 degrees
- moved Q8 8.82 mm to (90.0, 73.5), turned to 0 degrees
- moved R34 8.81 mm to (91.0, 89.2)
- moved Q6 8.76 mm to (117.0, 73.5), turned to 180 degrees
- moved J2 6.47 mm to (94.0, 95.9)
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Routing:
- net /Main battery connector: track 18.7 -> 36.3 mm
- net /Pyro Channel A Trigger: track 61.0 -> 50.6 mm
- net GND: track 91.4 -> 101.7 mm
- net /Pyro Channel D Trigger: track 47.5 -> 37.8 mm
- net /Pyro Channel C Trigger: track 50.8 -> 42.3 mm
- net +5V: track 26.3 -> 33.6 mm
- net /Main battery in: track 26.5 -> 32.9 mm
- net /Pyro Channel B Trigger: track 55.8 -> 49.4 mm
- net /Pyro Channel E Trigger: track 40.0 -> 34.4 mm
- net /Pyro Channel F Trigger: track 46.0 -> 40.6 mm
- net /Ignition Battery Voltage: track 41.5 -> 36.8 mm
- net /Pyrotechnic Channels/Pyro Channel A: track 11.2 -> 15.5 mm
- net /UART3 TX: track 13.4 -> 16.5 mm
- net /Pyro D Continuity LED: track 46.2 -> 43.8 mm
- net /Pyro C Continuity LED: track 52.9 -> 51.0 mm
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Other:
- outline, holes or cut-outs redrawn
- board text added: "STRIX v1.2"
- board text removed: "Pyros E,F"
- board text removed: "Pyrotechnic Channels A-D"
- board text removed: "STRIX v1.1"
- board text removed: "Screw Switches"
