File: Flight Computer.kicad_pcb (KiCad board)
At the start: 4 copper layers, 39 x 80 mm, 153 parts, among them J1 Screw Switches, J10 Micro_SD_Card, J2 Pyro Channels, J4 JST-PH, J5 External SPI, J6 Serial Wire Debug, J7 USB_C_Receptacle_USB2.0, J8 External UART, J9 External I2C, Q1 MMBT2222A, Q2 AO3400A, Q3 AO3400A, Q4 AO3401A, Q5 AO3400A, Q6 AO3400A, Q7 AO3400A, Q8 AO3400A, Q9 AO3401A, U1 STM32L476VETx, U11 SAM-M8Q, U2 USBLC6-2SC6, U7 W25Q128JVSIQ, U8 TPS61230DRC, U9 LM3670MF, Y1 16MHz

Commit message: Added new buck converter
Parts:
- removed C17, C21, C22, C23: 22u, Capacitor_SMD:C_0805_2012Metric
- removed C18: 10n, Capacitor_SMD:C_0402_1005Metric
- removed C19: 4.7u, Capacitor_SMD:C_0603_1608Metric
- removed C20: 10u, Capacitor_SMD:C_0805_2012Metric
- removed D15: B5819W SL, Diode_SMD:D_SOD-123
- removed F1: 2920L125PR, Fuse:Fuse_0805_2012Metric
- removed FB2: GZ2012D601TF, Inductor_SMD:L_0805_2012Metric
- removed J6: Serial Wire Debug, Connector_Molex:Molex_PicoBlade_53048-0410_1x04_P1.25mm_Horizontal
- removed L1: 1u, Inductor_SMD:L_Sunlord_SWPA4030S
- removed L2: 10u, Inductor_SMD:L_Sunlord_SWPA4030S
- removed Q4: AO3401A, Package_TO_SOT_SMD:SOT-23
- removed R22, R44: 47k, Resistor_SMD:R_0402_1005Metric
- removed R23: 1M, Resistor_SMD:R_0402_1005Metric
- removed R42: 510k, Resistor_SMD:R_0603_1608Metric
- removed R43: 100k, Resistor_SMD:R_0402_1005Metric
- removed U8: TPS61230DRC, Package_SON:Texas_S-PVSON-N10_ThermalVias
- removed U9: LM3670MF, Package_TO_SOT_SMD:TSOT-23-5
- added C26: 10u, Capacitor_SMD:C_0603_1608Metric, F.Cu at (115.5, 66.1)
- added C27: 33pF, Capacitor_SMD:C_0402_1005Metric, F.Cu at (114.0, 68.1)
- added C30: 10u, Capacitor_SMD:C_0805_2012Metric, F.Cu at (113.2, 63.3)
- added F2: 2920L125PR, Fuse:Fuse_0805_2012Metric, F.Cu at (117.4, 64.2)
- added FB3: GZ2012D601TF, Inductor_SMD:L_0805_2012Metric, F.Cu at (119.4, 64.3)
- added G***: LOGO, LOGO, F.Cu at (96.1, 65.0)
- added J3: External SPI, Connector_Molex:Molex_PicoBlade_53048-0510_1x05_P1.25mm_Horizontal, F.Cu at (100.0, 23.2)
- added L3: 1u, Inductor_SMD:L_Sunlord_SWPA4030S, F.Cu at (109.0, 63.8)
- added U6: ~, Package_TO_SOT_SMD:SOT-563, F.Cu at (112.9, 65.8)
- R1: value 100k -> 200k
- R5: value 200k -> 47k
- moved TP2 21.0 mm to (109.6, 56.9)
- moved TP1 17.0 mm to (114.1, 38.8)
- moved R1 8.81 mm to (112.8, 68.1), turned to 90 degrees
- moved R18 3.14 mm to (106.8, 56.5), turned to 0 degrees
- moved Q9 2.56 mm to (119.3, 68.2), turned to 90 degrees
- moved R5 2.41 mm to (111.6, 68.1), turned to -90 degrees
- moved J4 2.40 mm to (113.0, 58.2)
- moved Q1 1.56 mm to (106.8, 59.3), turned to -90 degrees
- moved C25 1.00 mm to (113.8, 37.1), turned to 90 degrees
- moved TP12 0.96 mm to (114.5, 53.4)
- moved R48 0.79 mm to (92.5, 22.1)
- moved R49 0.79 mm to (92.5, 19.9)
- moved R52 0.79 mm to (91.2, 22.1)
- moved R53 0.79 mm to (91.2, 19.9)
- moved R50 0.79 mm to (88.7, 22.1)
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Connections:
- BZ1 pad 1: +5V -> +3.3V
- J8 pad 1: +5V -> /Main battery in
- Q9 pad 1: /USB 5V in -> GND
- Q9 pad 2: /Connectors and Power Supply/Power Supply/Boost Converter Vin -> /Main battery in
- Q9 pad 3: /Main battery in -> /USB 5V in
- R1 pad 1: /USB 5V in -> +3.3V
- R1 pad 2: GND -> Net-(U6-FB)
- R18 pad 1: Net-(U1-PB12) -> Net-(U1-PE15)
- R28 pad 1: +5V -> +3.3V
- R5 pad 1: +5V -> Net-(U6-FB)
- R5 pad 2: Net-(U8-FB) -> GND
- TP1 pad 1: +5V -> /USB 5V in
- U1 pad 46: unconnected-(U1-PE15-Pad46) -> Net-(U1-PE15)
- U1 pad 51: Net-(U1-PB12) -> unconnected-(U1-PB12-Pad51)
Routing:
- net +5V: track 32.4 -> 0.00 mm, vias 4 -> 0
- net /Main battery in: track 34.0 -> 47.9 mm, vias 1 -> 2
- net /USB 5V in: track 64.4 -> 54.1 mm
- net /Pyro Channel D Trigger: track 37.8 -> 29.3 mm
- net /Pyro F Continuity LED: track 37.6 -> 45.8 mm
- net /Connectors and Power Supply/Power Supply/Buck Vin: track 7.65 -> 0.00 mm
- net /Pyro E Continuity LED: track 32.1 -> 39.6 mm
- net /Pyro Channel C Trigger: track 42.3 -> 35.2 mm
- net /Pyro Channel B Trigger: track 49.4 -> 42.7 mm
- net /Pyro Channel A Trigger: track 50.6 -> 44.2 mm
- net Net-(U1-PB12): track 5.54 -> 0.00 mm
- net +3.3V: track 64.6 -> 69.5 mm, vias 34 -> 28
- net Net-(U1-PE15): track 0.00 -> 4.86 mm
- net Net-(U8-PG): track 4.24 -> 0.00 mm, vias 2 -> 0
- net Net-(U8-FB): track 3.95 -> 0.00 mm
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- removed copper zone on F.Cu, net +3.3V
- removed copper zone on F.Cu, net +5V
- removed copper zone on F.Cu, net /Connectors and Power Supply/Power Supply/Boost Converter SW
- removed copper zone on F.Cu, net /Connectors and Power Supply/Power Supply/Boost Converter Vin
- removed copper zone on F.Cu, net /Connectors and Power Supply/Power Supply/Buck Out
- removed copper zone on F.Cu, net /Connectors and Power Supply/Power Supply/Buck Vin
Other:
- board text added: "GND DIO CLK RST +3.3"
- board text added: "STRIX V2.0"
- board text removed: "+"
- board text removed: "Batt+"
- board text removed: "Boost"
- board text removed: "Buck"
- board text removed: "GND DIO CLK RST"
- board text removed: "STRIX v1.2"

Commit message: finished preliminary v2 modifications
Parts:
- R46: value 200k -> 100k
Connections:
- J8 pad 1: /Main battery in -> /USB 5V in
Routing:
- net /Main battery in: track 47.9 -> 33.7 mm
- net /USB 5V in: track 54.1 -> 57.6 mm
- net GND: track 107.8 -> 109.3 mm, vias 86 -> 84
- net +3.3V: vias 28 -> 35
- added copper zone on F.Cu, net +3.3V
- added copper zone on F.Cu, net /Connectors and Power Supply/Power Supply/Buck_SW
- added copper zone on F.Cu, net /Connectors and Power Supply/Power Supply/Buck_VIN
Other:
- outline, holes or cut-outs redrawn
- board text added: "GND TX RX Bat"
- board text added: "Made with <3 by Rice Eclipse"
- board text removed: "GND TX RX +5"

Commit message: added switch to USB power and to bypass screw switch for main battery
Parts:
- removed the G*** at (96.1, 65.0)
- removed Q9: AO3401A, Package_TO_SOT_SMD:SOT-23
- added D15: D_Schottky, Diode_SMD:D_SOD-323, F.Cu at (118.3, 58.1)
- added SW1: USB Disconnect, Button_Switch_SMD:SW_SPDT_PCM12, F.Cu at (119.3, 64.4)
- added SW2: Screw Switch Bypass, Button_Switch_SMD:SW_SPDT_PCM12, F.Cu at (119.3, 88.1)
- added U8: MAX40200AUK, Package_TO_SOT_SMD:SOT-23-5, F.Cu at (115.0, 89.2)
- TP1: value 5V -> Buck In
- moved TP2 23.8 mm to (85.9, 56.6), turned to -90 degrees
- moved FB3 6.43 mm to (116.1, 69.9), turned to 180 degrees
- moved F2 3.70 mm to (115.1, 67.1), turned to 90 degrees
- moved R18 3.11 mm to (109.6, 58.0), turned to -90 degrees
- moved C26 2.39 mm to (114.9, 63.8), turned to 90 degrees
- moved R1 0.98 mm to (111.8, 68.1)
- moved R5 0.98 mm to (110.6, 68.1)
- moved C27 0.98 mm to (113.0, 68.0)
- moved C30 0.96 mm to (112.3, 63.4)
- moved L3 0.91 mm to (108.0, 63.8)
- moved U6 0.86 mm to (112.1, 65.8)
- moved J4 0.83 mm to (113.8, 57.9)
- moved Q1 0.38 mm to (106.8, 58.9), turned to 180 degrees
Connections:
- FB3 pad 1: /USB 5V in -> /Connectors and Power Supply/Vin_combined
- J8 pad 1: /USB 5V in -> /Connectors and Power Supply/Vin_combined
- TP1 pad 1: /USB 5V in -> /Connectors and Power Supply/Vin_combined
Routing:
- net /Connectors and Power Supply/Vin_combined: track 0.00 -> 26.2 mm, vias 0 -> 2
- net /Main battery in: track 33.7 -> 13.8 mm, vias 2 -> 0
- net /USB 5V in: track 57.6 -> 42.8 mm
- net Net-(D15-K): track 0.00 -> 6.64 mm
- net /Main battery connector: track 40.5 -> 46.3 mm
- net Net-(U1-PE15): track 4.86 -> 8.70 mm
- net GND: track 109.3 -> 107.3 mm, vias 84 -> 86
- net +3.3V: track 69.5 -> 68.1 mm
- net Net-(BZ1-+): track 7.16 -> 6.31 mm
- net /Pyro D Continuity LED: track 43.8 -> 43.0 mm
- net Net-(Q1-B): track 1.90 -> 2.50 mm
- net /Pyro C Continuity LED: track 51.0 -> 50.5 mm
Other:
- board text added: "2023/11/18"
- board text added: "Main battery"
- board text added: "USB Power"
- board text added: "off"
- board text added: "on"
- board text removed: "2023/10/23"
- board text removed: "Made with <3 by Rice Eclipse"

Commit message: Fixed BOM
Parts:
- moved R18 0.38 mm to (110.0, 58.0)
- moved Q1 0.34 mm to (107.1, 58.9)
Routing:
- net /Connectors and Power Supply/Vin_combined: track 26.2 -> 27.1 mm
- net /Pyro D Continuity Voltage: track 26.2 -> 25.6 mm

Commit message: Finished DRC
Parts:
- moved TP1 18.1 mm to (110.3, 56.5)
Routing:
- net /Connectors and Power Supply/Vin_combined: track 27.1 -> 52.9 mm
- net /USB 5V in: track 42.8 -> 40.7 mm
- net +3.3V: track 68.1 -> 69.2 mm
Other:
- board text added: "Vin"
- board text removed: "5V"
